File: hardware/tach_sensor.sch (KiCad schematic (older format))
At the start: 2 parts

Commit message: work in progress - components ordered
Connections:
- net labels added: +5VA
- net labels removed: +5V
Changed lines of the file:
@@
 $Descr A4 11693 8268
 encoding utf-8
-Sheet 9 18
+Sheet 9 17
 Title ""
 Date ""
@@
 Text HLabel 4500 3750 0    50   Input ~ 0
 HALL_SENSOR-
-$Comp
-L power:+5V #PWR029
-U 1 1 5C6646A4
-P 4600 3200
-F 0 "#PWR029" H 4600 3050 50  0001 C CNN
-F 1 "+5V" H 4615 3373 50  0000 C CNN
-F 2 "" H 4600 3200 50  0001 C CNN
-F 3 "" H 4600 3200 50  0001 C CNN
-	1    4600 3200
-	1    0    0    -1
-$EndComp
 Wire Wire Line
 	4600 3200 4600 3250
@@
 	1    0    0    -1
 $EndComp
+$Comp
+L power:+5VA #PWR018
+U 1 1 5C78A732
+P 4600 3200
+F 0 "#PWR018" H 4600 3050 50  0001 C CNN
+F 1 "+5VA" H 4615 3373 50  0000 C CNN
+F 2 "" H 4600 3200 50  0001 C CNN
+F 3 "" H 4600 3200 50  0001 C CNN
+	1    4600 3200
+	1    0    0    -1
+$EndComp
