File: hardware/speeduino_mini.kicad_pcb (KiCad board)
At the start: 2 copper layers, 102 parts, among them J1 O2, J10 Injector 4, J11 Injectors, J12 oil pressure, J13 oil pressure, J3 TPS, J4 IAT, J5 head temperature, J6 crank hall, J7 Injector 1, J8 Injector 2, J9 Injector 3, Q1 SQ2318AES-T1_GE3, Q2 SQ2318AES-T1_GE3, Q3 2N7002, Q4 Q_NMOS_DGS, Q5 SQ3457EV, U1 TPD4E001-Q1, U2 TPD4E001-Q1, U3 ATmega2561-16AU, U4 MPX4250AP1, U5 TC4424_SOIC, U6 TPD2E001-SOT-5, U7 RT7258, U8 LD1117S50TR_SOT223, Y1 CSTCE16M0V53-R0

Commit message: work in progress - components ordered
Parts:
- removed ICSP1: ICSP, Pin_Headers:Pin_Header_Straight_2x03_Pitch2.54mm_SMD
- added C38: 22uF, Capacitors_SMD:C_0805, F.Cu at (378.0, 101.6)
- added C39: 1u, Capacitors_SMD:C_0805, F.Cu at (378.0, 103.5)
- added C40: 22nF, Capacitors_SMD:C_0805, F.Cu at (379.9, 116.3)
- added C41: 220nF, Capacitors_SMD:C_0805, F.Cu at (381.4, 105.5)
- added C42: 0.22u, Capacitors_SMD:C_0805, F.Cu at (265.0, 150.9)
- added C43: 220pF, Capacitors_SMD:C_0805, F.Cu at (202.4, 31.9)
- added D3: ACGRKM4007-HF, Diodes_SMD:D_SOD-123F, F.Cu at (361.6, 112.5)
- added D4: D_Schottky, Diodes_SMD:D_SOD-323F, F.Cu at (381.5, 103.6)
- added D5: D_Zener, Diodes_SMD:D_SOD-323, F.Cu at (202.3, 29.8)
- added D6: D, Diodes_SMD:D_SOD-123, F.Cu at (202.4, 25.7)
- added J14: power, Speeduino Mini:ED120_3DS, F.Cu at (354.5, 109.6)
- added J2: Raspberry_Pi_2_3, Speeduino Mini:RaspberryPi_uHAT, F.Cu at (473.5, 51.0)
- added L3: 47uH, Speeduino Mini:BOURNS_SRR1260, F.Cu at (369.4, 109.6)
- added L4: 47uH, Speeduino Mini:BOURNS_SRR1260, F.Cu at (389.9, 109.6)
- added PC3: 47uF, Capacitors_SMD:C_1206, F.Cu at (397.6, 109.7)
- added PC4: 47uF, Capacitors_SMD:C_1206, F.Cu at (400.1, 109.7)
- added R25: 22k, Resistors_SMD:R_0805, F.Cu at (377.8, 116.3)
- added R26: 470, Resistors_SMD:R_0805, F.Cu at (264.8, 152.7)
- added R30: 47, Resistors_SMD:R_0805, F.Cu at (202.4, 27.8)
- added U10: SN74LVC2T45-VSSOP, Housings_SSOP:VSSOP-8_2.3x2mm_Pitch0.5mm, F.Cu at (463.9, 57.9)
- added U11: TLE8366, Housings_SOIC:SOIC-8-1EP_3.9x4.9mm_Pitch1.27mm, F.Cu at (379.5, 110.4)
- added U12: MCP2003B, Housings_SOIC:SOIC-8_3.9x4.9mm_Pitch1.27mm, F.Cu at (196.7, 29.7)
- added U9: SN74LVC2T45-VSSOP, Housings_SSOP:VSSOP-8_2.3x2mm_Pitch0.5mm, F.Cu at (461.4, 51.3)
- C21: value 0.01u -> 0.1uF
- C22: value 1u -> 100nF
- C37: value 100nF -> 22uF
- J11: value Injectors -> Ignitor Pack
- J6: value crank hall -> crankshaft position sensor; footprint Speeduino Mini:ED120_2DS -> Speeduino Mini:ED120_3DS
- R16: value 1k -> 10k
- R21, R22: value 150 -> 10k
- R23: value 10k -> 150
- R27: value 160 -> 33k; footprint Resistors_SMD:R_2512 -> Resistors_SMD:R_0805
- R28: value 160 -> 4k7; footprint Resistors_SMD:R_2512 -> Resistors_SMD:R_0805
- U5: value TC4424_SOIC -> SN74LVC2T45-VSSOP; footprint Housings_SOIC:SOIC-16W_7.5x10.3mm_Pitch1.27mm -> Housings_SSOP:VSSOP-8_2.3x2mm_Pitch0.5mm
- moved J3 431.4 mm to (436.0, 184.2), turned to 90 degrees
- moved J4 424.3 mm to (436.0, 171.5), turned to 90 degrees
- moved J5 419.6 mm to (436.0, 161.3), turned to 90 degrees
- moved J6 415.5 mm to (436.0, 148.6), turned to 90 degrees
- moved C12 415.3 mm to (428.4, 181.6), turned to 90 degrees
- moved R8 415.3 mm to (427.2, 185.5), turned to 0 degrees
- moved J12 412.2 mm to (436.0, 133.4), turned to 90 degrees
- moved R2 410.9 mm to (428.4, 174.0), turned to 90 degrees
- moved J13 410.7 mm to (436.0, 118.1), turned to 90 degrees
- moved C13 410.5 mm to (425.9, 181.6), turned to 90 degrees
- moved C14 408.3 mm to (428.4, 168.9), turned to 90 degrees
- moved C15 407.1 mm to (427.2, 171.5), turned to 0 degrees
- moved R4 405.8 mm to (428.4, 163.9), turned to 90 degrees
- moved C17 403.7 mm to (428.4, 158.8), turned to 90 degrees
- moved R3 403.3 mm to (425.9, 168.9), turned to 90 degrees
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Connections:
- C1 pad 1: +5VA -> +5VD
- C16 pad 1: +5V -> +5VD
- C2 pad 1: /MCU/RESET -> /Raspberry Pi Zero W/ATMEGA_RESET
- C21 pad 1: /Crank sensor/CRANK_Output -> /Crankshaft pos sensor/IN
- C22 pad 1: +5V -> +5VD
- C3 pad 1: +5VA -> +5VD
- C36 pad 1: +5V -> Net-(C36-Pad1)
- C37 pad 1: +5VA -> Net-(C37-Pad1)
- C5 pad 1: +5V -> +5VD
- C6 pad 1: +5V -> +5VD
- D1 pad 1: +5V -> +5VD
- D1 pad 2: /MCU/RESET -> /Raspberry Pi Zero W/ATMEGA_RESET
- J11 pad 1: /Ignitor/IGN1_OUT -> /MCU/OC1A
- J11 pad 3: /Ignitor/IGN2_OUT -> /MCU/OC1B
- J6 pad 1: /Crank sensor/HALL_SENSOR+ -> +5VA
- J6 pad 2: /Crank sensor/CRANK_Output -> /Crankshaft pos sensor/IN
- L2 pad 1: +5V -> +5VD
- L2 pad 2: +5VA -> Net-(C36-Pad1)
- PC2 pad 1: +5V -> +5VD
- R16 pad 1: +5V -> /Power/EN
- R16 pad 2: /Crank sensor/HALL_SENSOR+ -> Net-(C38-Pad1)
- R21 pad 1: Net-(R21-Pad1) -> GND
- R21 pad 2: /Ignitor/IGN1_IN -> /MCU/OC1B
- R22 pad 1: Net-(R22-Pad1) -> GND
- R22 pad 2: /Ignitor/IGN2_IN -> /MCU/OC1A
- R23 pad 1: GND -> Net-(R23-Pad1)
- R23 pad 2: Net-(R21-Pad1) -> /Raspberry Pi Zero W/ATMEGA_RESET
- R24 pad 1: GND -> Net-(J2-Pad16)
- R24 pad 2: Net-(R22-Pad1) -> Net-(J2-Pad1)
- R27 pad 1: /Ignitor/IGN1_OUT -> Net-(R27-Pad1)
- R27 pad 2: Net-(R27-Pad2) -> +12V
- R28 pad 1: /Ignitor/IGN2_OUT -> +5VD
- R28 pad 2: Net-(R28-Pad2) -> /Lin transceiver/RXD
- RN5A1 pad 1: +5V -> +5VD
- RN5A1 pad 2: /MCU/RESET -> /Raspberry Pi Zero W/ATMEGA_RESET
- U1 pad 5: +5VA -> +5VD
- U2 pad 5: +5VA -> +5VD
- U3 pad 1: (no net) -> /MCU/OC0B
- U3 pad 10: (no net) -> Net-(U3-Pad10)
- U3 pad 12: /MCU/MOSI -> Net-(U3-Pad12)
- U3 pad 13: /MCU/MISO -> Net-(U3-Pad13)
- U3 pad 14: (no net) -> /MCU/OC2A
- U3 pad 15: /Ignitor/IGN1_IN -> /MCU/OC1A
- U3 pad 16: /Ignitor/IGN2_IN -> /MCU/OC1B
- U3 pad 17: (no net) -> /Power/EN
- U3 pad 18: (no net) -> Net-(U3-Pad18)
- U3 pad 19: (no net) -> Net-(U3-Pad19)
- U3 pad 2: (no net) -> /MCU/RXD0
- U3 pad 20: /MCU/RESET -> /Raspberry Pi Zero W/ATMEGA_RESET
- U3 pad 21: +5V -> +5VD
- U3 pad 26: /Crank sensor/CRANK_Output -> /MCU/INT1
- U3 pad 27: (no net) -> /Lin transceiver/RXD
- U3 pad 28: (no net) -> /Lin transceiver/TXD
- U3 pad 29: (no net) -> Net-(U3-Pad29)
- U3 pad 3: (no net) -> /Raspberry Pi Zero W/RXD_PDO
- U3 pad 30: (no net) -> Net-(U3-Pad30)
- U3 pad 31: (no net) -> Net-(U3-Pad31)
- U3 pad 32: (no net) -> Net-(U3-Pad32)
- U3 pad 33: (no net) -> Net-(U3-Pad33)
- U3 pad 34: (no net) -> Net-(U3-Pad34)
- U3 pad 35: (no net) -> Net-(U3-Pad35)
- U3 pad 36: (no net) -> Net-(U3-Pad36)
- U3 pad 37: (no net) -> Net-(U3-Pad37)
- U3 pad 38: (no net) -> Net-(U3-Pad38)
- U3 pad 39: (no net) -> Net-(U3-Pad39)
- U3 pad 4: (no net) -> Net-(U3-Pad4)
- U3 pad 40: (no net) -> Net-(U3-Pad40)
- U3 pad 41: (no net) -> Net-(U3-Pad41)
- U3 pad 42: (no net) -> Net-(U3-Pad42)
- U3 pad 43: (no net) -> Net-(U3-Pad43)
- U3 pad 44: (no net) -> Net-(U3-Pad44)
- U3 pad 45: (no net) -> Net-(U3-Pad45)
- U3 pad 46: (no net) -> Net-(U3-Pad46)
- U3 pad 47: (no net) -> Net-(U3-Pad47)
- U3 pad 48: (no net) -> Net-(U3-Pad48)
- U3 pad 49: (no net) -> Net-(U3-Pad49)
- U3 pad 50: (no net) -> Net-(U3-Pad50)
- U3 pad 52: +5V -> +5VD
- U3 pad 64: +5VA -> Net-(C36-Pad1)
- U3 pad 8: (no net) -> Net-(U3-Pad8)
- U3 pad 9: (no net) -> Net-(U3-Pad9)
- U5 pad 1: (no net) -> +5VD
- U5 pad 2: Net-(R21-Pad1) -> /MCU/RXD0
- U5 pad 3: (no net) -> /MCU/SCK
- U5 pad 6: (no net) -> Net-(J2-Pad12)
- U5 pad 7: Net-(R22-Pad1) -> Net-(J2-Pad8)
- U5 pad 8: (no net) -> Net-(J2-Pad1)
- U6 pad 1: +5V -> +5VD
- U6 pad 5: /Crank sensor/CRANK_Output -> /MCU/INT1
- U8 pad 2: +5V -> +5VD
Other:
- board outline added: 100 x 100 mm
- board text added: "DigiKey 377-2312-ND https://www.budind.com/pdf/hbext9166.pdf"

Commit message: rev 1
Parts:
- removed R21, R22: 10k, Resistors_SMD:R_0805
- added C44: 0.1uF, Capacitors_SMD:C_0805, F.Cu at (148.6, 127.0)
- added C45: 0.22u, Capacitors_SMD:C_0805, F.Cu at (144.8, 127.0)
- added D7: ACGRKM4007-HF, Diodes_SMD:D_SOD-123F, F.Cu at (83.4, 86.4)
- added D8: ACGRKM4007-HF, TO_SOT_Packages_SMD:TO-277A, F.Cu at (84.3, 103.3)
- added J15: camshaft position sensor, Speeduino Mini:ED120_3DS, F.Cu at (142.9, 133.3)
- added Q6: SQ2318AES-T1_GE3, TO_SOT_Packages_SMD:SOT-23, F.Cu at (122.6, 126.2)
- added Q7: SQ2318AES-T1_GE3, TO_SOT_Packages_SMD:SOT-23, F.Cu at (132.7, 126.2)
- added R31: 33k, Resistors_SMD:R_0805, F.Cu at (88.0, 111.3)
- added R32: 470, Resistors_SMD:R_0805, F.Cu at (141.0, 127.0)
- added R33: 10k, Resistors_SMD:R_0805, F.Cu at (119.8, 124.2)
- added R34: 150, Resistors_SMD:R_0805, F.Cu at (122.6, 123.4)
- added R35: 10k, Resistors_SMD:R_0805, F.Cu at (129.8, 124.3)
- added R36: 150, Resistors_SMD:R_0805, F.Cu at (132.7, 123.3)
- D4: footprint Diodes_SMD:D_SOD-323F -> Diodes_SMD:D_SOD-123F
- J13: value oil pressure -> fuel pressure
- J2, U4: moved to B.Cu
- PC1: footprint Capacitors_Tantalum_SMD:CP_Tantalum_Case-R_EIA-2012-12_Reflow -> Capacitors_Tantalum_SMD:CP_Tantalum_Case-C_EIA-6032-28_Reflow
- U6: value TPD2E001-SOT-5 -> TPD4E001-Q1; footprint TO_SOT_Packages_SMD:SOT-553 -> TO_SOT_Packages_SMD:SOT-23-6
- moved J4 354.6 mm to (104.8, 45.1), turned to 180 degrees
- moved C15 347.2 mm to (101.1, 52.1), turned to 90 degrees
- moved C14 345.3 mm to (103.5, 52.1), turned to 270 degrees
- moved R2 342.3 mm to (108.6, 52.1)
- moved J5 341.5 mm to (114.9, 45.1), turned to 180 degrees
- moved R3 340.5 mm to (106.0, 52.1)
- moved J3 338.3 mm to (127.6, 45.1), turned to 180 degrees
- moved C18 332.4 mm to (111.1, 52.1)
- moved C17 332.4 mm to (113.7, 52.1), turned to 270 degrees
- moved C13 330.7 mm to (121.9, 51.4), turned to 0 degrees
- moved R5 329.6 mm to (116.2, 52.1), turned to 90 degrees
- moved C12 329.5 mm to (125.7, 51.4), turned to 180 degrees
- moved R4 329.2 mm to (118.7, 52.1)
- moved R8 326.4 mm to (129.5, 51.4), turned to 180 degrees
- moved J2 308.9 mm to (167.0, 89.2), turned to 90 degrees
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Connections:
- net /MCU/INT0 renamed /Camshaft position sensor/IN
- C11 pad 1: /MCU/A3 -> /MCU/A4
- C13 pad 1: /MCU/A2 -> /MCU/A5
- C15 pad 1: /MCU/A0 -> /MCU/A2
- C18 pad 1: /MCU/A1 -> /MCU/A3
- C20 pad 1: /MCU/A4 -> /MCU/A0
- C24 pad 1: +12V -> Net-(C24-Pad1)
- C25 pad 1: +12V -> Net-(C24-Pad1)
- C32 pad 1: /MCU/A5 -> /MCU/A6
- C34 pad 1: /MCU/A6 -> /MCU/A7
- C8 pad 1: /MCU/A7 -> /MCU/A1
- J10 pad 2: /Injector 2 and 4/INJ_OUT -> /Injector 4/INJ_OUT
- J11 pad 1: /MCU/OC1A -> /MCU/OC0B
- J11 pad 3: /MCU/OC1B -> /MCU/OC3A
- J2 pad 11: Net-(J2-Pad11) -> (no net)
- J2 pad 12: Net-(J2-Pad12) -> (no net)
- J2 pad 13: Net-(J2-Pad13) -> (no net)
- J2 pad 15: Net-(J2-Pad15) -> (no net)
- J2 pad 18: Net-(J2-Pad18) -> (no net)
- J2 pad 19: Net-(J2-Pad19) -> (no net)
- J2 pad 21: Net-(J2-Pad21) -> (no net)
- J2 pad 22: Net-(J2-Pad22) -> (no net)
- J2 pad 23: Net-(J2-Pad23) -> (no net)
- J2 pad 24: Net-(J2-Pad24) -> (no net)
- J2 pad 26: Net-(J2-Pad26) -> (no net)
- J2 pad 27: Net-(J2-Pad27) -> (no net)
- J2 pad 28: Net-(J2-Pad28) -> (no net)
- J2 pad 29: Net-(J2-Pad29) -> (no net)
- J2 pad 3: Net-(J2-Pad3) -> (no net)
- J2 pad 32: Net-(J2-Pad32) -> (no net)
- J2 pad 35: Net-(J2-Pad35) -> (no net)
- J2 pad 36: Net-(J2-Pad36) -> (no net)
- J2 pad 37: Net-(J2-Pad37) -> (no net)
- J2 pad 38: Net-(J2-Pad38) -> (no net)
- J2 pad 40: Net-(J2-Pad40) -> (no net)
- J2 pad 5: Net-(J2-Pad5) -> (no net)
- J2 pad 7: Net-(J2-Pad7) -> (no net)
- J7 pad 2: /Injector 1 and 3/INJ_OUT -> /Injector 1/INJ_OUT
- J8 pad 2: /Injector 2 and 4/INJ_OUT -> /Injector 2/INJ_OUT
- J9 pad 2: /Injector 1 and 3/INJ_OUT -> /Injector 3/INJ_OUT
- Q1 pad 2: /Injector 1 and 3/INJ_OUT -> GND
- Q1 pad 3: GND -> /Injector 1/INJ_OUT
- Q2 pad 2: /Injector 2 and 4/INJ_OUT -> GND
- Q2 pad 3: GND -> /Injector 2/INJ_OUT
- R10 pad 1: /MCU/A6 -> /MCU/A7
- R15 pad 1: /MCU/A4 -> /MCU/A0
- R17 pad 1: /Injector 1 and 3/INJ_CMD -> /Injector 1/INJ_CMD
- R18 pad 2: /Injector 1 and 3/INJ_CMD -> /Injector 1/INJ_CMD
- R19 pad 1: /Injector 2 and 4/INJ_CMD -> /Injector 2/INJ_CMD
- R20 pad 2: /Injector 2 and 4/INJ_CMD -> /Injector 2/INJ_CMD
- R3 pad 1: /MCU/A0 -> /MCU/A2
- R5 pad 1: /MCU/A1 -> /MCU/A3
- R6 pad 1: /MCU/A7 -> /MCU/A1
- R7 pad 1: /MCU/A3 -> /MCU/A4
- R8 pad 1: /MCU/A2 -> /MCU/A5
- R9 pad 1: /MCU/A5 -> /MCU/A6
- U1 pad 3: /MCU/A2 -> /MCU/A0
- U1 pad 6: /MCU/A0 -> /MCU/A2
- U10 pad 1: +5VD -> Net-(J2-Pad1)
- U10 pad 2: +5VD -> Net-(J2-Pad31)
- U10 pad 3: /Raspberry Pi Zero W/RXD_PDO -> Net-(J2-Pad10)
- U10 pad 5: +5VD -> GND
- U10 pad 6: Net-(J2-Pad10) -> /Raspberry Pi Zero W/RXD_PDO
- U10 pad 7: Net-(J2-Pad18) -> +5VD
- U10 pad 8: Net-(J2-Pad1) -> +5VD
- U11 pad 9: (no net) -> GND
- U12 pad 2: /Lin transceiver/CS -> Net-(R31-Pad1)
- U12 pad 8: Net-(U12-Pad8) -> (no net)
- U2 pad 1: /MCU/A5 -> /MCU/A7
- U2 pad 4: /MCU/A7 -> /MCU/A5
- U3 pad 10: Net-(U3-Pad10) -> (no net)
- U3 pad 12: Net-(U3-Pad12) -> (no net)
- U3 pad 13: Net-(U3-Pad13) -> (no net)
- U3 pad 14: /MCU/OC2A -> (no net)
- U3 pad 15: /MCU/OC1A -> /Injector 3/INJ_CMD
- U3 pad 16: /MCU/OC1B -> /Injector 4/INJ_CMD
- U3 pad 18: Net-(U3-Pad18) -> (no net)
- U3 pad 19: Net-(U3-Pad19) -> (no net)
- U3 pad 29: Net-(U3-Pad29) -> (no net)
- U3 pad 30: Net-(U3-Pad30) -> (no net)
- U3 pad 31: Net-(U3-Pad31) -> (no net)
- U3 pad 32: Net-(U3-Pad32) -> (no net)
- U3 pad 33: Net-(U3-Pad33) -> (no net)
- U3 pad 34: Net-(U3-Pad34) -> (no net)
- U3 pad 35: Net-(U3-Pad35) -> (no net)
- U3 pad 36: Net-(U3-Pad36) -> (no net)
- U3 pad 37: Net-(U3-Pad37) -> (no net)
- U3 pad 38: Net-(U3-Pad38) -> (no net)
- U3 pad 39: Net-(U3-Pad39) -> (no net)
- U3 pad 4: Net-(U3-Pad4) -> (no net)
- U3 pad 40: Net-(U3-Pad40) -> (no net)
- U3 pad 41: Net-(U3-Pad41) -> (no net)
- U3 pad 42: Net-(U3-Pad42) -> (no net)
- U3 pad 43: Net-(U3-Pad43) -> (no net)
- U3 pad 44: Net-(U3-Pad44) -> (no net)
- U3 pad 45: Net-(U3-Pad45) -> (no net)
- U3 pad 46: Net-(U3-Pad46) -> (no net)
- U3 pad 47: Net-(U3-Pad47) -> (no net)
- U3 pad 48: Net-(U3-Pad48) -> (no net)
- U3 pad 49: Net-(U3-Pad49) -> (no net)
- U3 pad 5: /Injector 1 and 3/INJ_CMD -> /MCU/OC3A
- U3 pad 50: Net-(U3-Pad50) -> (no net)
- U3 pad 6: /Injector 2 and 4/INJ_CMD -> /Injector 1/INJ_CMD
- U3 pad 7: /Injector Power Supply/EN -> /Injector 2/INJ_CMD
- U3 pad 8: Net-(U3-Pad8) -> (no net)
- U3 pad 9: Net-(U3-Pad9) -> /Injector Power Supply/EN
- U5 pad 6: Net-(J2-Pad12) -> Net-(J2-Pad33)
- U6 pad 1: +5VD -> /MCU/INT1
- U6 pad 2: (no net) -> GND
- U6 pad 4: GND -> (no net)
- U6 pad 5: /MCU/INT1 -> +5VD
- U7 pad 8: +12V -> Net-(C24-Pad1)
- U9 pad 3: Net-(U9-Pad3) -> (no net)
Routing:
- net +5VA: track 0.00 -> 356.7 mm, vias 0 -> 11
- net GND: track 0.00 -> 305.0 mm, vias 0 -> 36
- net +5VD: track 0.00 -> 186.1 mm, vias 0 -> 10
- net +12V: track 0.00 -> 123.8 mm
- net /Injector Power Supply/VOUT: track 0.00 -> 95.7 mm, vias 0 -> 4
- net /O2 Sensor Power/EN: track 0.00 -> 87.5 mm, vias 0 -> 2
- net /Raspberry Pi Zero W/ATMEGA_RESET: track 0.00 -> 76.4 mm, vias 0 -> 2
- net /MCU/A7: track 0.00 -> 70.5 mm, vias 0 -> 2
- net /MCU/A5: track 0.00 -> 58.8 mm
- net /MCU/A2: track 0.00 -> 58.4 mm
- net /MCU/A6: track 0.00 -> 58.1 mm
- net /MCU/INT1: track 0.00 -> 55.5 mm, vias 0 -> 2
- net /MCU/A1: track 0.00 -> 54.8 mm
- net /MCU/A3: track 0.00 -> 54.8 mm
- net /Power/EN: track 0.00 -> 51.8 mm, vias 0 -> 2
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- added copper zone on B.Cu, net GND
Other:
- board text added: "VW Bus ECU rev 1 Based on Speeduino 2019 Cedric Priscal"
- board text added: "https://github.com/cepr/vw-bus-project-ecu"

Commit message: Adding corrections for wrong raspberry pi pinout
Parts:
- D8: value ACGRKM4007-HF -> PMEG060V100EPDZ
Connections:
- J2 pad 11: (no net) -> GND
- J2 pad 15: (no net) -> Net-(J2-Pad15)
- J2 pad 18: (no net) -> Net-(J2-Pad18)
- J2 pad 19: (no net) -> Net-(J2-Pad10)
- J2 pad 27: (no net) -> GND
- J2 pad 33: Net-(J2-Pad33) -> Net-(J2-Pad1)
- J2 pad 8: Net-(J2-Pad8) -> Net-(J2-Pad15)
- R24 pad 1: Net-(J2-Pad16) -> Net-(J2-Pad31)
- U10 pad 2: Net-(J2-Pad31) -> Net-(J2-Pad18)
- U5 pad 6: Net-(J2-Pad33) -> Net-(J2-Pad16)
- U5 pad 7: Net-(J2-Pad8) -> Net-(J2-Pad15)
- U9 pad 7: Net-(J2-Pad16) -> Net-(J2-Pad31)
Routing:
- net Net-(J2-Pad33): track 5.43 -> 0.00 mm
- net Net-(J2-Pad31): track 5.43 -> 10.5 mm
- net Net-(J2-Pad8): track 2.68 -> 0.00 mm
- net Net-(J2-Pad15): track 0.00 -> 2.68 mm

Commit message: Rev 2 work in progress
Parts:
- removed D6: D, Diodes_SMD:D_SOD-123
- removed D7: ACGRKM4007-HF, Diodes_SMD:D_SOD-123F
- removed L2: 10uH, Inductors_SMD:L_0805
- removed Q4: Q_NMOS_DGS, Housings_SOIC:SOIC-8_3.9x4.9mm_Pitch1.27mm
- removed Q6, Q7: SQ2318AES-T1_GE3, TO_SOT_Packages_SMD:SOT-23
- added C46: 1uF, Capacitors_SMD:C_0805_HandSoldering, F.Cu at (153.7, 169.5)
- added D10: LED, LEDs:LED_0805_HandSoldering, F.Cu at (73.7, 184.8)
- added D11: B340A-13-F, Diodes_SMD:D_SMA_Handsoldering, F.Cu at (73.7, 169.5)
- added D12: LED, LEDs:LED_0805_HandSoldering, F.Cu at (83.8, 184.8)
- added D13: B340A-13-F, Diodes_SMD:D_SMA_Handsoldering, F.Cu at (83.8, 169.5)
- added D14: LED, LEDs:LED_0805_HandSoldering, F.Cu at (94.0, 184.8)
- added D15: B340A-13-F, Diodes_SMD:D_SMA_Handsoldering, F.Cu at (94.0, 169.5)
- added D16: LED, LEDs:LED_0805_HandSoldering, F.Cu at (121.9, 184.8)
- added D17: LED, LEDs:LED_0805_HandSoldering, F.Cu at (111.8, 184.8)
- added D18: LED, LEDs:LED_0805_HandSoldering, F.Cu at (101.6, 184.8)
- added D19: LED, LEDs:LED_0805_HandSoldering, F.Cu at (106.7, 184.8)
- added D9: B340A-13-F, Diodes_SMD:D_SMA_Handsoldering, F.Cu at (63.5, 169.5)
- added JP1: Jumper, Pin_Headers:Pin_Header_Straight_1x02_Pitch2.54mm, F.Cu at (66.0, 149.9)
- added JP10: Jumper, Pin_Headers:Pin_Header_Straight_1x02_Pitch2.54mm, F.Cu at (81.3, 152.4)
- added JP11: Jumper, Pin_Headers:Pin_Header_Straight_1x02_Pitch2.54mm, F.Cu at (91.4, 152.4)
- added JP12: Jumper, Pin_Headers:Pin_Header_Straight_1x02_Pitch2.54mm, F.Cu at (106.7, 157.5)
- added JP13: Jumper, Pin_Headers:Pin_Header_Straight_1x02_Pitch2.54mm, F.Cu at (123.2, 158.1)
- added JP14: Jumper, Pin_Headers:Pin_Header_Straight_1x02_Pitch2.54mm, F.Cu at (129.5, 160.7)
- added JP15: Jumper, Pin_Headers:Pin_Header_Straight_1x02_Pitch2.54mm, F.Cu at (135.9, 160.7)
- added JP16: Jumper, Pin_Headers:Pin_Header_Straight_1x02_Pitch2.54mm, F.Cu at (279.4, 161.3)
- added JP17: Jumper, Pin_Headers:Pin_Header_Straight_1x02_Pitch2.54mm, F.Cu at (193.0, 163.8)
- added JP18: Jumper, Pin_Headers:Pin_Header_Straight_1x02_Pitch2.54mm, F.Cu at (218.4, 163.8)
- added JP19: Jumper, Pin_Headers:Pin_Header_Straight_1x02_Pitch2.54mm, F.Cu at (208.3, 163.8)
- added JP2: Jumper, Pin_Headers:Pin_Header_Straight_1x02_Pitch2.54mm, F.Cu at (76.2, 149.9)
- added JP20: Jumper, Pin_Headers:Pin_Header_Straight_1x02_Pitch2.54mm, F.Cu at (137.8, 109.2)
- added JP21: Jumper, Pin_Headers:Pin_Header_Straight_1x02_Pitch2.54mm, F.Cu at (246.4, 163.8)
- added JP22: Jumper, Pin_Headers:Pin_Header_Straight_1x02_Pitch2.54mm, F.Cu at (177.8, 163.8)
- added JP23: Jumper, Pin_Headers:Pin_Header_Straight_1x02_Pitch2.54mm, F.Cu at (162.6, 163.8)
- added JP24: Jumper, Pin_Headers:Pin_Header_Straight_1x02_Pitch2.54mm, F.Cu at (250.8, 112.4)
- added JP25: Jumper, Pin_Headers:Pin_Header_Straight_1x02_Pitch2.54mm, F.Cu at (262.3, 112.4)
- added JP26: Jumper, Pin_Headers:Pin_Header_Straight_1x02_Pitch2.54mm, F.Cu at (264.8, 112.4)
- added JP27: Jumper, Pin_Headers:Pin_Header_Straight_1x02_Pitch2.54mm, F.Cu at (239.4, 112.4)
- added JP28: Jumper, Pin_Headers:Pin_Header_Straight_1x02_Pitch2.54mm, F.Cu at (234.3, 109.9)
- added JP29: Jumper, Pin_Headers:Pin_Header_Straight_1x02_Pitch2.54mm, F.Cu at (267.3, 109.9)
- added JP3: Jumper, Pin_Headers:Pin_Header_Straight_1x02_Pitch2.54mm, F.Cu at (86.4, 149.9)
- added JP30: Jumper, Pin_Headers:Pin_Header_Straight_1x02_Pitch2.54mm, F.Cu at (155.6, 128.9)
- added JP31: Jumper, Pin_Headers:Pin_Header_Straight_1x02_Pitch2.54mm, F.Cu at (106.7, 135.3)
- added JP32: Jumper, Pin_Headers:Pin_Header_Straight_1x02_Pitch2.54mm, F.Cu at (153.0, 135.3)
- added JP33: Jumper, Pin_Headers:Pin_Header_Straight_1x02_Pitch2.54mm, F.Cu at (241.3, 163.8)
- added JP34: Jumper, Pin_Headers:Pin_Header_Straight_1x02_Pitch2.54mm, F.Cu at (172.7, 163.8)
- added JP35: Jumper, Pin_Headers:Pin_Header_Straight_1x02_Pitch2.54mm, F.Cu at (157.5, 163.8)
- added JP36: Jumper, Pin_Headers:Pin_Header_Straight_1x02_Pitch2.54mm, F.Cu at (188.0, 163.8)
- added JP37: Jumper, Pin_Headers:Pin_Header_Straight_1x02_Pitch2.54mm, F.Cu at (213.4, 163.8)
- added JP38: Jumper, Pin_Headers:Pin_Header_Straight_1x02_Pitch2.54mm, F.Cu at (203.2, 163.8)
- added JP39: Jumper, Pin_Headers:Pin_Header_Straight_1x02_Pitch2.54mm, F.Cu at (226.1, 161.3)
- added JP4: Jumper, Pin_Headers:Pin_Header_Straight_1x02_Pitch2.54mm, F.Cu at (96.5, 149.9)
- added JP40: Jumper, Pin_Headers:Pin_Header_Straight_1x02_Pitch2.54mm, F.Cu at (231.1, 161.3)
- added JP41: Jumper, Pin_Headers:Pin_Header_Straight_1x02_Pitch2.54mm, F.Cu at (150.5, 158.1)
- added JP42: Jumper, Pin_Headers:Pin_Header_Straight_1x02_Pitch2.54mm, F.Cu at (148.0, 158.1)
- added JP43: Jumper, Pin_Headers:Pin_Header_Straight_1x02_Pitch2.54mm, F.Cu at (153.0, 160.7)
- added JP44: Jumper, Pin_Headers:Pin_Header_Straight_1x02_Pitch2.54mm, F.Cu at (142.9, 160.7)
- added JP45: Jumper, Pin_Headers:Pin_Header_Straight_1x02_Pitch2.54mm, F.Cu at (256.5, 158.8)
- added JP5: Jumper, Pin_Headers:Pin_Header_Straight_1x02_Pitch2.54mm, F.Cu at (111.8, 154.9)
- added JP6: Jumper, Pin_Headers:Pin_Header_Straight_1x02_Pitch2.54mm, F.Cu at (101.6, 154.9)
- added JP7: Jumper, Pin_Headers:Pin_Header_Straight_1x02_Pitch2.54mm, F.Cu at (116.8, 154.9)
- added JP8: Jumper, Pin_Headers:Pin_Header_Straight_1x02_Pitch2.54mm, F.Cu at (61.0, 152.4)
- added JP9: Jumper, Pin_Headers:Pin_Header_Straight_1x02_Pitch2.54mm, F.Cu at (71.1, 152.4)
- added R21: 10k, Resistors_SMD:R_0805_HandSoldering, F.Cu at (77.5, 165.1)
- added R22: R_US, Resistors_SMD:R_0805_HandSoldering, F.Cu at (71.1, 156.8)
- added R39: 10k, Resistors_SMD:R_0805_HandSoldering, F.Cu at (97.8, 165.1)
- added R42: R_US, Resistors_SMD:R_0805_HandSoldering, F.Cu at (97.8, 160.0)
- added R43: R_US, Resistors_SMD:R_0805_HandSoldering, F.Cu at (123.2, 170.2)
- added R44: R_US, Resistors_SMD:R_0805_HandSoldering, F.Cu at (111.8, 170.2)
- added R45: R_US, Resistors_SMD:R_0805_HandSoldering, F.Cu at (101.6, 170.2)
- added R46: 150, Resistors_SMD:R_0805_HandSoldering, F.Cu at (112.4, 161.3)
- added R47: 10k, Resistors_SMD:R_0805_HandSoldering, F.Cu at (112.4, 163.8)
- added R48: 10k, Resistors_SMD:R_0805_HandSoldering, F.Cu at (106.7, 162.6)
- added R49: R_US, Resistors_SMD:R_0805_HandSoldering, F.Cu at (106.7, 170.2)
- added R50: R_US, Resistors_SMD:R_0805_HandSoldering, F.Cu at (132.1, 140.3)
- added R51: R_US, Resistors_SMD:R_0805_HandSoldering, F.Cu at (228.0, 111.1)
- added U13: DRV103H, Housings_SOIC:TI_SO-PowerPAD-8, F.Cu at (73.7, 162.6)
- added U14: DRV103H, Housings_SOIC:TI_SO-PowerPAD-8, F.Cu at (83.8, 162.6)
- added U15: DRV103H, Housings_SOIC:TI_SO-PowerPAD-8, F.Cu at (94.1, 162.6)
- C1, C10, C11, C12, C13, C14, C15, C16, C17, C18, C19, C2, C20, C21, C22, C23, C3, C32, C33, C34, C35, C36, C37, C38, C39, C4, C40, C41, C42, C44, C45, C5, C7, C8, C9: footprint Capacitors_SMD:C_0805 -> Capacitors_SMD:C_0805_HandSoldering
- C24, C25, C28, C29, C30, C31: value 22uF -> C; footprint Capacitors_SMD:C_0805 -> Capacitors_SMD:C_0805_HandSoldering
- C26, C27: value 1u -> C; footprint Capacitors_SMD:C_0805 -> Capacitors_SMD:C_0805_HandSoldering
- C43: value 220pF -> 100nF; footprint Capacitors_SMD:C_0805 -> Capacitors_SMD:C_0805_HandSoldering
- C6: value 100nF -> 220pF; footprint Capacitors_SMD:C_0805 -> Capacitors_SMD:C_0805_HandSoldering
- D2, D3: value ACGRKM4007-HF -> LED; footprint Diodes_SMD:D_SOD-123F -> LEDs:LED_0805_HandSoldering
- D5: value D_Zener -> LED; footprint Diodes_SMD:D_SOD-323 -> LEDs:LED_0805_HandSoldering
- D8: value PMEG060V100EPDZ -> LED; footprint TO_SOT_Packages_SMD:TO-277A -> LEDs:LED_0805_HandSoldering
- J10: value Injector 4 -> Injector
- J2, U4: moved to F.Cu
- J7: value Injector 1 -> Injector
- J8: value Injector 2 -> Injector
- J9: value Injector 3 -> Injector
- L1: value 22uH -> 10uH; footprint Speeduino Mini:SRP1265A -> Inductors_SMD:L_0805_HandSoldering
- PC2: footprint Capacitors_SMD:C_1206 -> Capacitors_SMD:C_1206_HandSoldering
- Q1: value SQ2318AES-T1_GE3 -> 2N7002
- Q2: value SQ2318AES-T1_GE3 -> SQ3457EV; footprint TO_SOT_Packages_SMD:SOT-23 -> Housings_SSOP:TSOP-6_1.65x3.05mm_Pitch0.95mm
- R1, R10, R11, R12, R13, R14, R15, R16, R17, R2, R23, R24, R25, R26, R27, R29, R3, R32, R35, R4, R5, R6, R7, R8, R9, RN5A1: footprint Resistors_SMD:R_0805 -> Resistors_SMD:R_0805_HandSoldering
- R18, R20, R34, R36, R37: value 150 -> R_US; footprint Resistors_SMD:R_0805 -> Resistors_SMD:R_0805_HandSoldering
- R19, R33, R38: value 10k -> R_US; footprint Resistors_SMD:R_0805 -> Resistors_SMD:R_0805_HandSoldering
- R28: value 4k7 -> 33k; footprint Resistors_SMD:R_0805 -> Resistors_SMD:R_0805_HandSoldering
- R30: value 47 -> 4k7; footprint Resistors_SMD:R_0805 -> Resistors_SMD:R_0805_HandSoldering
- R31: value 33k -> R_US; footprint Resistors_SMD:R_0805 -> Resistors_SMD:R_0805_HandSoldering
- R40: value 78.7k -> R_US; footprint Resistors_SMD:R_0805 -> Resistors_SMD:R_0805_HandSoldering
- R41: value 20k -> R_US; footprint Resistors_SMD:R_0805 -> Resistors_SMD:R_0805_HandSoldering
- U10, U5, U9: value SN74LVC2T45-VSSOP -> SN74LVC2T45MDCTTEP; footprint Housings_SSOP:VSSOP-8_2.3x2mm_Pitch0.5mm -> Housings_SSOP:SSOP-8_2.95x2.8mm_Pitch0.65mm
- U12: value MCP2003B -> LD1117S50TR_SOT223; footprint Housings_SOIC:SOIC-8_3.9x4.9mm_Pitch1.27mm -> TO_SOT_Packages_SMD:SOT-223-3_TabPin2
- U7: value RT7258 -> DRV103H; footprint Speeduino Mini:SOP-8 -> Housings_SOIC:TI_SO-PowerPAD-8
- U8: value LD1117S50TR_SOT223 -> MCP2003B; footprint TO_SOT_Packages_SMD:SOT-223-3_TabPin2 -> Housings_SOIC:SOIC-8_3.9x4.9mm_Pitch1.27mm
- moved U4 180.9 mm to (268.0, 174.0)
- moved C11 173.7 mm to (279.4, 165.1), turned to 270 degrees
- moved J4 173.1 mm to (215.9, 177.8), turned to 0 degrees
- moved R7 169.3 mm to (276.9, 165.1), turned to 270 degrees
- moved C14 164.8 mm to (218.4, 170.2), turned to 0 degrees
- moved C15 164.7 mm to (218.4, 167.6), turned to 0 degrees
- moved J5 160.8 mm to (205.7, 177.8), turned to 0 degrees
- moved C10 160.5 mm to (259.1, 165.1)
- moved R3 159.9 mm to (215.3, 168.9), turned to 270 degrees
- moved R2 156.5 mm to (212.7, 168.9), turned to 270 degrees
- moved C9 156.2 mm to (256.5, 165.1)
- moved C17 151.3 mm to (208.3, 170.2), turned to 0 degrees
- moved C18 151.0 mm to (208.3, 167.6), turned to 0 degrees
- moved J3 148.0 mm to (193.0, 177.8), turned to 0 degrees
- moved R5 146.8 mm to (205.1, 168.9), turned to 270 degrees
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Connections:
- C1 pad 1: +5VD -> /MCU/VCC
- C10 pad 1: +5VA -> /MAP Sensor/+5V
- C11 pad 1: /MCU/A4 -> /MAP Sensor/OUT
- C13 pad 1: /MCU/A5 -> /Throttle Position Sensor /OUT
- C15 pad 1: /MCU/A2 -> /Intake Air Temperature Sensor/OUT
- C16 pad 1: +5VD -> +12V
- C18 pad 1: /MCU/A3 -> /Head Temperature Sensor/OUT
- C2 pad 1: /Raspberry Pi Zero W/ATMEGA_RESET -> /MCU/RESET
- C20 pad 1: /MCU/A0 -> /Battery Reference Voltage/OUT
- C22 pad 1: +5VD -> /MCU/VCC
- C25 pad 1: Net-(C24-Pad1) -> /Injector 1/+12V
- C27 pad 1: Net-(C27-Pad1) -> /Injector 2/+12V
- C27 pad 2: Net-(C27-Pad2) -> GND
- C28 pad 1: /Injector Power Supply/VOUT -> Net-(C28-Pad1)
- C29 pad 1: /Injector Power Supply/VOUT -> /Injector 3/+12V
- C3 pad 1: +5VD -> /MCU/VCC
- C30 pad 1: /Injector Power Supply/VOUT -> Net-(C30-Pad1)
- C31 pad 1: /Injector Power Supply/VOUT -> /Injector 4/+12V
- C32 pad 1: /MCU/A6 -> /Oil Pressure Sensor/OUT
- C34 pad 1: /MCU/A7 -> /Fuel Pressure/OUT
- C35 pad 1: Net-(C35-Pad1) -> /MCU/VCC
- C36 pad 1: Net-(C36-Pad1) -> /MCU/VCC
- C37 pad 1: Net-(C37-Pad1) -> /Power/+12V
- C42 pad 1: /MCU/INT1 -> /Crankshaft pos sensor/OUT
- C43 pad 1: /Lin transceiver/LIN -> /MCU/ATMEGA regulator/AVCC
- C5 pad 1: +5VD -> /MCU/VCC
- C6 pad 1: +5VD -> /MCU/LIN
- C8 pad 1: /MCU/A1 -> /O2 Sensor/OUT
- C9 pad 1: +5VA -> /MAP Sensor/+5V
- D1 pad 1: +5VD -> /MCU/VCC
- D1 pad 2: /Raspberry Pi Zero W/ATMEGA_RESET -> /MCU/RESET
- D2 pad 1: Net-(C35-Pad1) -> GND
- D2 pad 2: +12V -> Net-(D2-Pad2)
- D3 pad 1: Net-(C37-Pad1) -> GND
- D3 pad 2: +12V -> Net-(D3-Pad2)
- D5 pad 1: Net-(D5-Pad1) -> GND
- D5 pad 2: GND -> Net-(D5-Pad2)
- D8 pad 1: +12V -> Net-(D8-Pad1)
- D8 pad 2: +12V -> Net-(D8-Pad2)
- J10 pad 1: /Injector Power Supply/VOUT -> /Injector 4/+12V
- J10 pad 2: /Injector 4/INJ_OUT -> Net-(D15-Pad2)
- J11 pad 1: /MCU/OC0B -> /Ignitor/IN1
- J11 pad 2: +12V -> /Ignitor/sheet5CF8D1B3/OUT
- J11 pad 3: /MCU/OC3A -> /Ignitor/IN2
- J12 pad 1: +5VA -> Net-(J12-Pad1)
- J13 pad 1: +5VA -> Net-(J13-Pad1)
- J14 pad 2: /Lin transceiver/LIN -> /MCU/LIN
- J15 pad 1: +5VA -> Net-(J15-Pad1)
- J15 pad 2: /Camshaft position sensor/OUT -> /Camshaft position sensor/IN
- J2 pad 11: GND -> (no net)
- J2 pad 15: Net-(J2-Pad15) -> (no net)
- J2 pad 18: Net-(J2-Pad18) -> (no net)
- J2 pad 19: Net-(J2-Pad10) -> (no net)
- J2 pad 2: +5VA -> /Raspberry Pi Zero W/+5VA
- J2 pad 27: GND -> (no net)
- J2 pad 31: Net-(J2-Pad31) -> (no net)
- J2 pad 32: (no net) -> Net-(J2-Pad32)
- J2 pad 33: Net-(J2-Pad1) -> Net-(J2-Pad33)
- J2 pad 4: +5VA -> /Raspberry Pi Zero W/+5VA
- J2 pad 7: (no net) -> Net-(J2-Pad7)
- J2 pad 8: Net-(J2-Pad15) -> Net-(J2-Pad8)
- J3 pad 1: +5VA -> Net-(J3-Pad1)
- J6 pad 1: +5VA -> Net-(J6-Pad1)
- J7 pad 1: /Injector Power Supply/VOUT -> /Injector 1/+12V
- J7 pad 2: /Injector 1/INJ_OUT -> Net-(D9-Pad2)
- J8 pad 1: /Injector Power Supply/VOUT -> /Injector 2/+12V
- J8 pad 2: /Injector 2/INJ_OUT -> Net-(D11-Pad2)
- J9 pad 1: /Injector Power Supply/VOUT -> /Injector 3/+12V
- J9 pad 2: /Injector 3/INJ_OUT -> Net-(D13-Pad2)
- L1 pad 1: Net-(C27-Pad2) -> /MCU/VCC
- L1 pad 2: /Injector Power Supply/VOUT -> /MCU/ATMEGA regulator/AVCC
- L3 pad 1: Net-(C37-Pad1) -> /Power/+12V
- L4 pad 2: +5VA -> /Power/+5V
- PC1 pad 1: Net-(C35-Pad1) -> +12V
- PC2 pad 1: +5VD -> /MCU/VCC
- PC3 pad 1: +5VA -> /Power/+5V
- PC4 pad 1: +5VA -> /Power/+5V
- Q1 pad 3: /Injector 1/INJ_OUT -> Net-(Q1-Pad3)
- Q2 pad 1: Net-(Q2-Pad1) -> /Ignitor/sheet5CF8D1B3/OUT
- Q2 pad 2: GND -> /Ignitor/sheet5CF8D1B3/OUT
- Q2 pad 3: /Injector 2/INJ_OUT -> Net-(Q1-Pad3)
- Q5 pad 4: +12V -> /O2 Sensor Power/+12V
- R10 pad 1: /MCU/A7 -> /Fuel Pressure/OUT
- R15 pad 1: /MCU/A0 -> /Battery Reference Voltage/OUT
- R18 pad 1: Net-(Q1-Pad1) -> Net-(R18-Pad1)
- R18 pad 2: /Injector 1/INJ_CMD -> GND
- R19 pad 1: /Injector 2/INJ_CMD -> /Injector 1/+12V
- R19 pad 2: GND -> Net-(D8-Pad2)
- R2 pad 1: +5VA -> /Intake Air Temperature Sensor/VCC
- R20 pad 1: Net-(Q2-Pad1) -> Net-(R20-Pad1)
- R20 pad 2: /Injector 2/INJ_CMD -> GND
- R24 pad 1: Net-(J2-Pad31) -> Net-(J2-Pad16)
- R26 pad 1: /MCU/INT1 -> /Crankshaft pos sensor/OUT
- R27 pad 2: +12V -> /MCU/sheet5D16F277/+12V
- R28 pad 1: +5VD -> Net-(R28-Pad1)
- R28 pad 2: /Lin transceiver/RXD -> /MCU/sheet5D16F277/+5V
- R29 pad 1: +12V -> /O2 Sensor Power/+12V
- R3 pad 1: /MCU/A2 -> /Intake Air Temperature Sensor/OUT
- R30 pad 1: Net-(D6-Pad1) -> /MCU/sheet5D16F277/+5V
- R30 pad 2: Net-(D5-Pad1) -> /MCU/sheet5D16F277/RXD
- R31 pad 1: Net-(R31-Pad1) -> Net-(D2-Pad2)
- R31 pad 2: +5VD -> Net-(J2-Pad33)
- R33 pad 1: /Injector 3/INJ_CMD -> /Injector 2/+12V
- R33 pad 2: GND -> Net-(D10-Pad2)
- R34 pad 2: /Injector 3/INJ_CMD -> GND
- R35 pad 1: /Injector 4/INJ_CMD -> /Injector 3/INJ_CMD
- R36 pad 2: /Injector 4/INJ_CMD -> GND
- R37 pad 1: Net-(R37-Pad1) -> /Injector 3/+12V
- R37 pad 2: /Injector Power Supply/EN -> Net-(D12-Pad2)
- R38 pad 1: GND -> Net-(R38-Pad1)
- R38 pad 2: Net-(R37-Pad1) -> GND
- R4 pad 1: +5VA -> /Head Temperature Sensor/VCC
- R40 pad 1: /Injector Power Supply/VOUT -> Net-(R40-Pad1)
- R40 pad 2: Net-(R40-Pad2) -> GND
- R41 pad 1: Net-(R40-Pad2) -> /Injector 4/+12V
- R41 pad 2: GND -> Net-(D14-Pad2)
- R5 pad 1: /MCU/A3 -> /Head Temperature Sensor/OUT
- R6 pad 1: /MCU/A1 -> /O2 Sensor/OUT
- R7 pad 1: /MCU/A4 -> /MAP Sensor/OUT
- R8 pad 1: /MCU/A5 -> /Throttle Position Sensor /OUT
- R9 pad 1: /MCU/A6 -> /Oil Pressure Sensor/OUT
- RN5A1 pad 1: +5VD -> /MCU/VCC
- RN5A1 pad 2: /Raspberry Pi Zero W/ATMEGA_RESET -> /MCU/RESET
- U1 pad 5: +5VD -> /MCU/VCC
- U10 pad 2: Net-(J2-Pad18) -> (no net)
- U10 pad 7: +5VD -> /Raspberry Pi Zero W/+5VD
- U10 pad 8: +5VD -> /Raspberry Pi Zero W/+5VD
- U11 pad 4: +5VA -> /Power/+5V
- U12 pad 1: /Lin transceiver/RXD -> GND
- U12 pad 2: Net-(R31-Pad1) -> /MCU/VCC
- U12 pad 3: Net-(R27-Pad1) -> +12V
- U2 pad 5: +5VD -> /MCU/VCC
- U3 pad 1: /MCU/OC0B -> (no net)
- U3 pad 15: /Injector 3/INJ_CMD -> /MCU/OC1A
- U3 pad 16: /Injector 4/INJ_CMD -> /MCU/OC1B
- U3 pad 17: /Power/EN -> /MCU/PB7
- U3 pad 20: /Raspberry Pi Zero W/ATMEGA_RESET -> /MCU/RESET
- U3 pad 21: +5VD -> /MCU/VCC
- U3 pad 25: /Camshaft position sensor/IN -> /MCU/INT0
- U3 pad 27: /Lin transceiver/RXD -> Net-(JP41-Pad1)
- U3 pad 28: /Lin transceiver/TXD -> Net-(JP42-Pad1)
- U3 pad 3: /Raspberry Pi Zero W/RXD_PDO -> /MCU/TXD0
- U3 pad 51: /O2 Sensor Power/EN -> /MCU/PA0
- U3 pad 52: +5VD -> /MCU/VCC
- U3 pad 6: /Injector 1/INJ_CMD -> /MCU/OC3B
- U3 pad 64: Net-(C36-Pad1) -> /MCU/ATMEGA regulator/AVCC
- U3 pad 7: /Injector 2/INJ_CMD -> /MCU/OC3C
- U3 pad 9: /Injector Power Supply/EN -> (no net)
- U4 pad 3: +5VA -> /MAP Sensor/+5V
- U5 pad 1: +5VD -> /Raspberry Pi Zero W/+5VD
- U5 pad 2: /MCU/RXD0 -> /Raspberry Pi Zero W/TXD_PDI
- U5 pad 3: /MCU/SCK -> /Raspberry Pi Zero W/SCK
- U5 pad 6: Net-(J2-Pad16) -> Net-(J2-Pad7)
- U5 pad 7: Net-(J2-Pad15) -> Net-(J2-Pad8)
- U6 pad 3: /Camshaft position sensor/IN -> /MCU/INT0
- U6 pad 5: +5VD -> /MCU/VCC
- U7 pad 1: Net-(C27-Pad2) -> Net-(R20-Pad1)
- U7 pad 2: Net-(C27-Pad1) -> Net-(C24-Pad1)
- U7 pad 3: Net-(C26-Pad1) -> Net-(R18-Pad1)
- U7 pad 4: Net-(Q4-Pad4) -> GND
- U7 pad 5: GND -> Net-(D9-Pad2)
- U7 pad 6: Net-(R40-Pad2) -> /Injector 1/+12V
- U7 pad 7: Net-(R37-Pad1) -> Net-(D8-Pad1)
- U7 pad 8: Net-(C24-Pad1) -> /Injector 1/INJ_CMD
- U8 pad 1: GND -> /MCU/sheet5D16F277/RXD
- U8 pad 2: +5VD -> Net-(R28-Pad1)
- U8 pad 3: Net-(C35-Pad1) -> Net-(R27-Pad1)
- U9 pad 1: +5VD -> /Raspberry Pi Zero W/+5VD
- U9 pad 7: Net-(J2-Pad31) -> Net-(J2-Pad16)
Routing:
- net +5VA: track 356.7 -> 0.00 mm, vias 11 -> 0
- net +5VD: track 186.1 -> 0.00 mm, vias 10 -> 0
- net +12V: track 123.8 -> 20.5 mm
- net /Injector Power Supply/VOUT: track 95.7 -> 0.00 mm, vias 4 -> 0
- net /O2 Sensor Power/EN: track 87.5 -> 3.73 mm, vias 2 -> 0
- net /Raspberry Pi Zero W/ATMEGA_RESET: track 76.4 -> 2.57 mm, vias 2 -> 0
- net /MCU/A7: track 70.5 -> 2.81 mm, vias 2 -> 0
- net /MCU/A5: track 58.8 -> 5.45 mm
- net /MCU/A2: track 58.4 -> 5.75 mm
- net /MCU/A6: track 58.1 -> 5.49 mm
- net /MCU/A3: track 54.8 -> 3.14 mm
- net /MCU/INT1: track 55.5 -> 3.88 mm, vias 2 -> 0
- net /Lin transceiver/TXD: track 50.3 -> 0.00 mm, vias 2 -> 0
- net /MCU/A1: track 54.8 -> 5.45 mm
- net /Power/EN: track 51.8 -> 2.61 mm, vias 2 -> 0
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Other:
- board text added: "+"
- board text added: "-"
- board text added: "0V"
- board text added: "1"
- board text added: "12V"
- board text added: "2"
- board text added: "3"
- board text added: "4"
- board text added: "5V"
- board text added: "A"
- board text added: "B"
- board text added: "CAMSHAFT POS"
- board text added: "CRANKSHAFT POS"
- board text added: "FUEL PRESSURE"
- board text added: "HEAD TEMP"
- board text added: "IAT"
- board text added: "IGNITOR"
- board text added: "IN"
- board text added: "INJECTORS"
- board text added: "LIN"
- board text added: "O2 SENSOR"
- board text added: "OIL PRESSURE"
- board text added: "TPS"
