File: hardware/speeduino_mini.kicad_pcb (KiCad board)
At the start: 2 copper layers, 100 x 100 mm, 202 parts, among them J1 O2, J10 Injector, J11 Ignitor Pack, J12 oil pressure, J13 fuel pressure, J14 power, J15 camshaft position sensor, J2 Raspberry_Pi_2_3, J3 TPS, J4 IAT, J5 head temperature, J6 crankshaft position sensor, J7 Injector, J8 Injector, J9 Injector, Q1 2N7002, Q2 SQ3457EV, Q3 2N7002, Q5 SQ3457EV, U1 TPD4E001-Q1, U10 SN74LVC2T45MDCTTEP, U11 TLE8366, U12 LD1117S50TR_SOT223, U13 DRV103H, U14 DRV103H, U15 DRV103H, U2 TPD4E001-Q1, U3 ATmega2561-16AU, U4 MPX4250AP1, U5 SN74LVC2T45MDCTTEP, U6 TPD4E001-Q1, U7 DRV103H, U8 MCP2003B, U9 SN74LVC2T45MDCTTEP, Y1 CSTCE16M0V53-R0

Commit message: rev 2 work in progress
Parts:
- removed C44: 0.1uF, Capacitors_SMD:C_0805_HandSoldering
- removed C45: 0.22u, Capacitors_SMD:C_0805_HandSoldering
- removed J15: camshaft position sensor, Speeduino Mini:ED120_3DS
- removed JP39, JP40: Jumper, Pin_Headers:Pin_Header_Straight_1x02_Pitch2.54mm
- removed R32: 470, Resistors_SMD:R_0805_HandSoldering
- added H1: MountingHole, Mounting_Holes:MountingHole_4.3mm_M4_Pad_Via, F.Cu at (30.5, 73.7)
- added H2: MountingHole, Mounting_Holes:MountingHole_4.3mm_M4_Pad_Via, F.Cu at (30.5, 129.5)
- added H3: MountingHole, Mounting_Holes:MountingHole_4.3mm_M4_Pad_Via, F.Cu at (259.1, 73.7)
- added H4: MountingHole, Mounting_Holes:MountingHole_4.3mm_M4_Pad_Via, F.Cu at (259.1, 129.5)
- added JP46: Jumper, Pin_Headers:Pin_Header_Straight_1x02_Pitch2.54mm, F.Cu at (112.0, 98.6)
- added JP47: Jumper, Pin_Headers:Pin_Header_Straight_1x02_Pitch2.54mm, F.Cu at (81.5, 101.1)
- added JP48: Jumper, Pin_Headers:Pin_Header_Straight_1x02_Pitch2.54mm, F.Cu at (134.0, 94.6)
- added QR*****: QR_CODE, Speeduino Mini:QR_CODE, F.Cu at (58.4, 83.8)
- moved D1 159.0 mm to (82.5, 78.1), turned to 270 degrees
- moved RN5A1 154.5 mm to (85.1, 78.1), turned to 270 degrees
- moved C2 150.1 mm to (87.6, 78.1), turned to 90 degrees
- moved R1 150.0 mm to (85.1, 83.2), turned to 90 degrees
- moved C5 148.5 mm to (83.8, 88.3), turned to 90 degrees
- moved Y1 145.4 mm to (87.6, 83.2), turned to 90 degrees
- moved U6 142.6 mm to (87.0, 88.3), turned to 270 degrees
- moved U3 125.6 mm to (98.4, 83.8), turned to 270 degrees
- moved C4 120.8 mm to (109.9, 72.4), turned to 0 degrees
- moved L1 117.3 mm to (109.9, 74.9), turned to 180 degrees
- moved C43 114.0 mm to (109.9, 77.5), turned to 0 degrees
- moved U4 111.3 mm to (196.2, 88.9), turned to 90 degrees
- moved U1 110.2 mm to (109.7, 80.6), turned to 270 degrees
- moved U2 105.0 mm to (109.7, 85.1), turned to 90 degrees
- moved C1 104.7 mm to (113.3, 80.6), turned to 90 degrees
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Connections:
- C1 pad 1: /MCU/VCC -> +5VD
- C16 pad 1: +12V -> Net-(C16-Pad1)
- C22 pad 1: /MCU/VCC -> Net-(C22-Pad1)
- C3 pad 1: /MCU/VCC -> +5VD
- C35 pad 1: /MCU/VCC -> Net-(C22-Pad1)
- C36 pad 1: /MCU/VCC -> Net-(C22-Pad1)
- C5 pad 1: /MCU/VCC -> +5VD
- D1 pad 1: /MCU/VCC -> +5VD
- JP1 pad 1: /MCU/OC1A -> /MCU/OC1B
- JP15 pad 2: /MCU/A1 -> /MCU/A7
- JP2 pad 1: /MCU/OC1A -> /MCU/OC1B
- JP23 pad 2: /MCU/A7 -> /MCU/A1
- JP28 pad 2: (no net) -> +5VD
- JP3 pad 1: /MCU/OC1B -> /MCU/OC1A
- JP4 pad 1: /MCU/OC1B -> /MCU/OC1A
- JP43 pad 2: /MCU/VCC -> +5VD
- JP5 pad 1: /MCU/OC3C -> /MCU/OC3B
- JP6 pad 1: /MCU/OC3A -> /MCU/OC3C
- JP7 pad 1: /MCU/OC3B -> /MCU/OC3A
- L1 pad 1: /MCU/VCC -> +5VD
- PC1 pad 1: +12V -> Net-(C16-Pad1)
- PC2 pad 1: /MCU/VCC -> Net-(C22-Pad1)
- R13 pad 1: +12V -> /Battery Reference Voltage/+12V
- RN5A1 pad 1: /MCU/VCC -> +5VD
- U1 pad 5: /MCU/VCC -> +5VD
- U12 pad 2: /MCU/VCC -> Net-(C22-Pad1)
- U12 pad 3: +12V -> Net-(C16-Pad1)
- U2 pad 5: /MCU/VCC -> +5VD
- U3 pad 21: /MCU/VCC -> +5VD
- U3 pad 52: /MCU/VCC -> +5VD
- U6 pad 5: /MCU/VCC -> +5VD
Routing:
- net +5VD: track 0.00 -> 204.9 mm, vias 0 -> 2
- net /MCU/SCK: track 0.00 -> 176.9 mm, vias 0 -> 1
- net /MCU/RXD0: track 0.00 -> 165.0 mm, vias 0 -> 2
- net /MCU/RESET: track 8.64 -> 170.9 mm, vias 0 -> 2
- net /MCU/TXD0: track 0.00 -> 155.0 mm, vias 0 -> 2
- net +5VA: track 0.00 -> 142.6 mm
- net +12V: track 20.5 -> 142.1 mm
- net /MCU/A2: track 5.75 -> 112.3 mm, vias 0 -> 1
- net /MCU/A4: track 2.89 -> 105.9 mm, vias 0 -> 1
- net /MCU/A3: track 3.14 -> 103.7 mm, vias 0 -> 1
- net /MCU/INT1: track 3.88 -> 100.5 mm, vias 0 -> 1
- net /MCU/A5: track 5.45 -> 87.9 mm, vias 0 -> 1
- net /MCU/A6: track 5.49 -> 79.4 mm, vias 0 -> 1
- net /MCU/OC1B: track 0.00 -> 61.3 mm, vias 0 -> 1
- net /MCU/A1: track 5.45 -> 56.9 mm, vias 0 -> 2
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Other:
- board size 100 x 100 mm -> 238.8 x 66 mm
- board text added: "Powered By"
- board text added: "VW Bus ECU rev 2 Based on Speeduino 2019 Cedric Priscal"
- board text removed: "CAMSHAFT POS"
- board text removed: "DigiKey 377-2312-ND https://www.budind.com/pdf/hbext9166.pdf"
- board text removed: "VW Bus ECU rev 1 Based on Speeduino 2019 Cedric Priscal"

Commit message: hardware rev2 - layout complete
Parts:
- removed C3, C5: 100nF, Capacitors_SMD:C_0805_HandSoldering
- removed JP33, JP34, JP35, JP36, JP37, JP38, JP44, JP48: Jumper, Pin_Headers:Pin_Header_Straight_1x02_Pitch2.54mm
- removed QR*****: QR_CODE, Speeduino Mini:QR_CODE
- removed U1, U2, U6: TPD4E001-Q1, TO_SOT_Packages_SMD:SOT-23-6
- added D20: NUP1301,215, TO_SOT_Packages_SMD:SOT-23, F.Cu at (123.2, 81.3)
- added D21: NUP1301,215, TO_SOT_Packages_SMD:SOT-23, F.Cu at (127.0, 83.8)
- added D22: NUP1301,215, TO_SOT_Packages_SMD:SOT-23, F.Cu at (123.2, 86.4)
- added D23: NUP1301,215, TO_SOT_Packages_SMD:SOT-23, F.Cu at (127.0, 88.9)
- added D24: NUP1301,215, TO_SOT_Packages_SMD:SOT-23, F.Cu at (123.2, 91.4)
- added D25: NUP1301,215, TO_SOT_Packages_SMD:SOT-23, F.Cu at (127.0, 94.0)
- added D26: NUP1301,215, TO_SOT_Packages_SMD:SOT-23, F.Cu at (123.2, 96.5)
- added D6: NUP1301,215, TO_SOT_Packages_SMD:SOT-23, F.Cu at (123.2, 76.2)
- added D7: NUP1301,215, TO_SOT_Packages_SMD:SOT-23, F.Cu at (127.0, 78.7)
- added JP39: Jumper, Pin_Headers:Pin_Header_Straight_1x02_Pitch2.54mm, F.Cu at (119.4, 83.8)
- added JP40: Jumper, Pin_Headers:Pin_Header_Straight_1x02_Pitch2.54mm, F.Cu at (119.4, 86.4)
- added JP49: Jumper, Pin_Headers:Pin_Header_Straight_1x02_Pitch2.54mm, F.Cu at (119.4, 81.3)
- added JP50: Jumper, Pin_Headers:Pin_Header_Straight_1x02_Pitch2.54mm, F.Cu at (119.4, 88.9)
- added JP51: Jumper, Pin_Headers:Pin_Header_Straight_1x02_Pitch2.54mm, F.Cu at (119.4, 78.7)
- added JP52: Jumper, Pin_Headers:Pin_Header_Straight_1x02_Pitch2.54mm, F.Cu at (119.4, 91.4)
- added JP53: Jumper, Pin_Headers:Pin_Header_Straight_1x02_Pitch2.54mm, F.Cu at (119.4, 76.2)
- added JP54: Jumper, Pin_Headers:Pin_Header_Straight_1x02_Pitch2.54mm, F.Cu at (119.4, 94.0)
- added JP55: Jumper, Pin_Headers:Pin_Header_Straight_1x02_Pitch2.54mm, F.Cu at (119.4, 96.5)
- C1: value 100nF -> 0.47n
- moved C15 87.7 mm to (130.8, 78.7)
- moved R3 80.7 mm to (135.9, 78.7), turned to 0 degrees
- moved C14 79.5 mm to (141.0, 78.7), turned to 180 degrees
- moved C11 78.1 mm to (130.8, 76.2), turned to 0 degrees
- moved C18 77.4 mm to (130.8, 81.3)
- moved JP46 72.8 mm to (40.6, 83.8), turned to 90 degrees
- moved R7 72.5 mm to (135.9, 76.2), turned to 0 degrees
- moved R5 70.4 mm to (135.9, 81.3), turned to 0 degrees
- moved C17 69.3 mm to (141.0, 81.3), turned to 180 degrees
- moved J6 66.0 mm to (120.7, 121.9)
- moved JP18 64.5 mm to (148.6, 91.4), turned to 270 degrees
- moved JP16 64.1 mm to (148.6, 78.7), turned to 270 degrees
- moved C42 63.5 mm to (130.8, 96.5)
- moved PC1 63.2 mm to (47.0, 83.8), turned to 270 degrees
- moved JP19 57.7 mm to (148.6, 83.8), turned to 270 degrees
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Connections:
- C1 pad 1: +5VD -> Net-(C1-Pad1)
- C11 pad 1: /MAP Sensor/OUT -> /MCU/A0
- C12 pad 1: /Throttle Position Sensor /IN -> Net-(C12-Pad1)
- C13 pad 1: /Throttle Position Sensor /OUT -> /MCU/A3
- C14 pad 1: /Intake Air Temperature Sensor/IN -> Net-(C14-Pad1)
- C15 pad 1: /Intake Air Temperature Sensor/OUT -> /MCU/A1
- C17 pad 1: /Head Temperature Sensor/IN -> Net-(C17-Pad1)
- C18 pad 1: /Head Temperature Sensor/OUT -> /MCU/A2
- C20 pad 1: /Battery Reference Voltage/OUT -> /MCU/A7
- C21 pad 1: /Crankshaft pos sensor/IN -> Net-(C21-Pad1)
- C23 pad 1: /Oil Pressure Sensor/IN -> Net-(C23-Pad1)
- C32 pad 1: /Oil Pressure Sensor/OUT -> /MCU/A4
- C33 pad 1: /Fuel Pressure/IN -> Net-(C33-Pad1)
- C34 pad 1: /Fuel Pressure/OUT -> /MCU/A5
- C42 pad 1: /Crankshaft pos sensor/OUT -> /MCU/INT0
- C46 pad 1: /MCU/sheet5D16F277/+12V -> +12V
- C7 pad 1: /O2 Sensor/IN -> Net-(C7-Pad1)
- C8 pad 1: /O2 Sensor/OUT -> /MCU/A6
- J12 pad 1: Net-(J12-Pad1) -> +5VA
- J13 pad 1: Net-(J13-Pad1) -> +5VA
- J2 pad 25: GND -> (no net)
- J2 pad 39: GND -> (no net)
- J2 pad 9: GND -> (no net)
- J3 pad 1: Net-(J3-Pad1) -> +5VA
- J6 pad 1: Net-(J6-Pad1) -> +5VA
- JP15 pad 1: /O2 Sensor/OUT -> Net-(JP15-Pad1)
- JP15 pad 2: /MCU/A7 -> Net-(C1-Pad1)
- JP16 pad 1: /MAP Sensor/OUT -> /Intake Air Temperature Sensor/IN
- JP16 pad 2: /MCU/A4 -> Net-(C14-Pad1)
- JP17 pad 1: /Throttle Position Sensor /OUT -> /Head Temperature Sensor/IN
- JP17 pad 2: /MCU/A5 -> Net-(C17-Pad1)
- JP18 pad 1: /Intake Air Temperature Sensor/OUT -> /O2 Sensor/IN
- JP18 pad 2: /MCU/A2 -> Net-(C7-Pad1)
- JP19 pad 1: /Head Temperature Sensor/OUT -> /Throttle Position Sensor /IN
- JP19 pad 2: /MCU/A3 -> Net-(C12-Pad1)
- JP20 pad 1: /Battery Reference Voltage/OUT -> /Oil Pressure Sensor/IN
- JP20 pad 2: /MCU/A0 -> Net-(C23-Pad1)
- JP21 pad 1: /Crankshaft pos sensor/OUT -> /Fuel Pressure/IN
- JP21 pad 2: /MCU/INT1 -> Net-(C33-Pad1)
- JP22 pad 1: /Oil Pressure Sensor/OUT -> /Crankshaft pos sensor/IN
- JP22 pad 2: /MCU/A6 -> Net-(C21-Pad1)
- JP23 pad 1: /Fuel Pressure/OUT -> Net-(JP23-Pad1)
- JP23 pad 2: /MCU/A1 -> Net-(C19-Pad1)
- JP30 pad 1: /MCU/PB7 -> /MCU/PA1
- R10 pad 1: /Fuel Pressure/OUT -> /MCU/A5
- R10 pad 2: /Fuel Pressure/IN -> Net-(C33-Pad1)
- R13 pad 1: /Battery Reference Voltage/+12V -> +12V
- R13 pad 2: Net-(C19-Pad1) -> Net-(JP23-Pad1)
- R14 pad 1: Net-(C19-Pad1) -> Net-(JP23-Pad1)
- R15 pad 1: /Battery Reference Voltage/OUT -> /MCU/A7
- R2 pad 1: /Intake Air Temperature Sensor/VCC -> +5VA
- R26 pad 1: /Crankshaft pos sensor/OUT -> /MCU/INT0
- R26 pad 2: /Crankshaft pos sensor/IN -> Net-(C21-Pad1)
- R27 pad 2: /MCU/sheet5D16F277/+12V -> +12V
- R3 pad 1: /Intake Air Temperature Sensor/OUT -> /MCU/A1
- R3 pad 2: /Intake Air Temperature Sensor/IN -> Net-(C14-Pad1)
- R4 pad 1: /Head Temperature Sensor/VCC -> +5VA
- R5 pad 1: /Head Temperature Sensor/OUT -> /MCU/A2
- R5 pad 2: /Head Temperature Sensor/IN -> Net-(C17-Pad1)
- R6 pad 1: /O2 Sensor/OUT -> /MCU/A6
- R6 pad 2: /O2 Sensor/IN -> Net-(C7-Pad1)
- R7 pad 1: /MAP Sensor/OUT -> /MCU/A0
- R7 pad 2: Net-(R7-Pad2) -> Net-(C1-Pad1)
- R8 pad 1: /Throttle Position Sensor /OUT -> /MCU/A3
- R8 pad 2: /Throttle Position Sensor /IN -> Net-(C12-Pad1)
- R9 pad 1: /Oil Pressure Sensor/OUT -> /MCU/A4
- R9 pad 2: /Oil Pressure Sensor/IN -> Net-(C23-Pad1)
- U3 pad 17: /MCU/PB7 -> (no net)
- U3 pad 25: /MCU/INT0 -> Net-(JP55-Pad2)
- U3 pad 26: /MCU/INT1 -> (no net)
- U3 pad 50: (no net) -> /MCU/PA1
- U3 pad 54: /MCU/A7 -> Net-(JP54-Pad2)
- U3 pad 55: /MCU/A6 -> Net-(JP52-Pad2)
- U3 pad 56: /MCU/A5 -> Net-(JP50-Pad2)
- U3 pad 57: /MCU/A4 -> Net-(JP40-Pad2)
- U3 pad 58: /MCU/A3 -> Net-(JP39-Pad2)
- U3 pad 59: /MCU/A2 -> Net-(JP49-Pad2)
- U3 pad 60: /MCU/A1 -> Net-(JP51-Pad2)
- U3 pad 61: /MCU/A0 -> Net-(JP53-Pad2)
- U4 pad 1: Net-(R7-Pad2) -> Net-(JP15-Pad1)
- U8 pad 7: /MCU/sheet5D16F277/+12V -> +12V
Routing:
- net /MCU/INT1: track 100.5 -> 0.00 mm, vias 1 -> 0
- net /MCU/A2: track 112.3 -> 15.9 mm, vias 1 -> 0
- net /MCU/A4: track 105.9 -> 15.9 mm, vias 1 -> 0
- net /MCU/A3: track 103.7 -> 15.9 mm, vias 1 -> 0
- net /Intake Air Temperature Sensor/IN: track 12.1 -> 96.6 mm
- net /Head Temperature Sensor/IN: track 12.1 -> 86.2 mm
- net /MCU/A5: track 87.9 -> 15.9 mm, vias 1 -> 0
- net /MCU/A6: track 79.4 -> 15.9 mm, vias 1 -> 0
- net +12V: track 142.1 -> 201.1 mm
- net /Throttle Position Sensor /IN: track 10.7 -> 68.0 mm
- net /MCU/PA1: track 0.00 -> 48.1 mm, vias 0 -> 1
- net /Oil Pressure Sensor/IN: track 10.7 -> 52.5 mm
- net /MCU/A1: track 56.9 -> 15.9 mm, vias 2 -> 0
- net /Crankshaft pos sensor/IN: track 10.7 -> 44.1 mm
- net +5VD: track 204.9 -> 237.3 mm, vias 2 -> 7
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Other:
- board text added: "EN"
- board text added: "VW Bus ECU rev 2 Powered by Speeduino 2019 Cedric Priscal"
- board text removed: "VW Bus ECU rev 2 Based on Speeduino 2019 Cedric Priscal"

Commit message: rev 2 sent to fab
Parts:
- added J15: Conn_01x08_Female, Pin_Headers:Pin_Header_Straight_1x08_Pitch2.54mm, F.Cu at (101.0, 97.8)
- C1: value 0.47n -> 0.47nF 50V
- C10: value 0.01u -> 10nF 100V
- C11: value 0.33u -> 0.33uF 50V
- C12, C14, C17, C19, C21, C23, C33, C7: value 0.1uF -> 0.1uF 50V
- C13, C15, C18, C20, C32, C34, C42, C8: value 0.22u -> 0.22uF 50V
- C16, C22, C35, C36, C4, C43: value 100nF -> 0.1uF 50V
- C2: value 4.7nF -> 4.7nF 100V
- C24, C26, C28, C30: value C -> 1nF 50V
- C25, C27, C29, C31: value C -> 22uF 16V
- C37, C38: value 22uF -> 22uF 25V
- C39, C9: value 1u -> 1uF 35V
- C40: value 22nF -> 22nF 50V
- C41: value 220nF -> 0.22uF 50V
- C46: value 1uF -> 1uF 35V
- C6: value 220pF -> 0.22nF 200V
- D10, D12, D14, D5, D8: value LED -> LED RED 10mA 1.9V
- D16, D19, D3: value LED -> LED GREEN 2.5mA 2.7V
- D17, D18, D2: value LED -> LED BLUE 10mA 3V
- PC2: value 47uF -> 47uF 10V
- PC3, PC4: value 47uF -> 47uF 10V; footprint Capacitors_SMD:C_1206 -> Capacitors_SMD:C_1206_HandSoldering
- R18, R22, R36, R40: value R_US -> 47.5k
- R19, R33, R37, R41: value R_US -> 1k
- R20, R34, R38, R42: value R_US -> 26.1k
- R31, R44, R45: value R_US -> 200
- R43, R49: value R_US -> 3.74k
- R50: value R_US -> 910
- R51: value R_US -> 309
- moved H3 25.4 mm to (284.5, 73.7)
- moved H4 25.4 mm to (284.5, 129.5)
- moved C10 12.7 mm to (177.8, 92.7)
- moved C9 12.7 mm to (177.8, 95.2)
- moved D3 12.7 mm to (180.3, 114.3)
- moved J12 12.7 mm to (184.2, 121.9)
- moved J5 12.7 mm to (212.1, 121.9)
- moved JP13 12.7 mm to (142.2, 107.3)
- moved JP14 12.7 mm to (152.4, 107.3)
- moved JP28 12.7 mm to (233.7, 95.2)
- moved JP29 12.7 mm to (233.7, 128.3)
- moved JP31 12.7 mm to (160.0, 111.1)
- moved JP39 12.7 mm to (132.1, 83.8)
- moved JP40 12.7 mm to (132.1, 86.4)
- moved JP45 12.7 mm to (195.6, 97.8)
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Connections:
- U3 pad 35: (no net) -> Net-(J15-Pad1)
- U3 pad 36: (no net) -> Net-(J15-Pad2)
- U3 pad 37: (no net) -> Net-(J15-Pad3)
- U3 pad 38: (no net) -> Net-(J15-Pad4)
- U3 pad 39: (no net) -> Net-(J15-Pad5)
- U3 pad 40: (no net) -> Net-(J15-Pad6)
- U3 pad 41: (no net) -> Net-(J15-Pad7)
- U3 pad 42: (no net) -> Net-(J15-Pad8)
Routing:
- net Net-(J15-Pad1): track 0.00 -> 8.54 mm
- net Net-(J15-Pad8): track 0.00 -> 8.44 mm
- net +5VD: track 237.3 -> 230.6 mm, vias 7 -> 8
- net Net-(J15-Pad7): track 0.00 -> 6.70 mm
- net Net-(J15-Pad2): track 0.00 -> 6.15 mm
- net Net-(JP42-Pad1): track 24.4 -> 30.2 mm
- net Net-(JP41-Pad1): track 31.9 -> 37.2 mm
- net Net-(J15-Pad6): track 0.00 -> 5.07 mm
- net Net-(J15-Pad3): track 0.00 -> 4.67 mm
- net Net-(J15-Pad5): track 0.00 -> 4.23 mm
- net Net-(J15-Pad4): track 0.00 -> 3.95 mm
- net /MCU/RESET: track 154.8 -> 156.3 mm
Other:
- board size 238.8 x 66 mm -> 264.2 x 66 mm
