File: hardware/analog_sensor.sch (KiCad schematic (older format))
At the start: 3 parts

Commit message: work in progress - components ordered
Changed lines of the file:
@@
 $Descr A4 11693 8268
 encoding utf-8
-Sheet 16 18
+Sheet 3 18
 Title ""
 Date ""
@@
 AR Path="/5C7018CC/5C658961" Ref="R9"  Part="1"
 AR Path="/5C704FE9/5C658961" Ref="R10"  Part="1"
-F 0 "R10" V 6153 3700 50  0000 C CNN
+AR Path="/5C76A7EA/5C658961" Ref="R26"  Part="1"
+F 0 "R6" V 6153 3700 50  0000 C CNN
 F 1 "470" V 6244 3700 50  0000 C CNN
 F 2 "Resistors_SMD:R_0805" V 6380 3700 50  0001 C CNN
@@
 AR Path="/5C7018CC/5C658ABD" Ref="#PWR060"  Part="1"
 AR Path="/5C704FE9/5C658ABD" Ref="#PWR061"  Part="1"
-F 0 "#PWR061" H 6450 4050 50  0001 C CNN
+AR Path="/5C76A7EA/5C658ABD" Ref="#PWR070"  Part="1"
+F 0 "#PWR070" H 6450 4050 50  0001 C CNN
 F 1 "GND" H 6455 4127 50  0000 C CNN
 F 2 "" H 6450 4300 50  0001 C CNN
@@
 AR Path="/5C7018CC/5C6BBB80" Ref="C23"  Part="1"
 AR Path="/5C704FE9/5C6BBB80" Ref="C33"  Part="1"
-F 0 "C33" H 5615 4041 50  0000 L CNN
+AR Path="/5C76A7EA/5C6BBB80" Ref="C21"  Part="1"
+F 0 "C7" H 5615 4041 50  0000 L CNN
 F 1 "0.1uF" H 5615 3950 50  0000 L CNN
 F 2 "Capacitors_SMD:C_0805" H 5538 3800 50  0001 C CNN
@@
 AR Path="/5C7018CC/5C6BBB88" Ref="C32"  Part="1"
 AR Path="/5C704FE9/5C6BBB88" Ref="C34"  Part="1"
-F 0 "C34" H 7365 4041 50  0000 L CNN
+AR Path="/5C76A7EA/5C6BBB88" Ref="C42"  Part="1"
+F 0 "C8" H 7365 4041 50  0000 L CNN
 F 1 "0.22u" H 7365 3950 50  0000 L CNN
 F 2 "Capacitors_SMD:C_0805" H 7288 3800 50  0001 C CNN

Commit message: rev 1
Changed lines of the file:
@@
 EESchema Schematic File Version 4
 LIBS:speeduino_mini-cache
-EELAYER 26 0
+EELAYER 29 0
 EELAYER END
 $Descr A4 11693 8268
 encoding utf-8
-Sheet 3 18
+Sheet 19 21
 Title ""
 Date ""
@@
 AR Path="/5C704FE9/5C658961" Ref="R10"  Part="1"
 AR Path="/5C76A7EA/5C658961" Ref="R26"  Part="1"
-F 0 "R6" V 6153 3700 50  0000 C CNN
+AR Path="/5C97692A/5C658961" Ref="R32"  Part="1"
+F 0 "R32" V 6153 3700 50  0000 C CNN
 F 1 "470" V 6244 3700 50  0000 C CNN
 F 2 "Resistors_SMD:R_0805" V 6380 3700 50  0001 C CNN
@@
 AR Path="/5C704FE9/5C658ABD" Ref="#PWR061"  Part="1"
 AR Path="/5C76A7EA/5C658ABD" Ref="#PWR070"  Part="1"
-F 0 "#PWR070" H 6450 4050 50  0001 C CNN
+AR Path="/5C97692A/5C658ABD" Ref="#PWR079"  Part="1"
+F 0 "#PWR079" H 6450 4050 50  0001 C CNN
 F 1 "GND" H 6455 4127 50  0000 C CNN
 F 2 "" H 6450 4300 50  0001 C CNN
@@
 AR Path="/5C704FE9/5C6BBB80" Ref="C33"  Part="1"
 AR Path="/5C76A7EA/5C6BBB80" Ref="C21"  Part="1"
-F 0 "C7" H 5615 4041 50  0000 L CNN
+AR Path="/5C97692A/5C6BBB80" Ref="C44"  Part="1"
+F 0 "C44" H 5615 4041 50  0000 L CNN
 F 1 "0.1uF" H 5615 3950 50  0000 L CNN
 F 2 "Capacitors_SMD:C_0805" H 5538 3800 50  0001 C CNN
@@
 AR Path="/5C704FE9/5C6BBB88" Ref="C34"  Part="1"
 AR Path="/5C76A7EA/5C6BBB88" Ref="C42"  Part="1"
-F 0 "C8" H 7365 4041 50  0000 L CNN
+AR Path="/5C97692A/5C6BBB88" Ref="C45"  Part="1"
+F 0 "C45" H 7365 4041 50  0000 L CNN
 F 1 "0.22u" H 7365 3950 50  0000 L CNN
 F 2 "Capacitors_SMD:C_0805" H 7288 3800 50  0001 C CNN

Commit message: Rev 2 work in progress
Parts:
- C7, C8: footprint Capacitors_SMD:C_0805 -> Capacitors_SMD:C_0805_HandSoldering
- R8: footprint Resistors_SMD:R_0805 -> Resistors_SMD:R_0805_HandSoldering
Changed lines of the file:
@@
 $Descr A4 11693 8268
 encoding utf-8
-Sheet 19 21
+Sheet 4 23
 Title ""
 Date ""
@@
 AR Path="/5C76A7EA/5C658961" Ref="R26"  Part="1"
 AR Path="/5C97692A/5C658961" Ref="R32"  Part="1"
-F 0 "R32" V 6153 3700 50  0000 C CNN
+F 0 "R8" V 6153 3700 50  0000 C CNN
 F 1 "470" V 6244 3700 50  0000 C CNN
-F 2 "Resistors_SMD:R_0805" V 6380 3700 50  0001 C CNN
+F 2 "Resistors_SMD:R_0805_HandSoldering" V 6380 3700 50  0001 C CNN
 F 3 "~" H 6450 3700 50  0001 C CNN
 F 4 "311-470ARCT-ND" V 6335 3700 50  0000 C CNN "DIGIKEY"
@@
 AR Path="/5C76A7EA/5C6BBB80" Ref="C21"  Part="1"
 AR Path="/5C97692A/5C6BBB80" Ref="C44"  Part="1"
-F 0 "C44" H 5615 4041 50  0000 L CNN
+F 0 "C12" H 5615 4041 50  0000 L CNN
 F 1 "0.1uF" H 5615 3950 50  0000 L CNN
-F 2 "Capacitors_SMD:C_0805" H 5538 3800 50  0001 C CNN
+F 2 "Capacitors_SMD:C_0805_HandSoldering" H 5538 3800 50  0001 C CNN
 F 3 "~" H 5500 3950 50  0001 C CNN
 F 4 "478-6048-1-ND" H 5615 3859 50  0000 L CNN "DIGIKEY"
@@
 AR Path="/5C76A7EA/5C6BBB88" Ref="C42"  Part="1"
 AR Path="/5C97692A/5C6BBB88" Ref="C45"  Part="1"
-F 0 "C45" H 7365 4041 50  0000 L CNN
+F 0 "C13" H 7365 4041 50  0000 L CNN
 F 1 "0.22u" H 7365 3950 50  0000 L CNN
-F 2 "Capacitors_SMD:C_0805" H 7288 3800 50  0001 C CNN
+F 2 "Capacitors_SMD:C_0805_HandSoldering" H 7288 3800 50  0001 C CNN
 F 3 "~" H 7250 3950 50  0001 C CNN
 F 4 "1276-7012-1-ND" H 7365 3859 50  0000 L CNN "DIGIKEY"

Commit message: rev 2 work in progress
Changed lines of the file:
@@
 $Descr A4 11693 8268
 encoding utf-8
-Sheet 4 23
+Sheet 2 22
 Title ""
 Date ""
@@
 AR Path="/5C76A7EA/5C658961" Ref="R26"  Part="1"
 AR Path="/5C97692A/5C658961" Ref="R32"  Part="1"
-F 0 "R8" V 6153 3700 50  0000 C CNN
+F 0 "R6" V 6153 3700 50  0000 C CNN
 F 1 "470" V 6244 3700 50  0000 C CNN
 F 2 "Resistors_SMD:R_0805_HandSoldering" V 6380 3700 50  0001 C CNN
@@
 AR Path="/5C76A7EA/5C658ABD" Ref="#PWR070"  Part="1"
 AR Path="/5C97692A/5C658ABD" Ref="#PWR079"  Part="1"
-F 0 "#PWR079" H 6450 4050 50  0001 C CNN
+F 0 "#PWR070" H 6450 4050 50  0001 C CNN
 F 1 "GND" H 6455 4127 50  0000 C CNN
 F 2 "" H 6450 4300 50  0001 C CNN
@@
 AR Path="/5C76A7EA/5C6BBB80" Ref="C21"  Part="1"
 AR Path="/5C97692A/5C6BBB80" Ref="C44"  Part="1"
-F 0 "C12" H 5615 4041 50  0000 L CNN
+F 0 "C7" H 5615 4041 50  0000 L CNN
 F 1 "0.1uF" H 5615 3950 50  0000 L CNN
 F 2 "Capacitors_SMD:C_0805_HandSoldering" H 5538 3800 50  0001 C CNN
@@
 AR Path="/5C76A7EA/5C6BBB88" Ref="C42"  Part="1"
 AR Path="/5C97692A/5C6BBB88" Ref="C45"  Part="1"
-F 0 "C13" H 7365 4041 50  0000 L CNN
+F 0 "C8" H 7365 4041 50  0000 L CNN
 F 1 "0.22u" H 7365 3950 50  0000 L CNN
 F 2 "Capacitors_SMD:C_0805_HandSoldering" H 7288 3800 50  0001 C CNN

Commit message: hardware rev2 - layout complete
Parts:
- added JP18: Jumper, Pin_Headers:Pin_Header_Straight_1x02_Pitch2.54mm, symbol Device:Jumper
Connections:
- net IN: now also JP18.1; no longer C7.1, R8.2
- new net: C7.1, JP18.2, R8.2
Changed lines of the file:
@@
 $Descr A4 11693 8268
 encoding utf-8
-Sheet 2 22
+Sheet 13 22
 Title ""
 Date ""
@@
 Comment4 ""
 $EndDescr
-Text HLabel 5350 3700 0    50   Input ~ 0
+Text HLabel 4750 3700 0    50   Input ~ 0
 IN
 Text HLabel 7450 3700 2    50   Output ~ 0
@@
 AR Path="/5C76A7EA/5C658961" Ref="R26"  Part="1"
 AR Path="/5C97692A/5C658961" Ref="R32"  Part="1"
-F 0 "R6" V 6153 3700 50  0000 C CNN
+F 0 "R26" V 6153 3700 50  0000 C CNN
 F 1 "470" V 6244 3700 50  0000 C CNN
 F 2 "Resistors_SMD:R_0805_HandSoldering" V 6380 3700 50  0001 C CNN
@@
 AR Path="/5C76A7EA/5C6BBB80" Ref="C21"  Part="1"
 AR Path="/5C97692A/5C6BBB80" Ref="C44"  Part="1"
-F 0 "C7" H 5615 4041 50  0000 L CNN
+F 0 "C21" H 5615 4041 50  0000 L CNN
 F 1 "0.1uF" H 5615 3950 50  0000 L CNN
 F 2 "Capacitors_SMD:C_0805_HandSoldering" H 5538 3800 50  0001 C CNN
@@
 AR Path="/5C76A7EA/5C6BBB88" Ref="C42"  Part="1"
 AR Path="/5C97692A/5C6BBB88" Ref="C45"  Part="1"
-F 0 "C8" H 7365 4041 50  0000 L CNN
+F 0 "C42" H 7365 4041 50  0000 L CNN
 F 1 "0.22u" H 7365 3950 50  0000 L CNN
 F 2 "Capacitors_SMD:C_0805_HandSoldering" H 7288 3800 50  0001 C CNN
@@
 	1    0    0    -1
 $EndComp
+$Comp
+L Device:Jumper JP?
+U 1 1 5D012CE2
+P 5050 3700
+AR Path="/5D012CE2" Ref="JP?"  Part="1"
+AR Path="/5C64D270/5D012CE2" Ref="JP18"  Part="1"
+AR Path="/5C6588EC/5D012CE2" Ref="JP19"  Part="1"
+AR Path="/5C7018CC/5D012CE2" Ref="JP20"  Part="1"
+AR Path="/5C704FE9/5D012CE2" Ref="JP21"  Part="1"
+AR Path="/5C76A7EA/5D012CE2" Ref="JP22"  Part="1"
+F 0 "JP22" H 5050 3964 50  0000 C CNN
+F 1 "Jumper" H 5050 3873 50  0000 C CNN
+F 2 "Pin_Headers:Pin_Header_Straight_1x02_Pitch2.54mm" H 5050 3700 50  0001 C CNN
+F 3 "~" H 5050 3700 50  0001 C CNN
+	1    5050 3700
+	1    0    0    -1
+$EndComp

Commit message: rev 2 sent to fab
Parts:
- C7: value 0.1uF -> 0.1uF 50V; DIGIKEY 478-6048-1-ND -> (none); DigiKey (none) -> 478-6048-1-ND
- C8: value 0.22u -> 0.22uF 50V; DIGIKEY 1276-7012-1-ND -> (none); DigiKey (none) -> 445-5683-1-ND
- JP18: DigiKey (none) -> S9337-ND
- R8: DIGIKEY 311-470ARCT-ND -> (none); DigiKey (none) -> 311-470ARCT-ND
Changed lines of the file:
@@
 F 2 "Resistors_SMD:R_0805_HandSoldering" V 6380 3700 50  0001 C CNN
 F 3 "~" H 6450 3700 50  0001 C CNN
-F 4 "311-470ARCT-ND" V 6335 3700 50  0000 C CNN "DIGIKEY"
+F 4 "311-470ARCT-ND" H 0   0   50  0001 C CNN "DigiKey"
 	1    6450 3700
 	0    1    1    0
@@
 AR Path="/5C97692A/5C6BBB80" Ref="C44"  Part="1"
 F 0 "C21" H 5615 4041 50  0000 L CNN
-F 1 "0.1uF" H 5615 3950 50  0000 L CNN
+F 1 "0.1uF 50V" H 5615 3950 50  0000 L CNN
 F 2 "Capacitors_SMD:C_0805_HandSoldering" H 5538 3800 50  0001 C CNN
 F 3 "~" H 5500 3950 50  0001 C CNN
-F 4 "478-6048-1-ND" H 5615 3859 50  0000 L CNN "DIGIKEY"
+F 4 "478-6048-1-ND" H 0   0   50  0001 C CNN "DigiKey"
 	1    5500 3950
 	1    0    0    -1
@@
 AR Path="/5C97692A/5C6BBB88" Ref="C45"  Part="1"
 F 0 "C42" H 7365 4041 50  0000 L CNN
-F 1 "0.22u" H 7365 3950 50  0000 L CNN
+F 1 "0.22uF 50V" H 7365 3950 50  0000 L CNN
 F 2 "Capacitors_SMD:C_0805_HandSoldering" H 7288 3800 50  0001 C CNN
 F 3 "~" H 7250 3950 50  0001 C CNN
-F 4 "1276-7012-1-ND" H 7365 3859 50  0000 L CNN "DIGIKEY"
+F 4 "445-5683-1-ND" H 0   0   50  0001 C CNN "DigiKey"
 	1    7250 3950
 	1    0    0    -1
@@
 F 2 "Pin_Headers:Pin_Header_Straight_1x02_Pitch2.54mm" H 5050 3700 50  0001 C CNN
 F 3 "~" H 5050 3700 50  0001 C CNN
+F 4 "S9337-ND" H 0   0   50  0001 C CNN "DigiKey"
 	1    5050 3700
 	1    0    0    -1

Commit message: old commit from v1
Changed lines of the file:
@@
 EESchema Schematic File Version 4
-LIBS:speeduino_mini-cache
-EELAYER 29 0
+EELAYER 30 0
 EELAYER END
 $Descr A4 11693 8268
 encoding utf-8
-Sheet 13 22
+Sheet 4 23
 Title ""
 Date ""
@@
 AR Path="/5C76A7EA/5C658961" Ref="R26"  Part="1"
 AR Path="/5C97692A/5C658961" Ref="R32"  Part="1"
-F 0 "R26" V 6153 3700 50  0000 C CNN
+F 0 "R8" V 6153 3700 50  0000 C CNN
 F 1 "470" V 6244 3700 50  0000 C CNN
 F 2 "Resistors_SMD:R_0805_HandSoldering" V 6380 3700 50  0001 C CNN
@@
 AR Path="/5C76A7EA/5C658ABD" Ref="#PWR070"  Part="1"
 AR Path="/5C97692A/5C658ABD" Ref="#PWR079"  Part="1"
-F 0 "#PWR070" H 6450 4050 50  0001 C CNN
+F 0 "#PWR059" H 6450 4050 50  0001 C CNN
 F 1 "GND" H 6455 4127 50  0000 C CNN
 F 2 "" H 6450 4300 50  0001 C CNN
@@
 AR Path="/5C76A7EA/5C6BBB80" Ref="C21"  Part="1"
 AR Path="/5C97692A/5C6BBB80" Ref="C44"  Part="1"
-F 0 "C21" H 5615 4041 50  0000 L CNN
+F 0 "C12" H 5615 4041 50  0000 L CNN
 F 1 "0.1uF 50V" H 5615 3950 50  0000 L CNN
 F 2 "Capacitors_SMD:C_0805_HandSoldering" H 5538 3800 50  0001 C CNN
@@
 AR Path="/5C76A7EA/5C6BBB88" Ref="C42"  Part="1"
 AR Path="/5C97692A/5C6BBB88" Ref="C45"  Part="1"
-F 0 "C42" H 7365 4041 50  0000 L CNN
+F 0 "C13" H 7365 4041 50  0000 L CNN
 F 1 "0.22uF 50V" H 7365 3950 50  0000 L CNN
 F 2 "Capacitors_SMD:C_0805_HandSoldering" H 7288 3800 50  0001 C CNN
@@
 AR Path="/5C704FE9/5D012CE2" Ref="JP21"  Part="1"
 AR Path="/5C76A7EA/5D012CE2" Ref="JP22"  Part="1"
-F 0 "JP22" H 5050 3964 50  0000 C CNN
+F 0 "JP19" H 5050 3964 50  0000 C CNN
 F 1 "Jumper" H 5050 3873 50  0000 C CNN
 F 2 "Pin_Headers:Pin_Header_Straight_1x02_Pitch2.54mm" H 5050 3700 50  0001 C CNN
