File: hardware/atmega_regulator.sch (KiCad schematic (older format))
At the start: 9 parts, among them U12 LD1117S50TR_SOT223

Commit message: rev 2 work in progress
Parts:
- added JP46, JP47: Jumper, Pin_Headers:Pin_Header_Straight_1x02_Pitch2.54mm, symbol Device:Jumper
Connections:
- net +12V: now also JP46.1; no longer C16.1, PC1.1, U12.3 (VI)
- net VCC: now also JP47.2; no longer C22.1, C35.1, C36.1, PC2.1, U12.2 (VO)
- new net: C22.1, C35.1, C36.1, JP47.1, PC2.1, U12.2 (VO)
- new net: C16.1, JP46.2, PC1.1, U12.3 (VI)
Other:
- moved on the sheet: C16, C22, C35, C36, C43, L1, PC1, PC2, U12

Commit message: rev 2 sent to fab
Parts:
- C16, C22, C35, C36, C43: value 100nF -> 0.1uF 50V; DIGIKEY 478-6048-1-ND -> (none); DigiKey (none) -> 478-6048-1-ND
- JP46, JP47: DigiKey (none) -> S9337-ND
- L1: DIGIKEY 445-6396-1-ND -> (none); DigiKey (none) -> 445-6396-1-ND
- PC1: DIGIKEY 478-1773-1-ND -> (none); DigiKey (none) -> 478-1773-1-ND
- PC2: value 47uF -> 47uF 10V; DIGIKEY 490-12438-1-ND -> (none); DigiKey (none) -> 490-12438-1-ND
- U12: DIGIKEY 497-1243-1-ND -> (none); DigiKey (none) -> 497-1243-1-ND
Changed lines of the file:
@@
 AR Path="/5C610827/5D1A080F/5D1A1700" Ref="PC2"  Part="1"
 F 0 "PC2" H 5165 3791 50  0000 L CNN
-F 1 "47uF" H 5165 3700 50  0000 L CNN
+F 1 "47uF 10V" H 5165 3700 50  0000 L CNN
 F 2 "Capacitors_SMD:C_1206_HandSoldering" H 5088 3550 50  0001 C CNN
 F 3 "~" H 5050 3700 50  0001 C CNN
-F 4 "490-12438-1-ND" H 5165 3609 50  0000 L CNN "DIGIKEY"
+F 4 "490-12438-1-ND" H 0   0   50  0001 C CNN "DigiKey"
 	1    5050 3700
 	1    0    0    -1
@@
 F 2 "Capacitors_Tantalum_SMD:CP_Tantalum_Case-C_EIA-6032-28_Reflow" H 2438 3550 50  0001 C CNN
 F 3 "~" H 2400 3700 50  0001 C CNN
-F 4 "478-1773-1-ND" H 2518 3609 50  0000 L CNN "DIGIKEY"
+F 4 "478-1773-1-ND" H 0   0   50  0001 C CNN "DigiKey"
 	1    2400 3700
 	1    0    0    -1
@@
 AR Path="/5C610827/5D1A080F/5D1A171C" Ref="C16"  Part="1"
 F 0 "C16" H 3565 3791 50  0000 L CNN
-F 1 "100nF" H 3565 3700 50  0000 L CNN
+F 1 "0.1uF 50V" H 3565 3700 50  0000 L CNN
 F 2 "Capacitors_SMD:C_0805_HandSoldering" H 3488 3550 50  0001 C CNN
 F 3 "~" H 3450 3700 50  0001 C CNN
-F 4 "478-6048-1-ND" H 3565 3609 50  0000 L CNN "DIGIKEY"
+F 4 "478-6048-1-ND" H 0   0   50  0001 C CNN "DigiKey"
 	1    3450 3700
 	1    0    0    -1
@@
 F 2 "TO_SOT_Packages_SMD:SOT-223-3_TabPin2" H 4350 3700 50  0001 C CNN
 F 3 "http://www.st.com/st-web-ui/static/active/en/resource/technical/document/datasheet/CD00000544.pdf" H 4450 3250 50  0001 C CNN
-F 4 "497-1243-1-ND" H 4350 3650 50  0000 C CNN "DIGIKEY"
+F 4 "497-1243-1-ND" H 0   0   50  0001 C CNN "DigiKey"
 	1    4350 3500
 	1    0    0    -1
@@
 AR Path="/5C610827/5D1A080F/5D1A98C9" Ref="C22"  Part="1"
 F 0 "C22" H 6215 3791 50  0000 L CNN
-F 1 "100nF" H 6215 3700 50  0000 L CNN
+F 1 "0.1uF 50V" H 6215 3700 50  0000 L CNN
 F 2 "Capacitors_SMD:C_0805_HandSoldering" H 6138 3550 50  0001 C CNN
 F 3 "~" H 6100 3700 50  0001 C CNN
-F 4 "478-6048-1-ND" H 6215 3609 50  0000 L CNN "DIGIKEY"
+F 4 "478-6048-1-ND" H 0   0   50  0001 C CNN "DigiKey"
 	1    6100 3700
 	1    0    0    -1
@@
 AR Path="/5C610827/5D1A080F/5D1A98D0" Ref="C35"  Part="1"
 F 0 "C35" H 7265 3791 50  0000 L CNN
-F 1 "100nF" H 7265 3700 50  0000 L CNN
+F 1 "0.1uF 50V" H 7265 3700 50  0000 L CNN
 F 2 "Capacitors_SMD:C_0805_HandSoldering" H 7188 3550 50  0001 C CNN
 F 3 "~" H 7150 3700 50  0001 C CNN
-F 4 "478-6048-1-ND" H 7265 3609 50  0000 L CNN "DIGIKEY"
+F 4 "478-6048-1-ND" H 0   0   50  0001 C CNN "DigiKey"
 	1    7150 3700
 	1    0    0    -1
@@
 AR Path="/5C610827/5D1A080F/5D1A98D7" Ref="C36"  Part="1"
 F 0 "C36" H 8265 3791 50  0000 L CNN
-F 1 "100nF" H 8265 3700 50  0000 L CNN
+F 1 "0.1uF 50V" H 8265 3700 50  0000 L CNN
 F 2 "Capacitors_SMD:C_0805_HandSoldering" H 8188 3550 50  0001 C CNN
 F 3 "~" H 8150 3700 50  0001 C CNN
-F 4 "478-6048-1-ND" H 8265 3609 50  0000 L CNN "DIGIKEY"
+F 4 "478-6048-1-ND" H 0   0   50  0001 C CNN "DigiKey"
 	1    8150 3700
 	1    0    0    -1
@@
 AR Path="/5C610827/5D1A080F/5D1A98E4" Ref="C43"  Part="1"
 F 0 "C43" H 10065 3791 50  0000 L CNN
-F 1 "100nF" H 10065 3700 50  0000 L CNN
+F 1 "0.1uF 50V" H 10065 3700 50  0000 L CNN
 F 2 "Capacitors_SMD:C_0805_HandSoldering" H 9988 3550 50  0001 C CNN
 F 3 "~" H 9950 3700 50  0001 C CNN
-F 4 "478-6048-1-ND" H 10065 3609 50  0000 L CNN "DIGIKEY"
+F 4 "478-6048-1-ND" H 0   0   50  0001 C CNN "DigiKey"
 	1    9950 3700
 	1    0    0    -1
@@
 F 2 "Inductors_SMD:L_0805_HandSoldering" H 9400 3500 50  0001 C CNN
 F 3 "~" H 9400 3500 50  0001 C CNN
-F 4 "445-6396-1-ND" V 9498 3500 50  0000 C CNN "DIGIKEY"
+F 4 "445-6396-1-ND" H 0   0   50  0001 C CNN "DigiKey"
 	1    9400 3500
 	0    -1   -1   0
@@
 F 2 "Pin_Headers:Pin_Header_Straight_1x02_Pitch2.54mm" H 8800 3500 50  0001 C CNN
 F 3 "~" H 8800 3500 50  0001 C CNN
+F 4 "S9337-ND" H 0   0   50  0001 C CNN "DigiKey"
 	1    8800 3500
 	1    0    0    -1
@@
 F 2 "Pin_Headers:Pin_Header_Straight_1x02_Pitch2.54mm" H 1850 3500 50  0001 C CNN
 F 3 "~" H 1850 3500 50  0001 C CNN
+F 4 "S9337-ND" H 0   0   50  0001 C CNN "DigiKey"
 	1    1850 3500
 	1    0    0    -1
