File: hardware/ignitor.sch (KiCad schematic (older format))
At the start: 8 parts, among them U5 TC4424_SOIC

Commit message: Rev 2 work in progress
Parts:
- removed C22: 1u, Capacitors_SMD:C_0805, symbol Device:C
- removed R21, R22: 150, Resistors_SMD:R_0805, symbol Device:R
- removed R23, R24: 10k, Resistors_SMD:R_0805, symbol Device:R
- removed R27, R28: 160, Resistors_SMD:R_2512, symbol Device:R
- removed U5: TC4424_SOIC, Housings_SOIC:SOIC-16W_7.5x10.3mm_Pitch1.27mm, symbol speeduino_mini:TC4424_SOIC
- added D17, D18: LED, LEDs:LED_0805_HandSoldering, symbol Device:LED
- added J11: Ignitor Pack, Speeduino Mini:ED120_4DS, symbol Connector:Screw_Terminal_01x04
- added R44, R45: R_US, Resistors_SMD:R_0805_HandSoldering, symbol Device:R_US
Connections:
- net labels added: +12V, EN, IN1, IN2
- net labels removed: +5V, IGN1_IN, IGN1_OUT, IGN2_IN, IGN2_OUT
- wire segments 37 -> 18

Commit message: rev 2 sent to fab
Parts:
- D17, D18: value LED -> LED BLUE 10mA 3V; DigiKey (none) -> 732-4982-1-ND
- J11: DIGIKEY ED2227-ND -> (none); DigiKey (none) -> ED2227-ND
- R44, R45: value R_US -> 200; DigiKey (none) -> P200CCT-ND
Other:
- moved on the sheet: D18, R45
Changed lines of the file:
@@
 L Device:LED D?
 U 1 1 5CF8A0F2
-P 7000 4550
+P 7000 4750
 AR Path="/5C667F1A/5CF8A0F2" Ref="D?"  Part="1"
 AR Path="/5C668FC1/5CF8A0F2" Ref="D?"  Part="1"
@@
 AR Path="/5CF8A0F2" Ref="D?"  Part="1"
 AR Path="/5CF868AF/5CF8A0F2" Ref="D18"  Part="1"
-F 0 "D18" V 7039 4433 50  0000 R CNN
-F 1 "LED" V 6948 4433 50  0000 R CNN
-F 2 "LEDs:LED_0805_HandSoldering" H 7000 4550 50  0001 C CNN
-F 3 "~" H 7000 4550 50  0001 C CNN
-	1    7000 4550
+F 0 "D18" V 7084 4632 50  0000 R CNN
+F 1 "LED BLUE 10mA 3V" V 6993 4632 50  0000 R CNN
+F 2 "LEDs:LED_0805_HandSoldering" H 7000 4750 50  0001 C CNN
+F 3 "https://katalog.we-online.de/led/datasheet/150080BS75000.pdf" H 7000 4750 50  0001 C CNN
+F 4 "732-4982-1-ND" V 6902 4632 50  0000 R CNN "DigiKey"
+	1    7000 4750
 	0    -1   -1   0
 $EndComp
@@
 L Device:R_US R?
 U 1 1 5CF8A0F8
-P 7000 3900
+P 7000 4100
 AR Path="/5C667F1A/5CF8A0F8" Ref="R?"  Part="1"
 AR Path="/5C668FC1/5CF8A0F8" Ref="R?"  Part="1"
@@
 AR Path="/5CF8A0F8" Ref="R?"  Part="1"
 AR Path="/5CF868AF/5CF8A0F8" Ref="R45"  Part="1"
-F 0 "R45" H 6932 3854 50  0000 R CNN
-F 1 "R_US" H 6932 3945 50  0000 R CNN
-F 2 "Resistors_SMD:R_0805_HandSoldering" V 7040 3890 50  0001 C CNN
-F 3 "~" H 7000 3900 50  0001 C CNN
-	1    7000 3900
+F 0 "R45" H 6932 4009 50  0000 R CNN
+F 1 "200" H 6932 4100 50  0000 R CNN
+F 2 "Resistors_SMD:R_0805_HandSoldering" V 7040 4090 50  0001 C CNN
+F 3 "https://industrial.panasonic.com/cdbs/www-data/pdf/RDA0000/AOA0000C304.pdf" H 7000 4100 50  0001 C CNN
+F 4 "P200CCT-ND" H 6932 4191 50  0000 R CNN "DigiKey"
+	1    7000 4100
 	-1   0    0    1
 $EndComp
 Wire Wire Line
-	7000 4050 7000 4400
+	7000 4250 7000 4600
 Wire Wire Line
-	7000 3750 7000 3300
+	7000 3950 7000 3300
 Wire Wire Line
-	7000 4700 7000 5000
+	7000 4900 7000 5200
 $Comp
 L Device:LED D?
@@
 AR Path="/5CF8A101" Ref="D?"  Part="1"
 AR Path="/5CF868AF/5CF8A101" Ref="D17"  Part="1"
-F 0 "D17" V 5939 4633 50  0000 R CNN
-F 1 "LED" V 5848 4633 50  0000 R CNN
+F 0 "D17" V 5984 4632 50  0000 R CNN
+F 1 "LED BLUE 10mA 3V" V 5893 4632 50  0000 R CNN
 F 2 "LEDs:LED_0805_HandSoldering" H 5900 4750 50  0001 C CNN
 F 3 "~" H 5900 4750 50  0001 C CNN
+F 4 "732-4982-1-ND" V 5802 4632 50  0000 R CNN "DigiKey"
 	1    5900 4750
 	0    -1   -1   0
@@
 AR Path="/5CF8A107" Ref="R?"  Part="1"
 AR Path="/5CF868AF/5CF8A107" Ref="R44"  Part="1"
-F 0 "R44" H 5832 4054 50  0000 R CNN
-F 1 "R_US" H 5832 4145 50  0000 R CNN
+F 0 "R44" H 5832 4009 50  0000 R CNN
+F 1 "200" H 5832 4100 50  0000 R CNN
 F 2 "Resistors_SMD:R_0805_HandSoldering" V 5940 4090 50  0001 C CNN
-F 3 "~" H 5900 4100 50  0001 C CNN
+F 3 "https://industrial.panasonic.com/cdbs/www-data/pdf/RDA0000/AOA0000C304.pdf" H 5900 4100 50  0001 C CNN
+F 4 "P200CCT-ND" H 5832 4191 50  0000 R CNN "DigiKey"
 	1    5900 4100
 	-1   0    0    1
@@
 L power:GND #PWR?
 U 1 1 5CF8A116
-P 7000 5000
+P 7000 5200
 AR Path="/5CF8A116" Ref="#PWR?"  Part="1"
 AR Path="/5CF868AF/5CF8A116" Ref="#PWR0104"  Part="1"
-F 0 "#PWR0104" H 7000 4750 50  0001 C CNN
-F 1 "GND" H 7005 4827 50  0000 C CNN
-F 2 "" H 7000 5000 50  0001 C CNN
-F 3 "" H 7000 5000 50  0001 C CNN
-	1    7000 5000
+F 0 "#PWR0104" H 7000 4950 50  0001 C CNN
+F 1 "GND" H 7005 5027 50  0000 C CNN
+F 2 "" H 7000 5200 50  0001 C CNN
+F 3 "" H 7000 5200 50  0001 C CNN
+	1    7000 5200
 	1    0    0    -1
 $EndComp
@@
 F 2 "Speeduino Mini:ED120_4DS" H 8050 3400 50  0001 C CNN
 F 3 "~" H 8050 3400 50  0001 C CNN
-F 4 "ED2227-ND" H 8129 3255 50  0000 L CNN "DIGIKEY"
+F 4 "ED2227-ND" H 0   0   50  0001 C CNN "DigiKey"
 	1    8050 3400
 	1    0    0    -1
