File: hardware/injector.sch (KiCad schematic (older format))
At the start: 3 parts, among them Q1 SQ2318AES-T1_GE3

Commit message: rev 1
Parts:
- Q1: symbol Device:Q_NMOS_GDS -> Device:Q_NMOS_GSD
Changed lines of the file:
@@
 EESchema Schematic File Version 4
 LIBS:speeduino_mini-cache
-EELAYER 26 0
+EELAYER 29 0
 EELAYER END
 $Descr A4 11693 8268
 encoding utf-8
-Sheet 10 18
+Sheet 9 21
 Title ""
 Date ""
@@
 AR Path="/5C667F1A/5C667F34" Ref="R17"  Part="1"
 AR Path="/5C668FC1/5C667F34" Ref="R19"  Part="1"
-F 0 "R19" H 5070 4141 50  0000 L CNN
+AR Path="/5C9BF5B5/5C667F34" Ref="R33"  Part="1"
+AR Path="/5C9C0039/5C667F34" Ref="R35"  Part="1"
+F 0 "R17" H 5070 4141 50  0000 L CNN
 F 1 "10k" H 5070 4050 50  0000 L CNN
 F 2 "Resistors_SMD:R_0805" V 4930 4050 50  0001 C CNN
@@
 AR Path="/5C667F1A/5C667F5C" Ref="R18"  Part="1"
 AR Path="/5C668FC1/5C667F5C" Ref="R20"  Part="1"
-F 0 "R20" V 5303 3800 50  0000 C CNN
+AR Path="/5C9BF5B5/5C667F5C" Ref="R34"  Part="1"
+AR Path="/5C9C0039/5C667F5C" Ref="R36"  Part="1"
+F 0 "R18" V 5303 3800 50  0000 C CNN
 F 1 "150" V 5394 3800 50  0000 C CNN
 F 2 "Resistors_SMD:R_0805" V 5530 3800 50  0001 C CNN
@@
 AR Path="/5C667F1A/5C667FBF" Ref="#PWR031"  Part="1"
 AR Path="/5C668FC1/5C667FBF" Ref="#PWR032"  Part="1"
-F 0 "#PWR032" H 5000 4050 50  0001 C CNN
+AR Path="/5C9BF5B5/5C667FBF" Ref="#PWR0103"  Part="1"
+AR Path="/5C9C0039/5C667FBF" Ref="#PWR0104"  Part="1"
+F 0 "#PWR031" H 5000 4050 50  0001 C CNN
 F 1 "GND" H 5005 4127 50  0000 C CNN
 F 2 "" H 5000 4300 50  0001 C CNN
@@
 $EndComp
 $Comp
-L Device:Q_NMOS_GDS Q1
+L Device:Q_NMOS_GSD Q1
 U 1 1 5C6682FE
 P 6250 3800
 AR Path="/5C667F1A/5C6682FE" Ref="Q1"  Part="1"
 AR Path="/5C668FC1/5C6682FE" Ref="Q2"  Part="1"
-F 0 "Q2" H 6456 3891 50  0000 L CNN
+AR Path="/5C9BF5B5/5C6682FE" Ref="Q6"  Part="1"
+AR Path="/5C9C0039/5C6682FE" Ref="Q7"  Part="1"
+F 0 "Q1" H 6456 3891 50  0000 L CNN
 F 1 "SQ2318AES-T1_GE3" H 6456 3800 50  0000 L CNN
 F 2 "TO_SOT_Packages_SMD:SOT-23" H 6450 3900 50  0001 C CNN

Commit message: rev 1.1
Changed lines of the file:
@@
 $Descr A4 11693 8268
 encoding utf-8
-Sheet 9 21
+Sheet 21 21
 Title ""
 Date ""
@@
 AR Path="/5C9BF5B5/5C667F34" Ref="R33"  Part="1"
 AR Path="/5C9C0039/5C667F34" Ref="R35"  Part="1"
-F 0 "R17" H 5070 4141 50  0000 L CNN
+F 0 "R35" H 5070 4141 50  0000 L CNN
 F 1 "10k" H 5070 4050 50  0000 L CNN
 F 2 "Resistors_SMD:R_0805" V 4930 4050 50  0001 C CNN
@@
 AR Path="/5C9BF5B5/5C667F5C" Ref="R34"  Part="1"
 AR Path="/5C9C0039/5C667F5C" Ref="R36"  Part="1"
-F 0 "R18" V 5303 3800 50  0000 C CNN
+F 0 "R36" V 5303 3800 50  0000 C CNN
 F 1 "150" V 5394 3800 50  0000 C CNN
 F 2 "Resistors_SMD:R_0805" V 5530 3800 50  0001 C CNN
@@
 AR Path="/5C9BF5B5/5C667FBF" Ref="#PWR0103"  Part="1"
 AR Path="/5C9C0039/5C667FBF" Ref="#PWR0104"  Part="1"
-F 0 "#PWR031" H 5000 4050 50  0001 C CNN
+F 0 "#PWR0104" H 5000 4050 50  0001 C CNN
 F 1 "GND" H 5005 4127 50  0000 C CNN
 F 2 "" H 5000 4300 50  0001 C CNN
@@
 AR Path="/5C9BF5B5/5C6682FE" Ref="Q6"  Part="1"
 AR Path="/5C9C0039/5C6682FE" Ref="Q7"  Part="1"
-F 0 "Q1" H 6456 3891 50  0000 L CNN
+F 0 "Q7" H 6456 3891 50  0000 L CNN
 F 1 "SQ2318AES-T1_GE3" H 6456 3800 50  0000 L CNN
 F 2 "TO_SOT_Packages_SMD:SOT-23" H 6450 3900 50  0001 C CNN

Commit message: Rev 2 work in progress
Parts:
- removed Q1: SQ2318AES-T1_GE3, TO_SOT_Packages_SMD:SOT-23, symbol Device:Q_NMOS_GSD
- removed R18: 150, Resistors_SMD:R_0805, symbol Device:R
- added C24, C25: C, Capacitors_SMD:C_0805_HandSoldering, symbol Device:C
- added D8: LED, LEDs:LED_0805_HandSoldering, symbol Device:LED
- added D9: B340A-13-F, Diodes_SMD:D_SMA_Handsoldering, symbol Device:D_Schottky
- added J7: Injector, Speeduino Mini:ED120_2DS, symbol Connector:Screw_Terminal_01x02
- added R18, R19, R20: R_US, Resistors_SMD:R_0805_HandSoldering, symbol Device:R_US
- added U7: DRV103H, Housings_SOIC:TI_SO-PowerPAD-8, symbol DRV103H:DRV103H
- R17: footprint Resistors_SMD:R_0805 -> Resistors_SMD:R_0805_HandSoldering
Connections:
- net labels added: +12V
- net labels removed: INJ_OUT
- wire segments 10 -> 32

Commit message: rev 2 sent to fab
Parts:
- C24: value C -> 1nF 50V; DigiKey (none) -> 478-1371-1-ND
- C25: value C -> 22uF 16V; symbol Device:C -> Device:CP; DigiKey (none) -> 490-9956-1-ND
- D8: value LED -> LED RED 10mA 1.9V; DigiKey (none) -> 732-4984-1-ND
- J7: DIGIKEY ED1609-ND -> (none); DigiKey (none) -> ED1609-ND
- R17: symbol Device:R -> Device:R_US; DIGIKEY 311-10.0KCRCT-ND -> (none); DigiKey (none) -> 311-10.0KCRCT-ND
- R18: value R_US -> 47.5k; DigiKey (none) -> P47.5KCCT-ND
- R19: value R_US -> 1k; DigiKey (none) -> P1.0KDACT-ND
- R20: value R_US -> 26.1k; DigiKey (none) -> P26.1KCCT-ND
- U7: DigiKey (none) -> DRV103H-ND
Other:
- note added: "My injectors are working at 1.5A at 4V in DC operating.\nWhen applied 12V, the current raises from 0 to 2A in 1ms.\nDuty cycle set to 30%."
- moved on the sheet: C30, D14, D15, J10, R40, R41, R42, U15
