File: hardware/lin.sch (KiCad schematic (older format))
At the start: 7 parts, among them U12 MCP2003B

Commit message: rev 1
Parts:
- added R31: 33k, Resistors_SMD:R_0805, symbol Device:R
Connections:
- net labels removed: CS
- wire segments 14 -> 19
Other:
- moved on the sheet: R27
Changed lines of the file:
@@
 EESchema Schematic File Version 4
 LIBS:speeduino_mini-cache
-EELAYER 26 0
+EELAYER 29 0
 EELAYER END
 $Descr A4 11693 8268
 encoding utf-8
-Sheet 17 18
+Sheet 17 21
 Title ""
 Date ""
@@
 U 1 1 5C32548B
 P 6650 4900
-F 0 "U12" H 6400 4400 50  0000 L CNN
-F 1 "MCP2003B" H 6400 4300 50  0000 L CNN
+F 0 "U12" H 6350 4400 50  0000 L CNN
+F 1 "MCP2003B" H 6250 4300 50  0000 L CNN
 F 2 "Housings_SOIC:SOIC-8_3.9x4.9mm_Pitch1.27mm" H 6300 4650 50  0001 C CNN
-F 3 "" H 6300 4650 50  0001 C CNN
-F 4 "MCP2003BT-E/SNCT-ND" H 6600 4250 24  0000 C CNN "DIGIKEY"
+F 3 "http://www.microchip.com/mymicrochip/filehandler.aspx?ddocname=en584522" H 6300 4650 50  0001 C CNN
+F 4 "MCP2003BT-E/SNCT-ND" H 6250 4200 24  0000 L CNN "DIGIKEY"
 	1    6650 4900
 	1    0    0    -1
@@
 Wire Wire Line
 	6250 4800 5650 4800
-Wire Wire Line
-	6250 5000 6050 5000
-Text Label 6050 5000 0    50   ~ 0
-CS
 $Comp
 L power:+12V #PWR071
 U 1 1 5C32FFD3
-P 5000 3650
-F 0 "#PWR071" H 5000 3500 50  0001 C CNN
-F 1 "+12V" H 5015 3823 50  0000 C CNN
-F 2 "" H 5000 3650 50  0001 C CNN
-F 3 "" H 5000 3650 50  0001 C CNN
-	1    5000 3650
+P 4650 3650
+F 0 "#PWR071" H 4650 3500 50  0001 C CNN
+F 1 "+12V" H 4665 3823 50  0000 C CNN
+F 2 "" H 4650 3650 50  0001 C CNN
+F 3 "" H 4650 3650 50  0001 C CNN
+	1    4650 3650
 	1    0    0    -1
 $EndComp
@@
 L Device:R R27
 U 1 1 5C32FFF7
-P 5000 3800
-F 0 "R27" V 4750 3800 50  0000 C CNN
-F 1 "33k" V 4850 3800 50  0000 C CNN
-F 2 "Resistors_SMD:R_0805" V 4930 3800 50  0001 C CNN
-F 3 "~" H 5000 3800 50  0001 C CNN
-F 4 "311-33.0KCRCT-ND" V 4900 3800 24  0000 C CNN "DIGIKEY"
-	1    5000 3800
+P 4650 3800
+F 0 "R27" H 4580 3729 50  0000 R CNN
+F 1 "33k" H 4580 3820 50  0000 R CNN
+F 2 "Resistors_SMD:R_0805" V 4580 3800 50  0001 C CNN
+F 3 "~" H 4650 3800 50  0001 C CNN
+F 4 "311-33.0KCRCT-ND" H 4580 3891 24  0000 R CNN "DIGIKEY"
+	1    4650 3800
 	-1   0    0    1
 $EndComp
 Wire Wire Line
-	5000 3950 5000 5100
+	4650 3950 4650 5100
 $Comp
 L Device:R R28
 U 1 1 5C3325C7
 P 5850 3800
-F 0 "R28" H 5920 3846 50  0000 L CNN
-F 1 "4k7" H 5920 3755 50  0000 L CNN
+F 0 "R28" H 5920 3871 50  0000 L CNN
+F 1 "4k7" H 5920 3780 50  0000 L CNN
 F 2 "Resistors_SMD:R_0805" V 5780 3800 50  0001 C CNN
 F 3 "~" H 5850 3800 50  0001 C CNN
-F 4 "311-4.70KCRCT-ND" H 6050 3650 24  0000 C CNN "DIGIKEY"
+F 4 "311-4.70KCRCT-ND" H 5920 3709 24  0000 L CNN "DIGIKEY"
 	1    5850 3800
 	1    0    0    -1
@@
 U 1 1 5C336B62
 P 6850 3800
-F 0 "D6" V 6896 3721 50  0000 R CNN
-F 1 "D" V 6805 3721 50  0000 R CNN
+F 0 "D6" V 6921 3721 50  0000 R CNN
+F 1 "D" V 6830 3721 50  0000 R CNN
 F 2 "Diodes_SMD:D_SOD-123" H 6850 3800 50  0001 C CNN
 F 3 "~" H 6850 3800 50  0001 C CNN
-F 4 "1N4148W-FDICT-ND" V 6750 3600 24  0000 C CNN "DIGIKEY"
+F 4 "1N4148W-FDICT-ND" V 6759 3721 24  0000 R CNN "DIGIKEY"
 	1    6850 3800
 	0    -1   -1   0
@@
 U 1 1 5C33E7D7
 P 6600 4300
-F 0 "D5" H 6650 4050 50  0000 C CNN
-F 1 "D_Zener" H 6650 4150 50  0000 C CNN
+F 0 "D5" H 6600 4034 50  0000 C CNN
+F 1 "D_Zener" H 6600 4125 50  0000 C CNN
 F 2 "Diodes_SMD:D_SOD-323" H 6600 4300 50  0001 C CNN
 F 3 "~" H 6600 4300 50  0001 C CNN
-F 4 "RSB36VTE-17CT-ND" H 6650 4200 24  0000 C CNN "DIGIKEY"
+F 4 "RSB36VTE-17CT-ND" H 6600 4196 24  0000 C CNN "DIGIKEY"
 	1    6600 4300
 	-1   0    0    1
@@
 U 1 1 5C34BB03
 P 6850 4100
-F 0 "R30" H 6920 4146 50  0000 L CNN
-F 1 "47" H 6920 4055 50  0000 L CNN
+F 0 "R30" H 6920 4171 50  0000 L CNN
+F 1 "47" H 6920 4080 50  0000 L CNN
 F 2 "Resistors_SMD:R_0805" V 6780 4100 50  0001 C CNN
 F 3 "~" H 6850 4100 50  0001 C CNN
-F 4 "311-47ARCT-ND" H 7050 4000 24  0000 C CNN "DIGIKEY"
+F 4 "311-47ARCT-ND" H 6920 4009 24  0000 L CNN "DIGIKEY"
 	1    6850 4100
 	1    0    0    -1
@@
 L power:+5VD #PWR072
 U 1 1 5C79F658
-P 5850 3650
-F 0 "#PWR072" H 5850 3500 50  0001 C CNN
-F 1 "+5VD" H 5865 3823 50  0000 C CNN
-F 2 "" H 5850 3650 50  0001 C CNN
-F 3 "" H 5850 3650 50  0001 C CNN
-	1    5850 3650
+P 5850 3500
+F 0 "#PWR072" H 5850 3350 50  0001 C CNN
+F 1 "+5VD" H 5865 3673 50  0000 C CNN
+F 2 "" H 5850 3500 50  0001 C CNN
+F 3 "" H 5850 3500 50  0001 C CNN
+	1    5850 3500
 	1    0    0    -1
 $EndComp
@@
 	5650 4900 5850 4900
 Wire Wire Line
-	5000 5100 6250 5100
+	4650 5100 6250 5100
 NoConn ~ 6250 4600
+Wire Wire Line
+	5850 3500 5850 3550
+$Comp
+L Device:R R31
+U 1 1 5C879FFA
+P 5250 3800
+F 0 "R31" H 5180 3729 50  0000 R CNN
+F 1 "33k" H 5180 3820 50  0000 R CNN
+F 2 "Resistors_SMD:R_0805" V 5180 3800 50  0001 C CNN
+F 3 "~" H 5250 3800 50  0001 C CNN
+F 4 "311-33.0KCRCT-ND" H 5180 3891 24  0000 R CNN "DIGIKEY"
+	1    5250 3800
+	-1   0    0    1
+$EndComp
+Wire Wire Line
+	5850 3550 5250 3550
+Wire Wire Line
+	5250 3550 5250 3650
+Connection ~ 5850 3550
+Wire Wire Line
+	5850 3550 5850 3650
+Wire Wire Line
+	5250 3950 5250 5000
+Wire Wire Line
+	5250 5000 6250 5000
 $EndSCHEMATC

Commit message: Rev 2 work in progress
Parts:
- removed D5: D_Zener, Diodes_SMD:D_SOD-323, symbol Device:D_Zener
- removed D6: D, Diodes_SMD:D_SOD-123, symbol Device:D
- removed R30: 47, Resistors_SMD:R_0805, symbol Device:R
- added C46: 1uF, Capacitors_SMD:C_0805_HandSoldering, symbol Device:CP
- C43: footprint Capacitors_SMD:C_0805 -> Capacitors_SMD:C_0805_HandSoldering
- R27, R28, R31: footprint Resistors_SMD:R_0805 -> Resistors_SMD:R_0805_HandSoldering; symbol Device:R -> Device:R_US
Connections:
- net labels added: +5V
- net labels removed: +5VD
- wire segments 19 -> 22
Changed lines of the file:
@@
 $Descr A4 11693 8268
 encoding utf-8
-Sheet 17 21
+Sheet 21 23
 Title ""
 Date ""
@@
 Comment4 ""
 $EndDescr
-$Comp
-L speeduino_mini:MCP2003B U12
-U 1 1 5C32548B
-P 6650 4900
-F 0 "U12" H 6350 4400 50  0000 L CNN
-F 1 "MCP2003B" H 6250 4300 50  0000 L CNN
-F 2 "Housings_SOIC:SOIC-8_3.9x4.9mm_Pitch1.27mm" H 6300 4650 50  0001 C CNN
-F 3 "http://www.microchip.com/mymicrochip/filehandler.aspx?ddocname=en584522" H 6300 4650 50  0001 C CNN
-F 4 "MCP2003BT-E/SNCT-ND" H 6250 4200 24  0000 L CNN "DIGIKEY"
-	1    6650 4900
-	1    0    0    -1
-$EndComp
 $Bitmap
 Pos 2750 4300
@@
 EndData
 $EndBitmap
-Wire Wire Line
-	6250 4800 5650 4800
 $Comp
-L power:+12V #PWR071
-U 1 1 5C32FFD3
-P 4650 3650
-F 0 "#PWR071" H 4650 3500 50  0001 C CNN
-F 1 "+12V" H 4665 3823 50  0000 C CNN
-F 2 "" H 4650 3650 50  0001 C CNN
-F 3 "" H 4650 3650 50  0001 C CNN
-	1    4650 3650
+L power:GND #PWR?
+U 1 1 5D40EB58
+P 7100 3650
+AR Path="/5C7979FC/5D40EB58" Ref="#PWR?"  Part="1"
+AR Path="/5C610827/5D16F27C/5D40EB58" Ref="#PWR0126"  Part="1"
+F 0 "#PWR0126" H 7100 3400 50  0001 C CNN
+F 1 "GND" H 7105 3477 50  0000 C CNN
+F 2 "" H 7100 3650 50  0001 C CNN
+F 3 "" H 7100 3650 50  0001 C CNN
+	1    7100 3650
 	1    0    0    -1
 $EndComp
-$Comp
-L Device:R R27
-U 1 1 5C32FFF7
-P 4650 3800
-F 0 "R27" H 4580 3729 50  0000 R CNN
-F 1 "33k" H 4580 3820 50  0000 R CNN
-F 2 "Resistors_SMD:R_0805" V 4580 3800 50  0001 C CNN
-F 3 "~" H 4650 3800 50  0001 C CNN
-F 4 "311-33.0KCRCT-ND" H 4580 3891 24  0000 R CNN "DIGIKEY"
-	1    4650 3800
-	-1   0    0    1
-$EndComp
 Wire Wire Line
-	4650 3950 4650 5100
-$Comp
-L Device:R R28
-U 1 1 5C3325C7
-P 5850 3800
-F 0 "R28" H 5920 3871 50  0000 L CNN
-F 1 "4k7" H 5920 3780 50  0000 L CNN
-F 2 "Resistors_SMD:R_0805" V 5780 3800 50  0001 C CNN
-F 3 "~" H 5850 3800 50  0001 C CNN
-F 4 "311-4.70KCRCT-ND" H 5920 3709 24  0000 L CNN "DIGIKEY"
-	1    5850 3800
-	1    0    0    -1
-$EndComp
+	7100 3200 7100 3350
 Wire Wire Line
-	5850 4900 5850 3950
-$Comp
-L Device:D D6
-U 1 1 5C336B62
-P 6850 3800
-F 0 "D6" V 6921 3721 50  0000 R CNN
-F 1 "D" V 6830 3721 50  0000 R CNN
-F 2 "Diodes_SMD:D_SOD-123" H 6850 3800 50  0001 C CNN
-F 3 "~" H 6850 3800 50  0001 C CNN
-F 4 "1N4148W-FDICT-ND" V 6759 3721 24  0000 R CNN "DIGIKEY"
-	1    6850 3800
-	0    -1   -1   0
-$EndComp
-$Comp
-L power:+12V #PWR074
-U 1 1 5C336C79
-P 6850 3650
-F 0 "#PWR074" H 6850 3500 50  0001 C CNN
-F 1 "+12V" H 6865 3823 50  0000 C CNN
-F 2 "" H 6850 3650 50  0001 C CNN
-F 3 "" H 6850 3650 50  0001 C CNN
-	1    6850 3650
-	1    0    0    -1
-$EndComp
+	6850 3200 7100 3200
 $Comp
-L power:GND #PWR075
-U 1 1 5C338A7D
-P 6850 5750
-F 0 "#PWR075" H 6850 5500 50  0001 C CNN
-F 1 "GND" H 6855 5577 50  0000 C CNN
-F 2 "" H 6850 5750 50  0001 C CNN
-F 3 "" H 6850 5750 50  0001 C CNN
-	1    6850 5750
+L Device:CP C46
+U 1 1 5D40E4A4
+P 7100 3500
+F 0 "C46" H 7218 3546 50  0000 L CNN
+F 1 "1uF" H 7218 3455 50  0000 L CNN
+F 2 "Capacitors_SMD:C_0805_HandSoldering" H 7138 3350 50  0001 C CNN
+F 3 "~" H 7100 3500 50  0001 C CNN
+	1    7100 3500
 	1    0    0    -1
 $EndComp
 Wire Wire Line
-	6850 5750 6850 5450
+	6850 3200 6850 4350
+Text HLabel 5850 3500 1    50   Input ~ 0
++5V
+Connection ~ 6850 3200
 Wire Wire Line
-	7050 4900 7300 4900
-Connection ~ 7300 4900
+	4650 3200 6850 3200
 Wire Wire Line
-	7300 4900 7800 4900
+	4650 3650 4650 3200
+Wire Wire Line
+	6850 3100 6850 3200
+Text HLabel 6850 3100 1    50   Input ~ 0
++12V
+Wire Wire Line
+	5250 5000 6250 5000
+Wire Wire Line
+	5250 3950 5250 5000
+Wire Wire Line
+	5850 3550 5850 3650
+Connection ~ 5850 3550
+Wire Wire Line
+	5250 3550 5250 3650
+Wire Wire Line
+	5850 3550 5250 3550
 $Comp
-L Device:D_Zener D5
-U 1 1 5C33E7D7
-P 6600 4300
-F 0 "D5" H 6600 4034 50  0000 C CNN
-F 1 "D_Zener" H 6600 4125 50  0000 C CNN
-F 2 "Diodes_SMD:D_SOD-323" H 6600 4300 50  0001 C CNN
-F 3 "~" H 6600 4300 50  0001 C CNN
-F 4 "RSB36VTE-17CT-ND" H 6600 4196 24  0000 C CNN "DIGIKEY"
-	1    6600 4300
+L Device:R_US R31
+U 1 1 5C879FFA
+P 5250 3800
+AR Path="/5C7979FC/5C879FFA" Ref="R31"  Part="1"
+AR Path="/5C610827/5D16F27C/5C879FFA" Ref="R28"  Part="1"
+F 0 "R28" H 5180 3729 50  0000 R CNN
+F 1 "33k" H 5180 3820 50  0000 R CNN
+F 2 "Resistors_SMD:R_0805_HandSoldering" V 5180 3800 50  0001 C CNN
+F 3 "~" H 5250 3800 50  0001 C CNN
+F 4 "311-33.0KCRCT-ND" H 5180 3891 24  0000 R CNN "DIGIKEY"
+	1    5250 3800
 	-1   0    0    1
 $EndComp
-$Comp
-L power:GND #PWR073
-U 1 1 5C33E861
-P 6450 4300
-F 0 "#PWR073" H 6450 4050 50  0001 C CNN
-F 1 "GND" V 6455 4172 50  0000 R CNN
-F 2 "" H 6450 4300 50  0001 C CNN
-F 3 "" H 6450 4300 50  0001 C CNN
-	1    6450 4300
-	0    1    1    0
-$EndComp
 Wire Wire Line
-	6750 4300 6850 4300
+	5850 3500 5850 3550
+NoConn ~ 6250 4600
 Wire Wire Line
-	6850 4300 6850 4250
+	4650 5100 6250 5100
 Wire Wire Line
-	6850 4350 6850 4300
-Connection ~ 6850 4300
+	5650 4900 5850 4900
+Wire Wire Line
+	5850 4900 6250 4900
+Connection ~ 5850 4900
+Text HLabel 7800 4900 2    50   BiDi ~ 0
+LIN
+Text HLabel 5650 4900 0    50   Output ~ 0
+RXD
+Text HLabel 5650 4800 0    50   Input ~ 0
+TXD
+Wire Wire Line
+	7300 5450 7300 4900
 $Comp
-L Device:R R30
-U 1 1 5C34BB03
-P 6850 4100
-F 0 "R30" H 6920 4171 50  0000 L CNN
-F 1 "47" H 6920 4080 50  0000 L CNN
-F 2 "Resistors_SMD:R_0805" V 6780 4100 50  0001 C CNN
-F 3 "~" H 6850 4100 50  0001 C CNN
-F 4 "311-47ARCT-ND" H 6920 4009 24  0000 L CNN "DIGIKEY"
-	1    6850 4100
+L power:GND #PWR076
+U 1 1 5C35A885
+P 7300 5750
+AR Path="/5C7979FC/5C35A885" Ref="#PWR076"  Part="1"
+AR Path="/5C610827/5D16F27C/5C35A885" Ref="#PWR011"  Part="1"
+F 0 "#PWR011" H 7300 5500 50  0001 C CNN
+F 1 "GND" H 7305 5577 50  0000 C CNN
+F 2 "" H 7300 5750 50  0001 C CNN
+F 3 "" H 7300 5750 50  0001 C CNN
+	1    7300 5750
 	1    0    0    -1
 $EndComp
@@
 U 1 1 5C35A5FC
 P 7300 5600
-F 0 "C43" H 7415 5671 50  0000 L CNN
+AR Path="/5C7979FC/5C35A5FC" Ref="C43"  Part="1"
+AR Path="/5C610827/5D16F27C/5C35A5FC" Ref="C6"  Part="1"
+F 0 "C6" H 7415 5671 50  0000 L CNN
 F 1 "220pF" H 7415 5580 50  0000 L CNN
-F 2 "Capacitors_SMD:C_0805" H 7338 5450 50  0001 C CNN
+F 2 "Capacitors_SMD:C_0805_HandSoldering" H 7338 5450 50  0001 C CNN
 F 3 "~" H 7300 5600 50  0001 C CNN
 F 4 "1276-2617-1-ND" H 7415 5509 24  0000 L CNN "DIGIKEY"
@@
 	1    0    0    -1
 $EndComp
+Wire Wire Line
+	7300 4900 7800 4900
+Connection ~ 7300 4900
+Wire Wire Line
+	7050 4900 7300 4900
+Wire Wire Line
+	6850 5750 6850 5450
 $Comp
-L power:GND #PWR076
-U 1 1 5C35A885
-P 7300 5750
-F 0 "#PWR076" H 7300 5500 50  0001 C CNN
-F 1 "GND" H 7305 5577 50  0000 C CNN
-F 2 "" H 7300 5750 50  0001 C CNN
-F 3 "" H 7300 5750 50  0001 C CNN
-	1    7300 5750
+L power:GND #PWR075
+U 1 1 5C338A7D
+P 6850 5750
+AR Path="/5C7979FC/5C338A7D" Ref="#PWR075"  Part="1"
+AR Path="/5C610827/5D16F27C/5C338A7D" Ref="#PWR08"  Part="1"
+F 0 "#PWR08" H 6850 5500 50  0001 C CNN
+F 1 "GND" H 6855 5577 50  0000 C CNN
+F 2 "" H 6850 5750 50  0001 C CNN
+F 3 "" H 6850 5750 50  0001 C CNN
+	1    6850 5750
 	1    0    0    -1
 $EndComp
 Wire Wire Line
-	7300 5450 7300 4900
-Text HLabel 5650 4800 0    50   Input ~ 0
-TXD
-Text HLabel 5650 4900 0    50   Output ~ 0
-RXD
+	5850 4900 5850 3950
 $Comp
-L power:+5VD #PWR072
-U 1 1 5C79F658
-P 5850 3500
-F 0 "#PWR072" H 5850 3350 50  0001 C CNN
-F 1 "+5VD" H 5865 3673 50  0000 C CNN
-F 2 "" H 5850 3500 50  0001 C CNN
-F 3 "" H 5850 3500 50  0001 C CNN
-	1    5850 3500
+L Device:R_US R28
+U 1 1 5C3325C7
+P 5850 3800
+AR Path="/5C7979FC/5C3325C7" Ref="R28"  Part="1"
+AR Path="/5C610827/5D16F27C/5C3325C7" Ref="R30"  Part="1"
+F 0 "R30" H 5920 3871 50  0000 L CNN
+F 1 "4k7" H 5920 3780 50  0000 L CNN
+F 2 "Resistors_SMD:R_0805_HandSoldering" V 5780 3800 50  0001 C CNN
+F 3 "~" H 5850 3800 50  0001 C CNN
+F 4 "311-4.70KCRCT-ND" H 5920 3709 24  0000 L CNN "DIGIKEY"
+	1    5850 3800
 	1    0    0    -1
 $EndComp
-Text HLabel 7800 4900 2    50   BiDi ~ 0
-LIN
-Connection ~ 5850 4900
-Wire Wire Line
-	5850 4900 6250 4900
-Wire Wire Line
-	5650 4900 5850 4900
-Wire Wire Line
-	4650 5100 6250 5100
-NoConn ~ 6250 4600
 Wire Wire Line
-	5850 3500 5850 3550
+	4650 3950 4650 5100
 $Comp
-L Device:R R31
-U 1 1 5C879FFA
-P 5250 3800
-F 0 "R31" H 5180 3729 50  0000 R CNN
-F 1 "33k" H 5180 3820 50  0000 R CNN
-F 2 "Resistors_SMD:R_0805" V 5180 3800 50  0001 C CNN
-F 3 "~" H 5250 3800 50  0001 C CNN
-F 4 "311-33.0KCRCT-ND" H 5180 3891 24  0000 R CNN "DIGIKEY"
-	1    5250 3800
+L Device:R_US R27
+U 1 1 5C32FFF7
+P 4650 3800
+AR Path="/5C7979FC/5C32FFF7" Ref="R27"  Part="1"
+AR Path="/5C610827/5D16F27C/5C32FFF7" Ref="R27"  Part="1"
+F 0 "R27" H 4580 3729 50  0000 R CNN
+F 1 "33k" H 4580 3820 50  0000 R CNN
+F 2 "Resistors_SMD:R_0805_HandSoldering" V 4580 3800 50  0001 C CNN
+F 3 "~" H 4650 3800 50  0001 C CNN
+F 4 "311-33.0KCRCT-ND" H 4580 3891 24  0000 R CNN "DIGIKEY"
+	1    4650 3800
 	-1   0    0    1
 $EndComp
 Wire Wire Line
-	5850 3550 5250 3550
-Wire Wire Line
-	5250 3550 5250 3650
-Connection ~ 5850 3550
-Wire Wire Line
-	5850 3550 5850 3650
-Wire Wire Line
-	5250 3950 5250 5000
-Wire Wire Line
-	5250 5000 6250 5000
+	6250 4800 5650 4800
+$Comp
+L speeduino_mini:MCP2003B U12
+U 1 1 5C32548B
+P 6650 4900
+AR Path="/5C7979FC/5C32548B" Ref="U12"  Part="1"
+AR Path="/5C610827/5D16F27C/5C32548B" Ref="U8"  Part="1"
+F 0 "U8" H 6350 4400 50  0000 L CNN
+F 1 "MCP2003B" H 6250 4300 50  0000 L CNN
+F 2 "Housings_SOIC:SOIC-8_3.9x4.9mm_Pitch1.27mm" H 6300 4650 50  0001 C CNN
+F 3 "http://www.microchip.com/mymicrochip/filehandler.aspx?ddocname=en584522" H 6300 4650 50  0001 C CNN
+F 4 "MCP2003BT-E/SNCT-ND" H 6250 4200 24  0000 L CNN "DIGIKEY"
+	1    6650 4900
+	1    0    0    -1
+$EndComp
 $EndSCHEMATC

Commit message: rev 2 sent to fab
Parts:
- C43: value 220pF -> 0.22nF 200V; DIGIKEY 1276-2617-1-ND -> (none); DigiKey (none) -> 1276-2617-1-ND
- C46: value 1uF -> 1uF 35V; DigiKey (none) -> 1276-6517-1-ND
- R27, R31: DIGIKEY 311-33.0KCRCT-ND -> (none); DigiKey (none) -> 311-33.0KCRCT-ND
- R28: DIGIKEY 311-4.70KCRCT-ND -> (none); DigiKey (none) -> 311-4.70KCRCT-ND
- U12: DIGIKEY MCP2003BT-E/SNCT-ND -> (none); DigiKey (none) -> MCP2003BT-E/SNCT-ND
Changed lines of the file:
@@
 $Descr A4 11693 8268
 encoding utf-8
-Sheet 21 22
+Sheet 20 22
 Title ""
 Date ""
@@
 P 7100 3500
 F 0 "C46" H 7218 3546 50  0000 L CNN
-F 1 "1uF" H 7218 3455 50  0000 L CNN
+F 1 "1uF 35V" H 7218 3455 50  0000 L CNN
 F 2 "Capacitors_SMD:C_0805_HandSoldering" H 7138 3350 50  0001 C CNN
 F 3 "~" H 7100 3500 50  0001 C CNN
+F 4 "1276-6517-1-ND" H 0   0   50  0001 C CNN "DigiKey"
 	1    7100 3500
 	1    0    0    -1
@@
 F 2 "Resistors_SMD:R_0805_HandSoldering" V 5180 3800 50  0001 C CNN
 F 3 "~" H 5250 3800 50  0001 C CNN
-F 4 "311-33.0KCRCT-ND" H 5180 3891 24  0000 R CNN "DIGIKEY"
+F 4 "311-33.0KCRCT-ND" H 0   0   50  0001 C CNN "DigiKey"
 	1    5250 3800
 	-1   0    0    1
@@
 AR Path="/5C610827/5D16F27C/5C35A5FC" Ref="C6"  Part="1"
 F 0 "C6" H 7415 5671 50  0000 L CNN
-F 1 "220pF" H 7415 5580 50  0000 L CNN
+F 1 "0.22nF 200V" H 7415 5580 50  0000 L CNN
 F 2 "Capacitors_SMD:C_0805_HandSoldering" H 7338 5450 50  0001 C CNN
 F 3 "~" H 7300 5600 50  0001 C CNN
-F 4 "1276-2617-1-ND" H 7415 5509 24  0000 L CNN "DIGIKEY"
+F 4 "1276-2617-1-ND" H 0   0   50  0001 C CNN "DigiKey"
 	1    7300 5600
 	1    0    0    -1
@@
 F 2 "Resistors_SMD:R_0805_HandSoldering" V 5780 3800 50  0001 C CNN
 F 3 "~" H 5850 3800 50  0001 C CNN
-F 4 "311-4.70KCRCT-ND" H 5920 3709 24  0000 L CNN "DIGIKEY"
+F 4 "311-4.70KCRCT-ND" H 0   0   50  0001 C CNN "DigiKey"
 	1    5850 3800
 	1    0    0    -1
@@
 F 2 "Resistors_SMD:R_0805_HandSoldering" V 4580 3800 50  0001 C CNN
 F 3 "~" H 4650 3800 50  0001 C CNN
-F 4 "311-33.0KCRCT-ND" H 4580 3891 24  0000 R CNN "DIGIKEY"
+F 4 "311-33.0KCRCT-ND" H 0   0   50  0001 C CNN "DigiKey"
 	1    4650 3800
 	-1   0    0    1
@@
 F 2 "Housings_SOIC:SOIC-8_3.9x4.9mm_Pitch1.27mm" H 6300 4650 50  0001 C CNN
 F 3 "http://www.microchip.com/mymicrochip/filehandler.aspx?ddocname=en584522" H 6300 4650 50  0001 C CNN
-F 4 "MCP2003BT-E/SNCT-ND" H 6250 4200 24  0000 L CNN "DIGIKEY"
+F 4 "MCP2003BT-E/SNCT-ND" H 0   0   50  0001 C CNN "DigiKey"
 	1    6650 4900
 	1    0    0    -1
