File: hardware/mcu.sch (KiCad schematic (older format))
At the start: 14 parts, among them U1 TPD4E001-Q1, U2 TPD4E001-Q1, U3 ATmega2561-16AU, U6 TPD2E001-SOT-5, Y1 CSTCE16M0V53-R0

Commit message: work in progress - components ordered
Parts:
- removed ICSP1: ICSP, Pin_Headers:Pin_Header_Straight_2x03_Pitch2.54mm_SMD, symbol Connector_Generic:Conn_02x03_Odd_Even
- added C16, C22, C36, C6: 100nF, Capacitors_SMD:C_0805, symbol Device:C
- added L2: 10uH, Inductors_SMD:L_0805, symbol Device:L
Connections:
- net labels added: +5VD, PB7
- net labels removed: +5V, +5VA, MISO, MOSI, OC0A_0C1C
- wire segments 108 -> 117

Commit message: rev 1
Parts:
- removed U6: TPD2E001-SOT-5, TO_SOT_Packages_SMD:SOT-553, symbol speeduino_mini:TPD2E001-SOT-5
- added U6: TPD4E001-Q1, TO_SOT_Packages_SMD:SOT-23-6, symbol speeduino_mini:TPD4E001-Q1
Connections:
- net labels added: PE7
- net labels removed: OC2A
- wire segments 117 -> 116
- no-connect marks 0 -> 2
Other:
- moved on the sheet: C5
Changed lines of the file:
@@
 EESchema Schematic File Version 4
 LIBS:speeduino_mini-cache
-EELAYER 26 0
+EELAYER 29 0
 EELAYER END
 $Descr A4 11693 8268
 encoding utf-8
-Sheet 2 18
+Sheet 2 21
 Title ""
 Date ""
@@
 Text HLabel 750  4900 0    50   Input ~ 0
 A1
-Wire Wire Line
-	5700 5200 4450 5200
 Text HLabel 750  5200 0    50   Input ~ 0
 A4
@@
 Text HLabel 750  5400 0    50   Input ~ 0
 A6
-Wire Wire Line
-	5700 5300 3350 5300
-Wire Wire Line
-	750  5400 3250 5400
 $Comp
 L Device:Crystal_GND2 Y1
@@
 Text HLabel 750  5500 0    50   Input ~ 0
 A7
-Wire Wire Line
-	750  5500 4350 5500
 $Comp
 L speeduino_mini:TPD4E001-Q1 U1
@@
 	1550 7050 2300 7050
 Wire Wire Line
-	4350 6450 4350 5500
-Connection ~ 4350 5500
-Wire Wire Line
-	4350 5500 5700 5500
-Wire Wire Line
 	3350 6650 3250 6650
 Wire Wire Line
-	3250 6650 3250 5400
-Connection ~ 3250 5400
-Wire Wire Line
-	3250 5400 5700 5400
-Wire Wire Line
-	3350 6450 3350 5300
-Connection ~ 3350 5300
-Wire Wire Line
-	3350 5300 750  5300
-Wire Wire Line
 	4350 6650 4450 6650
-Wire Wire Line
-	4450 6650 4450 5200
-Connection ~ 4450 5200
-Wire Wire Line
-	4450 5200 750  5200
 Wire Wire Line
 	1050 6650 950  6650
@@
 	3850 6000 3850 5900
 Connection ~ 3850 6000
-Wire Wire Line
-	6900 5800 7300 5800
 Text HLabel 9650 5800 2    50   Input ~ 0
 INT1
-Wire Wire Line
-	6900 5700 7200 5700
 Wire Wire Line
 	6900 6000 9650 6000
@@
 TXD1
 $Comp
-L speeduino_mini:TPD2E001-SOT-5 U6
-U 1 1 5C87473B
-P 7800 4950
-F 0 "U6" H 8030 5041 50  0000 L CNN
-F 1 "TPD2E001-SOT-5" H 8030 4950 50  0000 L CNN
-F 2 "TO_SOT_Packages_SMD:SOT-553" H 8050 4850 50  0001 L CNN
-F 3 "http://www.ti.com/lit/ds/symlink/tpd2e001.pdf" H 8050 4750 50  0001 L CNN
-F 4 "296-21883-1-ND" H 8030 4859 50  0000 L CNN "DIGIKEY"
-	1    7800 4950
-	1    0    0    -1
-$EndComp
-$Comp
 L Device:C C5
 U 1 1 5C87485F
-P 8850 4950
-F 0 "C5" H 8965 5041 50  0000 L CNN
-F 1 "100nF" H 8965 4950 50  0000 L CNN
-F 2 "Capacitors_SMD:C_0805" H 8888 4800 50  0001 C CNN
-F 3 "~" H 8850 4950 50  0001 C CNN
-F 4 "478-6048-1-ND" H 8965 4859 50  0000 L CNN "DIGIKEY"
-	1    8850 4950
-	1    0    0    -1
-$EndComp
-Wire Wire Line
-	7800 4650 7800 4600
-Wire Wire Line
-	8850 4600 8850 4800
-Wire Wire Line
-	7800 5250 7800 5300
-Wire Wire Line
-	7800 5300 8350 5300
-Wire Wire Line
-	8850 5300 8850 5100
-$Comp
-L power:GND #PWR016
-U 1 1 5C8837B8
-P 8350 5300
-F 0 "#PWR016" H 8350 5050 50  0001 C CNN
-F 1 "GND" H 8355 5127 50  0000 C CNN
-F 2 "" H 8350 5300 50  0001 C CNN
-F 3 "" H 8350 5300 50  0001 C CNN
-	1    8350 5300
-	1    0    0    -1
-$EndComp
-Connection ~ 8350 5300
-Wire Wire Line
-	8350 5300 8850 5300
-Wire Wire Line
-	7500 4850 7200 4850
-Wire Wire Line
-	7200 4850 7200 5700
-Connection ~ 7200 5700
-Wire Wire Line
-	7200 5700 9650 5700
-Wire Wire Line
-	7500 5050 7300 5050
-Wire Wire Line
-	7300 5050 7300 5800
-Connection ~ 7300 5800
-Wire Wire Line
-	7300 5800 9650 5800
+P 9500 4600
+F 0 "C5" H 9615 4691 50  0000 L CNN
+F 1 "100nF" H 9615 4600 50  0000 L CNN
+F 2 "Capacitors_SMD:C_0805" H 9538 4450 50  0001 C CNN
+F 3 "~" H 9500 4600 50  0001 C CNN
+F 4 "478-6048-1-ND" H 9615 4509 50  0000 L CNN "DIGIKEY"
+	1    9500 4600
+	1    0    0    -1
+$EndComp
 Text HLabel 7100 4600 2    50   Output ~ 0
 PB7
@@
 Text HLabel 7100 4400 2    50   Output ~ 0
 OC1A
-Text HLabel 7100 4300 2    50   Output ~ 0
-OC2A
-Wire Wire Line
-	6900 4300 7100 4300
 Text HLabel 5550 6200 0    50   Output ~ 0
 OC3C
@@
 Text HLabel 7100 3000 2    50   Output ~ 0
 PA0
-Wire Wire Line
-	2150 4800 750  4800
-Wire Wire Line
-	5700 4800 2150 4800
-Connection ~ 2150 4800
-Wire Wire Line
-	2150 6650 2150 4800
-Wire Wire Line
-	1050 4900 750  4900
-Wire Wire Line
-	5700 4900 1050 4900
-Connection ~ 1050 4900
-Wire Wire Line
-	1050 6450 1050 4900
-Wire Wire Line
-	950  5000 750  5000
-Wire Wire Line
-	5700 5000 950  5000
-Connection ~ 950  5000
-Wire Wire Line
-	950  5000 950  6650
-Wire Wire Line
-	2050 5100 750  5100
-Wire Wire Line
-	5700 5100 2050 5100
-Connection ~ 2050 5100
-Wire Wire Line
-	2050 6450 2050 5100
 $Comp
 L Device:C C6
@@
 L power:+5VD #PWR015
 U 1 1 5C789D76
-P 8350 4600
-F 0 "#PWR015" H 8350 4450 50  0001 C CNN
-F 1 "+5VD" H 8365 4773 50  0000 C CNN
-F 2 "" H 8350 4600 50  0001 C CNN
-F 3 "" H 8350 4600 50  0001 C CNN
-	1    8350 4600
-	1    0    0    -1
-$EndComp
-Wire Wire Line
-	7800 4600 8350 4600
-Connection ~ 8350 4600
-Wire Wire Line
-	8350 4600 8850 4600
+P 8750 4000
+F 0 "#PWR015" H 8750 3850 50  0001 C CNN
+F 1 "+5VD" H 8765 4173 50  0000 C CNN
+F 2 "" H 8750 4000 50  0001 C CNN
+F 3 "" H 8750 4000 50  0001 C CNN
+	1    8750 4000
+	1    0    0    -1
+$EndComp
 Text HLabel 7100 4000 2    50   Input ~ 0
 SCK
@@
 	5300 3000 5400 3000
 Connection ~ 5400 3000
+$Comp
+L speeduino_mini:TPD4E001-Q1 U6
+U 1 1 5C8FE76E
+P 8750 4600
+F 0 "U6" H 8750 5321 50  0000 C CNN
+F 1 "TPD4E001-Q1" H 8750 5230 50  0000 C CNN
+F 2 "TO_SOT_Packages_SMD:SOT-23-6" H 8550 4000 50  0001 C CNN
+F 3 "http://www.ti.com/lit/ds/symlink/tpd4e001-q1.pdf" H 8750 4600 50  0001 C CNN
+F 4 "296-39344-1-ND" H 8750 5139 50  0000 C CNN "DIGIKEY"
+	1    8750 4600
+	1    0    0    -1
+$EndComp
+$Comp
+L power:GND #PWR016
+U 1 1 5C916728
+P 8750 5450
+F 0 "#PWR016" H 8750 5200 50  0001 C CNN
+F 1 "GND" H 8755 5277 50  0000 C CNN
+F 2 "" H 8750 5450 50  0001 C CNN
+F 3 "" H 8750 5450 50  0001 C CNN
+	1    8750 5450
+	1    0    0    -1
+$EndComp
+Wire Wire Line
+	8750 5100 8750 5150
+Wire Wire Line
+	8750 4000 8750 4150
+NoConn ~ 9250 4500
+NoConn ~ 9250 4700
+Wire Wire Line
+	9500 4750 9500 5150
+Wire Wire Line
+	9500 5150 8750 5150
+Connection ~ 8750 5150
+Wire Wire Line
+	8750 5150 8750 5450
+Wire Wire Line
+	9500 4450 9500 4150
+Wire Wire Line
+	9500 4150 8750 4150
+Connection ~ 8750 4150
+Wire Wire Line
+	6900 5700 7950 5700
+Wire Wire Line
+	8250 4700 7950 4700
+Wire Wire Line
+	8250 4500 8050 4500
+Wire Wire Line
+	6900 5800 8050 5800
+Wire Wire Line
+	7950 4700 7950 5700
+Connection ~ 7950 5700
+Wire Wire Line
+	7950 5700 9650 5700
+Wire Wire Line
+	8050 4500 8050 5800
+Connection ~ 8050 5800
+Wire Wire Line
+	8050 5800 9650 5800
+Text HLabel 5550 6400 0    50   Output ~ 0
+PE7
+Wire Wire Line
+	5700 6400 5550 6400
+Wire Wire Line
+	750  4800 950  4800
+Wire Wire Line
+	750  5100 2050 5100
+Wire Wire Line
+	750  4900 1050 4900
+Wire Wire Line
+	750  5000 2150 5000
+Wire Wire Line
+	750  5500 3350 5500
+Wire Wire Line
+	750  5300 4350 5300
+Wire Wire Line
+	750  5400 3250 5400
+Wire Wire Line
+	950  6650 950  4800
+Connection ~ 950  4800
+Wire Wire Line
+	950  4800 5700 4800
+Wire Wire Line
+	1050 6450 1050 4900
+Connection ~ 1050 4900
+Wire Wire Line
+	1050 4900 5700 4900
+Wire Wire Line
+	2150 6650 2150 5000
+Connection ~ 2150 5000
+Wire Wire Line
+	2150 5000 5700 5000
+Wire Wire Line
+	2050 6450 2050 5100
+Connection ~ 2050 5100
+Wire Wire Line
+	2050 5100 5700 5100
+Wire Wire Line
+	750  5200 4450 5200
+Wire Wire Line
+	4450 6650 4450 5200
+Connection ~ 4450 5200
+Wire Wire Line
+	4450 5200 5700 5200
+Wire Wire Line
+	4350 6450 4350 5300
+Connection ~ 4350 5300
+Wire Wire Line
+	4350 5300 5700 5300
+Wire Wire Line
+	3250 6650 3250 5400
+Connection ~ 3250 5400
+Wire Wire Line
+	3250 5400 5700 5400
+Wire Wire Line
+	3350 6450 3350 5500
+Connection ~ 3350 5500
+Wire Wire Line
+	3350 5500 5700 5500
 $EndSCHEMATC

Commit message: Rev 2 work in progress
Parts:
- removed C16, C22, C36, C6: 100nF, Capacitors_SMD:C_0805, symbol Device:C
- removed L2: 10uH, Inductors_SMD:L_0805, symbol Device:L
- added JP41, JP42, JP43, JP44: Jumper, Pin_Headers:Pin_Header_Straight_1x02_Pitch2.54mm, symbol Device:Jumper
- C1, C2, C3, C4, C5: footprint Capacitors_SMD:C_0805 -> Capacitors_SMD:C_0805_HandSoldering
- R1, RN5A1: footprint Resistors_SMD:R_0805 -> Resistors_SMD:R_0805_HandSoldering
Connections:
- net labels added: +12V, LIN, VCC
- net labels removed: +5VD, OC0B, PE7, RXD1, TXD1
- wire segments 116 -> 103
- no-connect marks 2 -> 20
Other:
- note added: "EFUSE=0xFC (BODLEVEL=100 for 16MHz operation)\nHFUSE=0x99 (default)\nLFUSE=0xFF (for 16MHz operation, same as Arduino Mega)"
- note added: "ONLY 16 bits timers are 1,3,4,5"

Commit message: rev 2 work in progress
Connections:
- wire segments 103 -> 104
Changed lines of the file:
@@
 $Descr A4 11693 8268
 encoding utf-8
-Sheet 20 23
+Sheet 19 22
 Title ""
 Date ""
@@
 $EndSheet
 $Sheet
-S 5050 1300 750  350
+S 4450 1300 750  350
 U 5D1A080F
 F0 "ATMEGA regulator" 50
 F1 "atmega_regulator.sch" 50
-F2 "+12V" I L 5050 1400 50
-F3 "VCC" O R 5800 1550 50
-F4 "AVCC" O R 5800 1400 50
+F2 "+12V" I L 4450 1400 50
+F3 "VCC" O R 5200 1550 50
+F4 "AVCC" O R 5200 1400 50
 $EndSheet
 Wire Wire Line
-	5800 1550 6300 1550
-Wire Wire Line
 	6300 1550 6300 2700
-Wire Wire Line
-	5800 1400 6400 1400
 Wire Wire Line
 	6400 1400 6400 2700
@@
 Text Label 11850 6300 2    50   ~ 0
 VCC
-Text HLabel 4550 1400 0    50   Input ~ 0
+Text HLabel 3350 1400 0    50   Input ~ 0
 +12V
-Wire Wire Line
-	4550 1400 5050 1400
-Text Label 4700 1400 0    50   ~ 0
+Text Label 3500 1400 0    50   ~ 0
 +12V
 Text Label 11850 6700 2    50   ~ 0
@@
 Wire Wire Line
 	11450 6700 11850 6700
+Wire Wire Line
+	5200 1550 6300 1550
+Wire Wire Line
+	5200 1400 6400 1400
+Wire Wire Line
+	3350 1400 4450 1400
+Text HLabel 6650 1550 2    50   Output ~ 0
+VCC
+Wire Wire Line
+	6300 1550 6650 1550
+Connection ~ 6300 1550
 $EndSCHEMATC

Commit message: hardware rev2 - layout complete
Parts:
- removed C1, C3, C5: 100nF, Capacitors_SMD:C_0805_HandSoldering, symbol Device:C
- removed JP44: Jumper, Pin_Headers:Pin_Header_Straight_1x02_Pitch2.54mm, symbol Device:Jumper
- removed U1, U2, U6: TPD4E001-Q1, TO_SOT_Packages_SMD:SOT-23-6, symbol speeduino_mini:TPD4E001-Q1
- added D20, D21, D22, D23, D24, D25, D26, D6, D7: NUP1301,215, TO_SOT_Packages_SMD:SOT-23, symbol Device:D_Schottky_x2_Serial_AKC
- added JP39, JP40, JP49, JP50, JP51, JP52, JP53, JP54, JP55: Jumper, Pin_Headers:Pin_Header_Straight_1x02_Pitch2.54mm, symbol Device:Jumper
Connections:
- net labels added: PA1
- net labels removed: INT1, PB7
- wire segments 104 -> 69
- no-connect marks 20 -> 34
Other:
- moved on the sheet: C4

Commit message: rev 2 sent to fab
Parts:
- added J15: Conn_01x08_Female, Pin_Headers:Pin_Header_Straight_1x08_Pitch2.54mm, symbol Connector:Conn_01x08_Female
- C2: value 4.7nF -> 4.7nF 100V; DIGIKEY 478-9887-1-ND -> (none); DigiKey (none) -> 478-9887-1-ND
- C4: value 100nF -> 0.1uF 50V; DIGIKEY 478-6048-1-ND -> (none); DigiKey (none) -> 478-6048-1-ND
- D1: DIGIKEY MSS1P3L-M3/89AGICT-ND -> (none); DigiKey (none) -> MSS1P3L-M3/89AGICT-ND
- JP39, JP40, JP41, JP42, JP43, JP49, JP50, JP51, JP52, JP53, JP54, JP55: DigiKey (none) -> S9337-ND
- R1: DIGIKEY 311-1.00MCRCT-ND -> (none); DigiKey (none) -> 311-1.00MCRCT-ND
- RN5A1: DIGIKEY 311-10.0KCRCT-ND -> (none); DigiKey (none) -> 311-10.0KCRCT-ND
- U3: DIGIKEY ATMEGA2561-16AURCT-ND -> (none); DigiKey (none) -> ATMEGA2561-16AURCT-ND
- Y1: DIGIKEY 490-17948-1-ND -> (none); DigiKey (none) -> 490-17948-1-ND
Connections:
- net at U3.35 (PC0): now also J15.1 (Pin_1)
- net at U3.36 (PC1): now also J15.2 (Pin_2)
- net at U3.37 (PC2): now also J15.3 (Pin_3)
- net at U3.38 (PC3): now also J15.4 (Pin_4)
- net at U3.39 (PC4): now also J15.5 (Pin_5)
- net at U3.40 (PC5): now also J15.6 (Pin_6)
- net at U3.41 (PC6): now also J15.7 (Pin_7)
- net at U3.42 (PC7): now also J15.8 (Pin_8)
- no-connect marks 34 -> 26
Other:
- moved on the sheet: JP55
Changed lines of the file:
@@
 F 2 "Housings_QFP:TQFP-64_14x14mm_Pitch0.8mm" H 6300 4700 50  0001 C CIN
 F 3 "http://www.microchip.com/mymicrochip/filehandler.aspx?ddocname=en589901" H 6300 4700 50  0001 C CNN
-F 4 "ATMEGA2561-16AURCT-ND" H 6300 2200 50  0000 C CNN "DIGIKEY"
+F 4 "ATMEGA2561-16AURCT-ND" H 0   0   50  0001 C CNN "DigiKey"
 	1    6300 4700
 	1    0    0    -1
@@
 F 2 "Speeduino Mini:Resonator_SMD_Murata-3pin_3.2x1.3mm" H 4400 3300 50  0001 C CNN
 F 3 "https://www.murata.com/en/products/productdata/8801162231838/SPEC-CSTNE16M0V530000R0.pdf" H 4400 3300 50  0001 C CNN
-F 4 "490-17948-1-ND" V 4491 3431 50  0000 L CNN "DIGIKEY"
+F 4 "490-17948-1-ND" H 0   0   50  0001 C CNN "DigiKey"
 	1    4400 3300
 	0    1    1    0
@@
 F 2 "Resistors_SMD:R_0805_HandSoldering" V 3130 3300 50  0001 C CNN
 F 3 "~" H 3200 3300 50  0001 C CNN
-F 4 "311-1.00MCRCT-ND" H 3270 3209 50  0000 L CNN "DIGIKEY"
+F 4 "311-1.00MCRCT-ND" H 0   0   50  0001 C CNN "DigiKey"
 	1    3200 3300
 	1    0    0    -1
@@
 P 4600 2500
 F 0 "C2" H 4715 2591 50  0000 L CNN
-F 1 "4.7nF" H 4715 2500 50  0000 L CNN
+F 1 "4.7nF 100V" H 4715 2500 50  0000 L CNN
 F 2 "Capacitors_SMD:C_0805_HandSoldering" H 4638 2350 50  0001 C CNN
 F 3 "~" H 4600 2500 50  0001 C CNN
-F 4 "478-9887-1-ND" H 4715 2409 50  0000 L CNN "DIGIKEY"
+F 4 "478-9887-1-ND" H 0   0   50  0001 C CNN "DigiKey"
 	1    4600 2500
 	1    0    0    -1
@@
 F 2 "Speeduino Mini:MicroSMP" H 4600 2200 50  0001 C CNN
 F 3 "http://www.vishay.com/docs/89020/mss1p3l.pdf" H 4600 2200 50  0001 C CNN
-F 4 "MSS1P3L-M3/89AGICT-ND" V 4691 2279 50  0000 L CNN "DIGIKEY"
+F 4 "MSS1P3L-M3/89AGICT-ND" H 0   0   50  0001 C CNN "DigiKey"
 	1    4600 2200
 	0    1    1    0
@@
 F 2 "Resistors_SMD:R_0805_HandSoldering" V 3530 2200 50  0001 C CNN
 F 3 "~" H 3600 2200 50  0001 C CNN
-F 4 "311-10.0KCRCT-ND" H 3670 2109 50  0000 L CNN "DIGIKEY"
+F 4 "311-10.0KCRCT-ND" H 0   0   50  0001 C CNN "DigiKey"
 	1    3600 2200
 	1    0    0    -1
@@
 P 4800 3800
 F 0 "C4" H 4915 3891 50  0000 L CNN
-F 1 "100nF" H 4915 3800 50  0000 L CNN
+F 1 "0.1uF 50V" H 4915 3800 50  0000 L CNN
 F 2 "Capacitors_SMD:C_0805_HandSoldering" H 4838 3650 50  0001 C CNN
 F 3 "~" H 4800 3800 50  0001 C CNN
-F 4 "478-6048-1-ND" H 4915 3709 50  0000 L CNN "DIGIKEY"
+F 4 "478-6048-1-ND" H 0   0   50  0001 C CNN "DigiKey"
 	1    4800 3800
 	1    0    0    -1
@@
 Text Notes 9100 1650 0    50   ~ 0
 ONLY 16 bits timers are 1,3,4,5
-NoConn ~ 6900 4800
-NoConn ~ 6900 4900
-NoConn ~ 6900 5000
-NoConn ~ 6900 5100
-NoConn ~ 6900 5200
-NoConn ~ 6900 5300
-NoConn ~ 6900 5400
-NoConn ~ 6900 5500
 NoConn ~ 6900 4300
 NoConn ~ 6900 4200
@@
 F 2 "Pin_Headers:Pin_Header_Straight_1x02_Pitch2.54mm" H 9300 6300 50  0001 C CNN
 F 3 "~" H 9300 6300 50  0001 C CNN
+F 4 "S9337-ND" H 0   0   50  0001 C CNN "DigiKey"
 	1    9300 6300
 	1    0    0    -1
@@
 F 2 "Pin_Headers:Pin_Header_Straight_1x02_Pitch2.54mm" H 9300 6700 50  0001 C CNN
 F 3 "~" H 9300 6700 50  0001 C CNN
+F 4 "S9337-ND" H 0   0   50  0001 C CNN "DigiKey"
 	1    9300 6700
 	1    0    0    -1
@@
 F 2 "Pin_Headers:Pin_Header_Straight_1x02_Pitch2.54mm" H 11150 6300 50  0001 C CNN
 F 3 "~" H 11150 6300 50  0001 C CNN
+F 4 "S9337-ND" H 0   0   50  0001 C CNN "DigiKey"
 	1    11150 6300
 	1    0    0    -1
@@
 F 2 "Pin_Headers:Pin_Header_Straight_1x02_Pitch2.54mm" H 3350 4900 50  0001 C CNN
 F 3 "~" H 3350 4900 50  0001 C CNN
+F 4 "S9337-ND" H 0   0   50  0001 C CNN "DigiKey"
 	1    3350 4900
 	1    0    0    -1
@@
 F 2 "Pin_Headers:Pin_Header_Straight_1x02_Pitch2.54mm" H 2500 5000 50  0001 C CNN
 F 3 "~" H 2500 5000 50  0001 C CNN
+F 4 "S9337-ND" H 0   0   50  0001 C CNN "DigiKey"
 	1    2500 5000
 	1    0    0    -1
@@
 F 2 "Pin_Headers:Pin_Header_Straight_1x02_Pitch2.54mm" H 1600 5100 50  0001 C CNN
 F 3 "~" H 1600 5100 50  0001 C CNN
+F 4 "S9337-ND" H 0   0   50  0001 C CNN "DigiKey"
 	1    1600 5100
 	1    0    0    -1
@@
 F 2 "Pin_Headers:Pin_Header_Straight_1x02_Pitch2.54mm" H 1600 5200 50  0001 C CNN
 F 3 "~" H 1600 5200 50  0001 C CNN
+F 4 "S9337-ND" H 0   0   50  0001 C CNN "DigiKey"
 	1    1600 5200
 	1    0    0    1
@@
 F 2 "Pin_Headers:Pin_Header_Straight_1x02_Pitch2.54mm" H 2500 5300 50  0001 C CNN
 F 3 "~" H 2500 5300 50  0001 C CNN
+F 4 "S9337-ND" H 0   0   50  0001 C CNN "DigiKey"
 	1    2500 5300
 	1    0    0    1
@@
 F 2 "Pin_Headers:Pin_Header_Straight_1x02_Pitch2.54mm" H 3350 5400 50  0001 C CNN
 F 3 "~" H 3350 5400 50  0001 C CNN
+F 4 "S9337-ND" H 0   0   50  0001 C CNN "DigiKey"
 	1    3350 5400
 	1    0    0    1
@@
 F 2 "Pin_Headers:Pin_Header_Straight_1x02_Pitch2.54mm" H 4200 5500 50  0001 C CNN
 F 3 "~" H 4200 5500 50  0001 C CNN
+F 4 "S9337-ND" H 0   0   50  0001 C CNN "DigiKey"
 	1    4200 5500
 	1    0    0    1
@@
 F 2 "Pin_Headers:Pin_Header_Straight_1x02_Pitch2.54mm" H 4200 4800 50  0001 C CNN
 F 3 "~" H 4200 4800 50  0001 C CNN
+F 4 "S9337-ND" H 0   0   50  0001 C CNN "DigiKey"
 	1    4200 4800
 	1    0    0    -1
@@
 L Device:Jumper JP?
 U 1 1 5CFA790F
-P 7600 5700
+P 8400 5700
 AR Path="/5CFA790F" Ref="JP?"  Part="1"
 AR Path="/5C610827/5CFA790F" Ref="JP55"  Part="1"
-F 0 "JP55" H 7600 5964 50  0000 C CNN
-F 1 "Jumper" H 7600 5873 50  0000 C CNN
-F 2 "Pin_Headers:Pin_Header_Straight_1x02_Pitch2.54mm" H 7600 5700 50  0001 C CNN
-F 3 "~" H 7600 5700 50  0001 C CNN
-	1    7600 5700
-	-1   0    0    -1
-$EndComp
-Wire Wire Line
-	6900 5700 7300 5700
-Wire Wire Line
-	7900 5700 9600 5700
+F 0 "JP55" H 8400 5964 50  0000 C CNN
+F 1 "Jumper" H 8400 5873 50  0000 C CNN
+F 2 "Pin_Headers:Pin_Header_Straight_1x02_Pitch2.54mm" H 8400 5700 50  0001 C CNN
+F 3 "~" H 8400 5700 50  0001 C CNN
+F 4 "S9337-ND" H 0   0   50  0001 C CNN "DigiKey"
+	1    8400 5700
+	-1   0    0    -1
+$EndComp
+Wire Wire Line
+	6900 5700 8100 5700
+Wire Wire Line
+	8700 5700 9600 5700
 Wire Wire Line
 	10550 6700 11850 6700
@@
 NoConn ~ 6900 6300
 NoConn ~ 6900 6400
+$Comp
+L Connector:Conn_01x08_Female J15
+U 1 1 5CEE8189
+P 7350 5100
+F 0 "J15" H 7378 5076 50  0000 L CNN
+F 1 "Conn_01x08_Female" H 7378 4985 50  0000 L CNN
+F 2 "Pin_Headers:Pin_Header_Straight_1x08_Pitch2.54mm" H 7350 5100 50  0001 C CNN
+F 3 "~" H 7350 5100 50  0001 C CNN
+	1    7350 5100
+	1    0    0    -1
+$EndComp
+Wire Wire Line
+	6900 4800 7150 4800
+Wire Wire Line
+	7150 4900 6900 4900
+Wire Wire Line
+	6900 5000 7150 5000
+Wire Wire Line
+	7150 5100 6900 5100
+Wire Wire Line
+	6900 5200 7150 5200
+Wire Wire Line
+	7150 5300 6900 5300
+Wire Wire Line
+	6900 5400 7150 5400
+Wire Wire Line
+	7150 5500 6900 5500
 $EndSCHEMATC

Commit message: old commit from v1
Parts:
- U3: symbol MCU_Microchip_ATmega:ATmega2561-16AU -> speeduino_mini-rescue:ATmega2561-16AU-MCU_Microchip_ATmega
Other:
- note added: "ICP1: PD4\nICP3: PE7"
- note added: "JUMP TO PD4 (Input Capture Pin for timer 1)"
Changed lines of the file:
@@
 EESchema Schematic File Version 4
-LIBS:speeduino_mini-cache
-EELAYER 29 0
+EELAYER 30 0
 EELAYER END
 $Descr A4 11693 8268
 encoding utf-8
-Sheet 19 22
+Sheet 19 23
 Title ""
 Date ""
@@
 $EndDescr
 $Comp
-L MCU_Microchip_ATmega:ATmega2561-16AU U3
+L speeduino_mini-rescue:ATmega2561-16AU-MCU_Microchip_ATmega U3
 U 1 1 5C710FBC
 P 6300 4700
+AR Path="/5C710FBC" Ref="U3"  Part="1"
+AR Path="/5C610827/5C710FBC" Ref="U3"  Part="1"
 F 0 "U3" H 6300 2400 50  0000 C CNN
 F 1 "ATmega2561-16AU" H 6300 2300 50  0000 C CNN
@@
 Wire Wire Line
 	7150 5500 6900 5500
+Text Notes 5150 6750 0    50   ~ 0
+ICP1: PD4\nICP3: PE7
+Text Notes 7000 5700 0    50   ~ 0
+JUMP TO PD4 (Input Capture Pin for timer 1)
 $EndSCHEMATC
