File: hardware/power.sch (KiCad schematic (older format))
At the start: 10 parts, among them U8 LD1117S50TR_SOT223

Commit message: work in progress - components ordered
Parts:
- removed C16, C36, C6: 100nF, Capacitors_SMD:C_0805, symbol Device:C
- removed L2: 10uH, Inductors_SMD:L_0805, symbol Device:L
- added C38: 22uF, Capacitors_SMD:C_0805, symbol Device:C
- added C39: 1u, Capacitors_SMD:C_0805, symbol Device:C
- added C40: 22nF, Capacitors_SMD:C_0805, symbol Device:C
- added C41: 220nF, Capacitors_SMD:C_0805, symbol Device:C
- added D3: ACGRKM4007-HF, Diodes_SMD:D_SOD-123F, symbol Diode:1N4148
- added D4: D_Schottky, Diodes_SMD:D_SOD-323F, symbol Device:D_Schottky
- added L3, L4: 47uH, Speeduino Mini:BOURNS_SRR1260, symbol Device:L
- added PC3, PC4: 47uF, Capacitors_SMD:C_1206, symbol Device:C
- added R16: 10k, Resistors_SMD:R_0805, symbol Device:R
- added R25: 22k, Resistors_SMD:R_0805, symbol Device:R
- added U11: TLE8366, Housings_SOIC:SOIC-8-1EP_3.9x4.9mm_Pitch1.27mm, symbol speeduino_mini:TLE8366
- C37: value 100nF -> 22uF; DIGIKEY 478-6048-1-ND -> 490-9956-1-ND
Connections:
- net labels added: +5VD, EN
- net labels removed: +5V
- wire segments 36 -> 73
Other:
- note added: "5V regulator for ATmega2561 - always ON"
- note added: "5V regulator for sensors and Raspberry PI\n2A max, enabled by default, can be forced OFF by ATmega2561\nRaspberry PI will turn ON if ATmega unprogrammed for firmware loading"
- moved on the sheet: C35, PC1, PC2, U8

Commit message: rev 1
Parts:
- added D7: ACGRKM4007-HF, Diodes_SMD:D_SOD-123F, symbol Diode:1N4148
- D4: footprint Diodes_SMD:D_SOD-323F -> Diodes_SMD:D_SOD-123F
- PC1: footprint Capacitors_Tantalum_SMD:CP_Tantalum_Case-R_EIA-2012-12_Reflow -> Capacitors_Tantalum_SMD:CP_Tantalum_Case-C_EIA-6032-28_Reflow
Connections:
- wire segments 73 -> 79
Changed lines of the file:
@@
 EESchema Schematic File Version 4
 LIBS:speeduino_mini-cache
-EELAYER 26 0
+EELAYER 29 0
 EELAYER END
 $Descr A4 11693 8268
 encoding utf-8
-Sheet 14 18
+Sheet 14 21
 Title ""
 Date ""
@@
 F 0 "PC1" H 7268 1841 50  0000 L CNN
 F 1 "47uF" H 7268 1750 50  0000 L CNN
-F 2 "Capacitors_Tantalum_SMD:CP_Tantalum_Case-R_EIA-2012-12_Reflow" H 7188 1600 50  0001 C CNN
+F 2 "Capacitors_Tantalum_SMD:CP_Tantalum_Case-C_EIA-6032-28_Reflow" H 7188 1600 50  0001 C CNN
 F 3 "~" H 7150 1750 50  0001 C CNN
 F 4 "478-1773-1-ND" H 7268 1659 50  0000 L CNN "DIGIKEY"
@@
 F 0 "D4" V 6459 5479 50  0000 L CNN
 F 1 "D_Schottky" V 6550 5479 50  0000 L CNN
-F 2 "Diodes_SMD:D_SOD-323F" H 6550 5400 50  0001 C CNN
+F 2 "Diodes_SMD:D_SOD-123F" H 6550 5400 50  0001 C CNN
 F 3 "~" H 6550 5400 50  0001 C CNN
 F 4 "NRVTS245ESFT1GOSCT-ND" V 6641 5479 50  0000 L CNN "DIGIKEY"
@@
 $EndComp
 Wire Wire Line
-	1250 3050 1250 3300
-Wire Wire Line
-	1250 3600 1250 4250
+	1250 3050 1250 3250
+Wire Wire Line
+	1250 3600 1250 3650
 $Comp
 L Device:L L?
@@
 	4100 4650 3950 4650
 Connection ~ 4100 4650
+$Comp
+L Diode:1N4148 D?
+U 1 1 5C866CDA
+P 2150 3450
+AR Path="/5C610827/5C866CDA" Ref="D?"  Part="1"
+AR Path="/5C95BECF/5C866CDA" Ref="D7"  Part="1"
+F 0 "D7" V 2241 3371 50  0000 R CNN
+F 1 "ACGRKM4007-HF" V 2150 3371 50  0000 R CNN
+F 2 "Diodes_SMD:D_SOD-123F" H 2150 3275 50  0001 C CNN
+F 3 "http://www.comchiptech.com/admin/files/product/ACGRKM4001-HF%20Thru.%20ACGRKM4007-HF%20RevC.pdf" H 2150 3450 50  0001 C CNN
+F 4 "641-1634-1-ND" V 2059 3371 50  0000 R CNN "DIGIKEY"
+	1    2150 3450
+	0    -1   -1   0
+$EndComp
+Wire Wire Line
+	2150 3300 2150 3250
+Wire Wire Line
+	2150 3250 1250 3250
+Connection ~ 1250 3250
+Wire Wire Line
+	1250 3250 1250 3300
+Wire Wire Line
+	2150 3600 2150 3650
+Wire Wire Line
+	2150 3650 1250 3650
+Connection ~ 1250 3650
+Wire Wire Line
+	1250 3650 1250 4250
 $EndSCHEMATC

Commit message: Rev 2 work in progress
Parts:
- removed C35: 100nF, Capacitors_SMD:C_0805, symbol Device:C
- removed D2, D3, D7: ACGRKM4007-HF, Diodes_SMD:D_SOD-123F, symbol Diode:1N4148
- removed PC1: 47uF, Capacitors_Tantalum_SMD:CP_Tantalum_Case-C_EIA-6032-28_Reflow, symbol Device:CP
- removed PC2: 47uF, Capacitors_SMD:C_1206, symbol Device:C
- removed U8: LD1117S50TR_SOT223, TO_SOT_Packages_SMD:SOT-223-3_TabPin2, symbol Regulator_Linear:LD1117S50TR_SOT223
- added D3: LED, LEDs:LED_0805_HandSoldering, symbol Device:LED
- added R50: R_US, Resistors_SMD:R_0805_HandSoldering, symbol Device:R_US
- C37, C38, C39, C40, C41: footprint Capacitors_SMD:C_0805 -> Capacitors_SMD:C_0805_HandSoldering
- R16, R25: footprint Resistors_SMD:R_0805 -> Resistors_SMD:R_0805_HandSoldering
Connections:
- net labels added: +5V
- net labels removed: +5VA, +5VD
- wire segments 79 -> 47
Other:
- note removed: "5V regulator for ATmega2561 - always ON"
- moved on the sheet: C37, C38, C39, C40, C41, D4, L3, L4, PC3, PC4, R16, R25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

Commit message: rev 2 sent to fab
Parts:
- C37, C38: value 22uF -> 22uF 25V; DIGIKEY 490-9956-1-ND -> (none); DigiKey (none) -> 490-12389-1-ND
- C39: value 1u -> 1uF 35V; DIGIKEY 1276-6517-1-ND -> (none); DigiKey (none) -> 1276-6517-1-ND
- C40: value 22nF -> 22nF 50V; DIGIKEY 399-6945-1-ND -> (none); DigiKey (none) -> 399-6986-1-ND
- C41: value 220nF -> 0.22uF 50V; DIGIKEY 1276-7012-1-ND -> (none); DigiKey (none) -> 445-5683-1-ND
- D3: value LED -> LED GREEN 2.5mA 2.7V; DigiKey (none) -> 732-4983-1-ND
- D4: DIGIKEY NRVTS245ESFT1GOSCT-ND -> (none); DigiKey (none) -> NRVTS245ESFT1GOSCT-ND
- L3, L4: DIGIKEY SRR1260-470MCT-ND -> (none); DigiKey (none) -> SRR1260-470MCT-ND
- PC3, PC4: value 47uF -> 47uF 10V; footprint Capacitors_SMD:C_1206 -> Capacitors_SMD:C_1206_HandSoldering; DIGIKEY 490-12438-1-ND -> (none); DigiKey (none) -> 490-12438-1-ND
- R16: DIGIKEY 311-10.0KCRCT-ND -> (none); DigiKey (none) -> 311-10.0KCRCT-ND
- R25: DIGIKEY RMCF0805JT22K0CT-ND -> (none); DigiKey (none) -> RMCF0805JT22K0CT-ND
- R50: value R_US -> 910; DigiKey (none) -> P910ACT-ND
- U11: DIGIKEY TLE8366EV50XUMA1CT-ND -> (none); DigiKey (none) -> TLE8366EV50XUMA1CT-ND
Changed lines of the file:
@@
 F 2 "Housings_SOIC:SOIC-8-1EP_3.9x4.9mm_Pitch1.27mm" H 5200 3400 50  0001 C CNN
 F 3 "https://www.infineon.com/dgdl/Infineon-TLE8366-DS-v01_00-EN.pdf?fileId=5546d46258fc0bc1015969d2def641fa" H 5300 3300 50  0001 C CNN
-F 4 "TLE8366EV50XUMA1CT-ND" H 5300 4673 50  0000 C CNN "DIGIKEY"
+F 4 "TLE8366EV50XUMA1CT-ND" H 0   0   50  0001 C CNN "DigiKey"
 	1    5300 4100
 	1    0    0    -1
@@
 P 3650 4300
 F 0 "C40" H 3765 4391 50  0000 L CNN
-F 1 "22nF" H 3765 4300 50  0000 L CNN
+F 1 "22nF 50V" H 3765 4300 50  0000 L CNN
 F 2 "Capacitors_SMD:C_0805_HandSoldering" H 3688 4150 50  0001 C CNN
 F 3 "~" H 3650 4300 50  0001 C CNN
-F 4 "399-6945-1-ND" H 3765 4209 50  0000 L CNN "DIGIKEY"
+F 4 "399-6986-1-ND" H 0   0   50  0001 C CNN "DigiKey"
 	1    3650 4300
 	1    0    0    -1
@@
 F 2 "Resistors_SMD:R_0805_HandSoldering" V 3580 4750 50  0001 C CNN
 F 3 "~" H 3650 4750 50  0001 C CNN
-F 4 "RMCF0805JT22K0CT-ND" H 3720 4659 50  0000 L CNN "DIGIKEY"
+F 4 "RMCF0805JT22K0CT-ND" H 0   0   50  0001 C CNN "DigiKey"
 	1    3650 4750
 	1    0    0    -1
@@
 P 6100 3900
 F 0 "C41" H 6215 3991 50  0000 L CNN
-F 1 "220nF" H 6215 3900 50  0000 L CNN
+F 1 "0.22uF 50V" H 6215 3900 50  0000 L CNN
 F 2 "Capacitors_SMD:C_0805_HandSoldering" H 6138 3750 50  0001 C CNN
 F 3 "~" H 6100 3900 50  0001 C CNN
-F 4 "1276-7012-1-ND" H 6215 3809 50  0000 L CNN "DIGIKEY"
+F 4 "445-5683-1-ND" H 0   0   50  0001 C CNN "DigiKey"
 	1    6100 3900
 	1    0    0    -1
@@
 F 2 "Diodes_SMD:D_SOD-123F" H 6100 4550 50  0001 C CNN
 F 3 "~" H 6100 4550 50  0001 C CNN
-F 4 "NRVTS245ESFT1GOSCT-ND" V 6191 4629 50  0000 L CNN "DIGIKEY"
+F 4 "NRVTS245ESFT1GOSCT-ND" H 0   0   50  0001 C CNN "DigiKey"
 	1    6100 4550
 	0    1    1    0
@@
 AR Path="/5C95BECF/5C6DE8A2" Ref="C37"  Part="1"
 F 0 "C37" H 915 4191 50  0000 L CNN
-F 1 "22uF" H 915 4100 50  0000 L CNN
+F 1 "22uF 25V" H 915 4100 50  0000 L CNN
 F 2 "Capacitors_SMD:C_0805_HandSoldering" H 838 3950 50  0001 C CNN
 F 3 "~" H 800 4100 50  0001 C CNN
-F 4 "490-9956-1-ND" H 915 4009 50  0000 L CNN "DIGIKEY"
+F 4 "490-12389-1-ND" H 0   0   50  0001 C CNN "DigiKey"
 	1    800  4100
 	1    0    0    -1
@@
 AR Path="/5C95BECF/5C6DE8AA" Ref="C38"  Part="1"
 F 0 "C38" H 1915 4191 50  0000 L CNN
-F 1 "22uF" H 1915 4100 50  0000 L CNN
+F 1 "22uF 25V" H 1915 4100 50  0000 L CNN
 F 2 "Capacitors_SMD:C_0805_HandSoldering" H 1838 3950 50  0001 C CNN
 F 3 "~" H 1800 4100 50  0001 C CNN
-F 4 "490-9956-1-ND" H 1915 4009 50  0000 L CNN "DIGIKEY"
+F 4 "490-12389-1-ND" H 0   0   50  0001 C CNN "DigiKey"
 	1    1800 4100
 	1    0    0    -1
@@
 AR Path="/5C95BECF/5C6ED2D9" Ref="C39"  Part="1"
 F 0 "C39" H 2815 4191 50  0000 L CNN
-F 1 "1u" H 2815 4100 50  0000 L CNN
+F 1 "1uF 35V" H 2815 4100 50  0000 L CNN
 F 2 "Capacitors_SMD:C_0805_HandSoldering" H 2738 3950 50  0001 C CNN
 F 3 "~" H 2700 4100 50  0001 C CNN
-F 4 "1276-6517-1-ND" H 2815 4009 50  0000 L CNN "DIGIKEY"
+F 4 "1276-6517-1-ND" H 0   0   50  0001 C CNN "DigiKey"
 	1    2700 4100
 	1    0    0    -1
@@
 F 2 "Speeduino Mini:BOURNS_SRR1260" H 1300 3400 50  0001 C CNN
 F 3 "https://www.bourns.com/docs/Product-Datasheets/SRP1265A.pdf" H 1300 3400 50  0001 C CNN
-F 4 "SRR1260-470MCT-ND" V 1398 3400 50  0000 C CNN "DIGIKEY"
+F 4 "SRR1260-470MCT-ND" H 0   0   50  0001 C CNN "DigiKey"
 	1    1300 3400
 	0    -1   -1   0
@@
 F 2 "Speeduino Mini:BOURNS_SRR1260" H 7550 4100 50  0001 C CNN
 F 3 "https://www.bourns.com/docs/Product-Datasheets/SRP1265A.pdf" H 7550 4100 50  0001 C CNN
-F 4 "SRR1260-470MCT-ND" V 7648 4100 50  0000 C CNN "DIGIKEY"
+F 4 "SRR1260-470MCT-ND" H 0   0   50  0001 C CNN "DigiKey"
 	1    7550 4100
 	0    -1   -1   0
@@
 AR Path="/5C95BECF/5C6FB7EB" Ref="PC3"  Part="1"
 F 0 "PC3" H 8265 4641 50  0000 L CNN
-F 1 "47uF" H 8265 4550 50  0000 L CNN
-F 2 "Capacitors_SMD:C_1206" H 8188 4400 50  0001 C CNN
+F 1 "47uF 10V" H 8265 4550 50  0000 L CNN
+F 2 "Capacitors_SMD:C_1206_HandSoldering" H 8188 4400 50  0001 C CNN
 F 3 "~" H 8150 4550 50  0001 C CNN
-F 4 "490-12438-1-ND" H 8265 4459 50  0000 L CNN "DIGIKEY"
+F 4 "490-12438-1-ND" H 0   0   50  0001 C CNN "DigiKey"
 	1    8150 4550
 	1    0    0    -1
@@
 AR Path="/5C95BECF/5C6FD18A" Ref="PC4"  Part="1"
 F 0 "PC4" H 9415 4691 50  0000 L CNN
-F 1 "47uF" H 9415 4600 50  0000 L CNN
-F 2 "Capacitors_SMD:C_1206" H 9338 4450 50  0001 C CNN
+F 1 "47uF 10V" H 9415 4600 50  0000 L CNN
+F 2 "Capacitors_SMD:C_1206_HandSoldering" H 9338 4450 50  0001 C CNN
 F 3 "~" H 9300 4600 50  0001 C CNN
-F 4 "490-12438-1-ND" H 9415 4509 50  0000 L CNN "DIGIKEY"
+F 4 "490-12438-1-ND" H 0   0   50  0001 C CNN "DigiKey"
 	1    9300 4600
 	1    0    0    -1
@@
 F 2 "Resistors_SMD:R_0805_HandSoldering" V 3580 3600 50  0001 C CNN
 F 3 "~" H 3650 3600 50  0001 C CNN
-F 4 "311-10.0KCRCT-ND" H 3580 3691 50  0000 R CNN "DIGIKEY"
+F 4 "311-10.0KCRCT-ND" H 0   0   50  0001 C CNN "DigiKey"
 	1    3650 3600
 	-1   0    0    1
@@
 AR Path="/5C95BECF/5D22D293" Ref="D3"  Part="1"
 F 0 "D3" V 10339 4633 50  0000 R CNN
-F 1 "LED" V 10248 4633 50  0000 R CNN
+F 1 "LED GREEN 2.5mA 2.7V" V 10248 4633 50  0000 R CNN
 F 2 "LEDs:LED_0805_HandSoldering" H 10300 4750 50  0001 C CNN
 F 3 "~" H 10300 4750 50  0001 C CNN
+F 4 "732-4983-1-ND" H 0   0   50  0001 C CNN "DigiKey"
 	1    10300 4750
 	0    -1   -1   0
@@
 AR Path="/5C95BECF/5D22D299" Ref="R50"  Part="1"
 F 0 "R50" H 10232 4304 50  0000 R CNN
-F 1 "R_US" H 10232 4395 50  0000 R CNN
+F 1 "910" H 10232 4395 50  0000 R CNN
 F 2 "Resistors_SMD:R_0805_HandSoldering" V 10340 4340 50  0001 C CNN
 F 3 "~" H 10300 4350 50  0001 C CNN
+F 4 "P910ACT-ND" H 0   0   50  0001 C CNN "DigiKey"
 	1    10300 4350
 	-1   0    0    1
