File: hardware/speeduino_mini.sch (KiCad schematic (older format))
At the start: 12 parts, among them J1 O2, J10 Injector 4, J11 Injectors, J12 oil pressure, J13 oil pressure, J3 TPS, J4 IAT, J5 head temperature, J6 crank hall, J7 Injector 1, J8 Injector 2, J9 Injector 3

Commit message: work in progress - components ordered
Parts:
- removed J6: crank hall, Speeduino Mini:ED120_2DS, symbol Connector:Screw_Terminal_01x02
- added J14: power, Speeduino Mini:ED120_3DS, symbol Connector:Screw_Terminal_01x03
- added J6: crankshaft position sensor, Speeduino Mini:ED120_3DS, symbol Connector:Screw_Terminal_01x03
- added R21, R22: 10k, Resistors_SMD:R_0805, symbol Device:R
- J11: value Injectors -> Ignitor Pack
Connections:
- net +12V: now also J14.1 (Pin_1)
- net +5VA: now also J6.1 (Pin_1)
- net GND: now also J14.3 (Pin_3), J6.3 (Pin_3), R21.1, R22.1
- net Ignitor/IGN1_OUT renamed MCU/OC1A
- net MCU/OC1A: now also R22.2
- net Ignitor/IGN2_OUT renamed MCU/OC1B
- net MCU/OC1B: now also R21.2
- new net Crankshaft pos sensor/IN: J6.2 (Pin_2)
- new net Lin transceiver/LIN: J14.2 (Pin_2)
- no-connect marks 3 -> 2
Other:
- moved on the sheet: J11, J12, J13

Commit message: rev 1
Parts:
- removed R21, R22: 10k, Resistors_SMD:R_0805, symbol Device:R
- added J15: camshaft position sensor, Speeduino Mini:ED120_3DS, symbol Connector:Screw_Terminal_01x03
- J13: value oil pressure -> fuel pressure
Connections:
- net MCU/OC1A is gone; now on net MCU/OC0B: J11.1 (Pin_1)
- net +5VA: now also J15.1 (Pin_1)
- net GND: now also J15.3 (Pin_3)
- net Injector 1 and 3/INJ_OUT renamed Injector 1/INJ_OUT
- net Injector 1/INJ_OUT: no longer J9.2 (Pin_2)
- net Injector 2 and 4/INJ_OUT renamed Injector 2/INJ_OUT
- net Injector 2/INJ_OUT: no longer J10.2 (Pin_2)
- net MCU/OC1B renamed MCU/OC3A
- new net Camshaft position sensor/OUT: J15.2 (Pin_2)
- new net Injector 3/INJ_OUT: J9.2 (Pin_2)
- new net Injector 4/INJ_OUT: J10.2 (Pin_2)
- no-connect marks 2 -> 0
Other:
- note added: "Ignitor pack consumes 18mA in idle.\nTODO: add a switch"
- note added: "Pull-downs in the ignitor pack"
- moved on the sheet: J10, J7, J8, J9

Commit message: Rev 2 work in progress
Parts:
- removed J10: Injector 4, Speeduino Mini:ED120_2DS, symbol Connector:Screw_Terminal_01x02
- removed J11: Ignitor Pack, Speeduino Mini:ED120_4DS, symbol Connector:Screw_Terminal_01x04
- removed J7: Injector 1, Speeduino Mini:ED120_2DS, symbol Connector:Screw_Terminal_01x02
- removed J8: Injector 2, Speeduino Mini:ED120_2DS, symbol Connector:Screw_Terminal_01x02
- removed J9: Injector 3, Speeduino Mini:ED120_2DS, symbol Connector:Screw_Terminal_01x02
- added JP1, JP10, JP11, JP12, JP13, JP14, JP15, JP16, JP17, JP18, JP19, JP2, JP20, JP21, JP22, JP23, JP24, JP25, JP26, JP27, JP28, JP29, JP3, JP30, JP31, JP32, JP33, JP34, JP35, JP36, JP37, JP38, JP39, JP4, JP40, JP45, JP5, JP6, JP7, JP8, JP9: Jumper, Pin_Headers:Pin_Header_Straight_1x02_Pitch2.54mm, symbol Device:Jumper
Connections:
- net +12V: now also JP10.2, JP11.2, JP12.2, JP13.1, JP31.2, JP8.2, JP9.2
- net +5VA: now also JP29.2, JP32.2, JP33.2, JP34.2, JP35.2, JP36.2, JP37.2, JP38.2, JP39.1, JP45.1; no longer J12.1 (Pin_1), J13.1 (Pin_1), J15.1 (Pin_1), J3.1 (Pin_1), J6.1 (Pin_1)
- net Battery Reference Voltage/OUT: now also JP20.1
- net Camshaft position sensor/IN: now also J15.2 (Pin_2)
- net Camshaft position sensor/OUT: now also JP40.2; no longer J15.2 (Pin_2)
- net Crankshaft pos sensor/OUT: now also JP21.1
- net Fuel Pressure/OUT: now also JP23.1
- net Head Temperature Sensor/OUT: now also JP19.1
- net Injector 1/INJ_CMD: now also JP1.2
- net Injector 2/INJ_CMD: now also JP2.2
- net Injector 3/INJ_CMD: now also JP3.2
- net Injector 4/INJ_CMD: now also JP4.2
- net Intake Air Temperature Sensor/OUT: now also JP18.1
- net MAP Sensor/OUT: now also JP16.1
- net MCU/A1: now also JP15.2
- net MCU/A5: now also JP17.2
- net MCU/A6: now also JP22.2
- net MCU/OC3A: now also JP6.1
- net MCU/PA0: now also JP14.2
- net MCU/PB7: now also JP30.1
- net MCU/RESET: now also JP27.1
- net MCU/RXD0: now also JP25.1
- net MCU/SCK: now also JP26.1
- net MCU/TXD0: now also JP24.1
- net Lin transceiver/LIN renamed MCU/LIN
- new net: J3.1 (Pin_1), JP36.1
- new net: J12.1 (Pin_1), JP34.1
- new net: J13.1 (Pin_1), JP35.1
- new net: J6.1 (Pin_1), JP33.1
- new net: J15.1 (Pin_1), JP39.2
- new net +5VD: JP28.2
- new net Head Temperature Sensor/VCC: JP38.1
- new net Ignitor/+12V: JP12.1
- new net Ignitor/EN: JP5.2
- new net Ignitor/IN1: JP6.2
- new net Ignitor/IN2: JP7.2
- new net Injector 1/+12V: JP8.1
- new net Injector 2/+12V: JP9.1
- new net Injector 3/+12V: JP10.1
- new net Injector 4/+12V: JP11.1
- new net Intake Air Temperature Sensor/VCC: JP37.1
- new net MAP Sensor/+5V: JP45.2
- new net MCU/A0: JP20.2
- new net MCU/A2: JP18.2
- new net MCU/A3: JP19.2
- new net MCU/A4: JP16.2
- new net MCU/A7: JP23.2
- new net MCU/INT0: JP40.1
- new net MCU/INT1: JP21.2
- new net MCU/OC1A: JP1.1, JP2.1
- new net MCU/OC1B: JP3.1, JP4.1
- new net MCU/OC3B: JP7.1
- new net MCU/OC3C: JP5.1
- new net O2 Sensor Power/+12V: JP13.2
- new net O2 Sensor Power/EN: JP14.1
- new net O2 Sensor/OUT: JP15.1
- new net Oil Pressure Sensor/OUT: JP22.1
- new net Power/+12V: JP31.1
- new net Power/+5V: JP32.1
- new net Power/EN: JP30.2
- new net Raspberry Pi Zero W/+5VA: JP29.1
- new net Raspberry Pi Zero W/+5VD: JP28.1
- new net Raspberry Pi Zero W/ATMEGA_RESET: JP27.2
- new net Raspberry Pi Zero W/RXD_PDO: JP24.2
- new net Raspberry Pi Zero W/SCK: JP26.2
- new net Raspberry Pi Zero W/TXD_PDI: JP25.2
- new net Throttle Position Sensor /OUT: JP17.1
Other:
- note added: "TODO add fuel pump driver?"
- note added: "TODO: add pinIdle ?"
- note removed: "Ignitor pack consumes 18mA in idle.\nTODO: add a switch"
- note removed: "Pull-downs in the ignitor pack"
- moved on the sheet: J1, J12, J13, J14, J15, J3, J4, J5, J6

Commit message: rev 2 work in progress
Parts:
- removed J15: camshaft position sensor, Speeduino Mini:ED120_3DS, symbol Connector:Screw_Terminal_01x03
- removed JP39, JP40: Jumper, Pin_Headers:Pin_Header_Straight_1x02_Pitch2.54mm, symbol Device:Jumper
- added H1, H2, H3, H4: MountingHole, Mounting_Holes:MountingHole_4.3mm_M4_Pad_Via, symbol Mechanical:MountingHole
- added JP48: Jumper, Pin_Headers:Pin_Header_Straight_1x02_Pitch2.54mm, symbol Device:Jumper
Connections:
- net +12V: now also JP48.2
- net MCU/A1: now also JP23.2; no longer JP15.2
- net MCU/A7: now also JP15.2; no longer JP23.2
- net MCU/OC1A: now also JP3.1, JP4.1; no longer JP1.1, JP2.1
- net MCU/OC1B: now also JP1.1, JP2.1; no longer JP3.1, JP4.1
- net MCU/OC3A: now also JP7.1; no longer JP6.1
- net MCU/OC3B: now also JP5.1; no longer JP7.1
- net MCU/OC3C: now also JP6.1; no longer JP5.1
- new net Battery Reference Voltage/+12V: JP48.1
- no-connect marks 0 -> 1
Changed lines of the file:
@@
 $Descr A4 11693 8268
 encoding utf-8
-Sheet 1 23
+Sheet 1 22
 Title ""
 Date ""
@@
 	1    0    0    -1
 $EndComp
-$Sheet
-S 7600 7300 1050 200
-U 5C97692A
-F0 "Camshaft position sensor" 50
-F1 "analog_sensor.sch" 50
-F2 "IN" I R 8650 7400 50
-F3 "OUT" O L 7600 7400 50
-$EndSheet
-$Comp
-L Connector:Screw_Terminal_01x03 J15
-U 1 1 5C985C13
-P 9500 7400
-F 0 "J15" H 9580 7487 50  0000 L CNN
-F 1 "camshaft position sensor" H 9580 7396 50  0000 L CNN
-F 2 "Speeduino Mini:ED120_3DS" H 9500 7400 50  0001 C CNN
-F 3 "~" H 9500 7400 50  0001 C CNN
-F 4 "ED1610-ND" H 9580 7305 50  0000 L CNN "DIGIKEY"
-	1    9500 7400
-	1    0    0    -1
-$EndComp
-$Comp
-L power:GND #PWR078
-U 1 1 5C985C1F
-P 9300 7500
-F 0 "#PWR078" H 9300 7250 50  0001 C CNN
-F 1 "GND" H 9305 7327 50  0000 C CNN
-F 2 "" H 9300 7500 50  0001 C CNN
-F 3 "" H 9300 7500 50  0001 C CNN
-	1    9300 7500
-	-1   0    0    -1
-$EndComp
-Wire Wire Line
-	8650 7400 9300 7400
 $Sheet
 S 7600 2000 1050 200
@@
 F3 "A2" I L 4750 3900 50
 F4 "A0" I L 4750 5050 50
-F5 "A1" I L 4750 1650 50
+F5 "A1" I L 4750 7550 50
 F6 "A4" I L 4750 2200 50
 F7 "TXD0" O R 6500 4050 50
@@
 F9 "A5" I L 4750 3050 50
 F10 "A6" I L 4750 6700 50
-F11 "A7" I L 4750 7550 50
+F11 "A7" I L 4750 1650 50
 F12 "INT1" I L 4750 5850 50
-F13 "INT0" I R 6500 7400 50
-F16 "OC1B" O R 6500 2100 50
-F17 "OC1A" O R 6500 1300 50
-F18 "OC3C" O R 6500 2900 50
-F19 "OC3B" O R 6500 3600 50
-F20 "OC3A" O R 6500 3250 50
-F21 "PA0" O L 4750 1250 50
-F22 "SCK" I R 6500 4850 50
-F23 "RESET" I R 6500 5250 50
-F24 "PB7" O R 6500 6250 50
-F25 "+12V" I R 6500 7850 50
-F26 "LIN" B R 6500 5750 50
+F13 "INT0" I L 4750 5750 50
+F14 "OC1B" O R 6500 1300 50
+F15 "OC1A" O R 6500 2100 50
+F16 "OC3C" O R 6500 3250 50
+F17 "OC3B" O R 6500 2900 50
+F18 "OC3A" O R 6500 3600 50
+F19 "PA0" O L 4750 1250 50
+F20 "SCK" I R 6500 4850 50
+F21 "RESET" I R 6500 5250 50
+F22 "PB7" O R 6500 6250 50
+F23 "+12V" I R 6500 7850 50
+F24 "LIN" B R 6500 5750 50
+F25 "VCC" O R 6500 5550 50
 $EndSheet
 $Comp
@@
 L power:+12V #PWR0125
 U 1 1 5D2F4157
-P 2000 4950
-F 0 "#PWR0125" H 2000 4800 50  0001 C CNN
-F 1 "+12V" H 2015 5123 50  0000 C CNN
-F 2 "" H 2000 4950 50  0001 C CNN
-F 3 "" H 2000 4950 50  0001 C CNN
-	1    2000 4950
-	1    0    0    -1
-$EndComp
-Wire Wire Line
-	2000 4950 2000 5050
+P 1400 5050
+F 0 "#PWR0125" H 1400 4900 50  0001 C CNN
+F 1 "+12V" H 1415 5223 50  0000 C CNN
+F 2 "" H 1400 5050 50  0001 C CNN
+F 3 "" H 1400 5050 50  0001 C CNN
+	1    1400 5050
+	0    -1   -1   0
+$EndComp
 Wire Wire Line
 	2000 5050 2200 5050
@@
 Wire Wire Line
 	2200 3600 2100 3600
-$Comp
-L Device:Jumper JP39
-U 1 1 5D3B3476
-P 8550 7100
-F 0 "JP39" H 8550 7364 50  0000 C CNN
-F 1 "Jumper" H 8550 7273 50  0000 C CNN
-F 2 "Pin_Headers:Pin_Header_Straight_1x02_Pitch2.54mm" H 8550 7100 50  0001 C CNN
-F 3 "~" H 8550 7100 50  0001 C CNN
-	1    8550 7100
-	1    0    0    -1
-$EndComp
-Wire Wire Line
-	8250 7100 8150 7100
-Wire Wire Line
-	8850 7100 9000 7100
-Wire Wire Line
-	9000 7100 9000 7300
-Wire Wire Line
-	9000 7300 9300 7300
-$Comp
-L Device:Jumper JP40
-U 1 1 5D3CB83D
-P 7150 7400
-F 0 "JP40" H 7150 7664 50  0000 C CNN
-F 1 "Jumper" H 7150 7573 50  0000 C CNN
-F 2 "Pin_Headers:Pin_Header_Straight_1x02_Pitch2.54mm" H 7150 7400 50  0001 C CNN
-F 3 "~" H 7150 7400 50  0001 C CNN
-	1    7150 7400
-	1    0    0    -1
-$EndComp
-Wire Wire Line
-	6850 7400 6500 7400
-Wire Wire Line
-	7450 7400 7600 7400
 Wire Wire Line
 	6500 5750 9350 5750
@@
 $EndComp
 $Comp
-L power:+5VA #PWR?
-U 1 1 5D4E8283
-P 8150 7100
-F 0 "#PWR?" H 8150 6950 50  0001 C CNN
-F 1 "+5VA" H 8165 7273 50  0000 C CNN
-F 2 "" H 8150 7100 50  0001 C CNN
-F 3 "" H 8150 7100 50  0001 C CNN
-	1    8150 7100
-	-1   0    0    -1
-$EndComp
+L Device:Jumper JP48
+U 1 1 5CE6BED5
+P 1700 5050
+F 0 "JP48" H 1700 5314 50  0000 C CNN
+F 1 "Jumper" H 1700 5223 50  0000 C CNN
+F 2 "Pin_Headers:Pin_Header_Straight_1x02_Pitch2.54mm" H 1700 5050 50  0001 C CNN
+F 3 "~" H 1700 5050 50  0001 C CNN
+	1    1700 5050
+	-1   0    0    -1
+$EndComp
+NoConn ~ 4750 5750
+$Comp
+L Mechanical:MountingHole H1
+U 1 1 5CF25801
+P 10500 800
+F 0 "H1" H 10600 846 50  0000 L CNN
+F 1 "MountingHole" H 10600 755 50  0000 L CNN
+F 2 "Mounting_Holes:MountingHole_4.3mm_M4_Pad_Via" H 10500 800 50  0001 C CNN
+F 3 "~" H 10500 800 50  0001 C CNN
+	1    10500 800
+	1    0    0    -1
+$EndComp
+$Comp
+L Mechanical:MountingHole H2
+U 1 1 5CF25EA8
+P 10500 1000
+F 0 "H2" H 10600 1046 50  0000 L CNN
+F 1 "MountingHole" H 10600 955 50  0000 L CNN
+F 2 "Mounting_Holes:MountingHole_4.3mm_M4_Pad_Via" H 10500 1000 50  0001 C CNN
+F 3 "~" H 10500 1000 50  0001 C CNN
+	1    10500 1000
+	1    0    0    -1
+$EndComp
+$Comp
+L Mechanical:MountingHole H3
+U 1 1 5CF260A5
+P 10500 1200
+F 0 "H3" H 10600 1246 50  0000 L CNN
+F 1 "MountingHole" H 10600 1155 50  0000 L CNN
+F 2 "Mounting_Holes:MountingHole_4.3mm_M4_Pad_Via" H 10500 1200 50  0001 C CNN
+F 3 "~" H 10500 1200 50  0001 C CNN
+	1    10500 1200
+	1    0    0    -1
+$EndComp
+$Comp
+L Mechanical:MountingHole H4
+U 1 1 5CF26378
+P 10500 1400
+F 0 "H4" H 10600 1446 50  0000 L CNN
+F 1 "MountingHole" H 10600 1355 50  0000 L CNN
+F 2 "Mounting_Holes:MountingHole_4.3mm_M4_Pad_Via" H 10500 1400 50  0001 C CNN
+F 3 "~" H 10500 1400 50  0001 C CNN
+	1    10500 1400
+	1    0    0    -1
+$EndComp
+$Comp
+L power:+5VD #PWR0133
+U 1 1 5CF6B9DD
+P 6650 5550
+F 0 "#PWR0133" H 6650 5400 50  0001 C CNN
+F 1 "+5VD" V 6665 5678 50  0000 L CNN
+F 2 "" H 6650 5550 50  0001 C CNN
+F 3 "" H 6650 5550 50  0001 C CNN
+	1    6650 5550
+	0    1    1    0
+$EndComp
+Wire Wire Line
+	6500 5550 6650 5550
 $EndSCHEMATC

Commit message: hardware rev2 - layout complete
Parts:
- removed JP15, JP16, JP17, JP18, JP19, JP20, JP21, JP22, JP23, JP33, JP34, JP35, JP36, JP37, JP38, JP48: Jumper, Pin_Headers:Pin_Header_Straight_1x02_Pitch2.54mm, symbol Device:Jumper
Connections:
- net +5VA: now also J12.1 (Pin_1), J13.1 (Pin_1), J3.1 (Pin_1), J6.1 (Pin_1)
- net MCU/PB7 renamed MCU/PA1
- no-connect marks 1 -> 0

Commit message: rev 2 sent to fab
Parts:
- H1, H2, H3, H4: DigiKey (none) -> 1772-4097-ND
- J1: DIGIKEY ED2227-ND -> (none); DigiKey (none) -> ED2227-ND
- J12, J13, J14, J3, J6: DIGIKEY ED1610-ND -> (none); DigiKey (none) -> ED1610-ND
- J4, J5: DIGIKEY ED1609-ND -> (none); DigiKey (none) -> ED1609-ND
- JP1, JP10, JP11, JP12, JP13, JP14, JP2, JP24, JP25, JP26, JP27, JP28, JP29, JP3, JP30, JP31, JP32, JP4, JP45, JP5, JP6, JP7, JP8, JP9: DigiKey (none) -> S9337-ND
Changed lines of the file:
@@
 F 2 "Speeduino Mini:ED120_3DS" H 1250 3050 50  0001 C CNN
 F 3 "~" H 1250 3050 50  0001 C CNN
-F 4 "ED1610-ND" H 1330 2955 50  0000 L CNN "DIGIKEY"
+F 4 "ED1610-ND" H 0   0   50  0001 C CNN "DigiKey"
 	1    1250 3050
 	-1   0    0    -1
@@
 F 2 "Speeduino Mini:ED120_2DS" H 1250 3850 50  0001 C CNN
 F 3 "http://www.on-shore.com/wp-content/uploads/2015/09/ed120ds.pdf" H 1250 3850 50  0001 C CNN
-F 4 "ED1609-ND" H 1330 3705 50  0000 L CNN "DIGIKEY"
+F 4 "ED1609-ND" H 0   0   50  0001 C CNN "DigiKey"
 	1    1250 3850
 	-1   0    0    -1
@@
 F 2 "Speeduino Mini:ED120_3DS" H 1350 6700 50  0001 C CNN
 F 3 "~" H 1350 6700 50  0001 C CNN
-F 4 "ED1610-ND" H 1430 6605 50  0000 L CNN "DIGIKEY"
+F 4 "ED1610-ND" H 0   0   50  0001 C CNN "DigiKey"
 	1    1350 6700
 	-1   0    0    -1
@@
 F 2 "Speeduino Mini:ED120_3DS" H 1350 7550 50  0001 C CNN
 F 3 "~" H 1350 7550 50  0001 C CNN
-F 4 "ED1610-ND" H 1430 7455 50  0000 L CNN "DIGIKEY"
+F 4 "ED1610-ND" H 0   0   50  0001 C CNN "DigiKey"
 	1    1350 7550
 	-1   0    0    -1
@@
 F 2 "Speeduino Mini:ED120_4DS" H 1250 1450 50  0001 C CNN
 F 3 "~" H 1250 1450 50  0001 C CNN
-F 4 "ED2227-ND" H 1330 1305 50  0000 L CNN "DIGIKEY"
+F 4 "ED2227-ND" H 0   0   50  0001 C CNN "DigiKey"
 	1    1250 1450
 	-1   0    0    -1
@@
 F 2 "Speeduino Mini:ED120_3DS" H 10200 5150 50  0001 C CNN
 F 3 "~" H 10200 5150 50  0001 C CNN
-F 4 "ED1610-ND" H 10280 5055 50  0000 L CNN "DIGIKEY"
+F 4 "ED1610-ND" H 0   0   50  0001 C CNN "DigiKey"
 	1    10200 5150
 	1    0    0    -1
@@
 F 2 "Pin_Headers:Pin_Header_Straight_1x02_Pitch2.54mm" H 7100 1300 50  0001 C CNN
 F 3 "~" H 7100 1300 50  0001 C CNN
+F 4 "S9337-ND" H 0   0   50  0001 C CNN "DigiKey"
 	1    7100 1300
 	1    0    0    -1
@@
 F 2 "Pin_Headers:Pin_Header_Straight_1x02_Pitch2.54mm" H 9050 1300 50  0001 C CNN
 F 3 "~" H 9050 1300 50  0001 C CNN
+F 4 "S9337-ND" H 0   0   50  0001 C CNN "DigiKey"
 	1    9050 1300
 	1    0    0    -1
@@
 F 2 "Pin_Headers:Pin_Header_Straight_1x02_Pitch2.54mm" H 7100 1700 50  0001 C CNN
 F 3 "~" H 7100 1700 50  0001 C CNN
+F 4 "S9337-ND" H 0   0   50  0001 C CNN "DigiKey"
 	1    7100 1700
 	1    0    0    -1
@@
 F 2 "Pin_Headers:Pin_Header_Straight_1x02_Pitch2.54mm" H 9050 1700 50  0001 C CNN
 F 3 "~" H 9050 1700 50  0001 C CNN
+F 4 "S9337-ND" H 0   0   50  0001 C CNN "DigiKey"
 	1    9050 1700
 	1    0    0    -1
@@
 F 2 "Pin_Headers:Pin_Header_Straight_1x02_Pitch2.54mm" H 7100 2100 50  0001 C CNN
 F 3 "~" H 7100 2100 50  0001 C CNN
+F 4 "S9337-ND" H 0   0   50  0001 C CNN "DigiKey"
 	1    7100 2100
 	1    0    0    -1
@@
 F 2 "Pin_Headers:Pin_Header_Straight_1x02_Pitch2.54mm" H 7100 2500 50  0001 C CNN
 F 3 "~" H 7100 2500 50  0001 C CNN
+F 4 "S9337-ND" H 0   0   50  0001 C CNN "DigiKey"
 	1    7100 2500
 	1    0    0    -1
@@
 F 2 "Pin_Headers:Pin_Header_Straight_1x02_Pitch2.54mm" H 9050 2100 50  0001 C CNN
 F 3 "~" H 9050 2100 50  0001 C CNN
+F 4 "S9337-ND" H 0   0   50  0001 C CNN "DigiKey"
 	1    9050 2100
 	1    0    0    -1
@@
 F 2 "Pin_Headers:Pin_Header_Straight_1x02_Pitch2.54mm" H 9050 2500 50  0001 C CNN
 F 3 "~" H 9050 2500 50  0001 C CNN
+F 4 "S9337-ND" H 0   0   50  0001 C CNN "DigiKey"
 	1    9050 2500
 	1    0    0    -1
@@
 F 2 "Pin_Headers:Pin_Header_Straight_1x02_Pitch2.54mm" H 9050 2900 50  0001 C CNN
 F 3 "~" H 9050 2900 50  0001 C CNN
+F 4 "S9337-ND" H 0   0   50  0001 C CNN "DigiKey"
 	1    9050 2900
 	1    0    0    -1
@@
 F 2 "Pin_Headers:Pin_Header_Straight_1x02_Pitch2.54mm" H 7100 2900 50  0001 C CNN
 F 3 "~" H 7100 2900 50  0001 C CNN
+F 4 "S9337-ND" H 0   0   50  0001 C CNN "DigiKey"
 	1    7100 2900
 	1    0    0    -1
@@
 F 2 "Pin_Headers:Pin_Header_Straight_1x02_Pitch2.54mm" H 7100 3250 50  0001 C CNN
 F 3 "~" H 7100 3250 50  0001 C CNN
+F 4 "S9337-ND" H 0   0   50  0001 C CNN "DigiKey"
 	1    7100 3250
 	1    0    0    -1
@@
 F 2 "Pin_Headers:Pin_Header_Straight_1x02_Pitch2.54mm" H 7100 3600 50  0001 C CNN
 F 3 "~" H 7100 3600 50  0001 C CNN
+F 4 "S9337-ND" H 0   0   50  0001 C CNN "DigiKey"
 	1    7100 3600
 	1    0    0    -1
@@
 F 2 "Pin_Headers:Pin_Header_Straight_1x02_Pitch2.54mm" H 4200 1250 50  0001 C CNN
 F 3 "~" H 4200 1250 50  0001 C CNN
+F 4 "S9337-ND" H 0   0   50  0001 C CNN "DigiKey"
 	1    4200 1250
 	1    0    0    -1
@@
 F 2 "Pin_Headers:Pin_Header_Straight_1x02_Pitch2.54mm" H 1750 1100 50  0001 C CNN
 F 3 "~" H 1750 1100 50  0001 C CNN
+F 4 "S9337-ND" H 0   0   50  0001 C CNN "DigiKey"
 	1    1750 1100
 	1    0    0    -1
@@
 F 2 "Pin_Headers:Pin_Header_Straight_1x02_Pitch2.54mm" H 7150 4050 50  0001 C CNN
 F 3 "~" H 7150 4050 50  0001 C CNN
+F 4 "S9337-ND" H 0   0   50  0001 C CNN "DigiKey"
 	1    7150 4050
 	1    0    0    -1
@@
 F 2 "Pin_Headers:Pin_Header_Straight_1x02_Pitch2.54mm" H 7150 4450 50  0001 C CNN
 F 3 "~" H 7150 4450 50  0001 C CNN
+F 4 "S9337-ND" H 0   0   50  0001 C CNN "DigiKey"
 	1    7150 4450
 	1    0    0    -1
@@
 F 2 "Pin_Headers:Pin_Header_Straight_1x02_Pitch2.54mm" H 7150 5250 50  0001 C CNN
 F 3 "~" H 7150 5250 50  0001 C CNN
+F 4 "S9337-ND" H 0   0   50  0001 C CNN "DigiKey"
 	1    7150 5250
 	1    0    0    -1
@@
 F 2 "Pin_Headers:Pin_Header_Straight_1x02_Pitch2.54mm" H 7150 4850 50  0001 C CNN
 F 3 "~" H 7150 4850 50  0001 C CNN
+F 4 "S9337-ND" H 0   0   50  0001 C CNN "DigiKey"
 	1    7150 4850
 	1    0    0    -1
@@
 F 2 "Pin_Headers:Pin_Header_Straight_1x02_Pitch2.54mm" H 9050 4050 50  0001 C CNN
 F 3 "~" H 9050 4050 50  0001 C CNN
+F 4 "S9337-ND" H 0   0   50  0001 C CNN "DigiKey"
 	1    9050 4050
 	1    0    0    -1
@@
 F 2 "Pin_Headers:Pin_Header_Straight_1x02_Pitch2.54mm" H 9050 4450 50  0001 C CNN
 F 3 "~" H 9050 4450 50  0001 C CNN
+F 4 "S9337-ND" H 0   0   50  0001 C CNN "DigiKey"
 	1    9050 4450
 	1    0    0    -1
@@
 F 2 "Pin_Headers:Pin_Header_Straight_1x02_Pitch2.54mm" H 7150 6250 50  0001 C CNN
 F 3 "~" H 7150 6250 50  0001 C CNN
+F 4 "S9337-ND" H 0   0   50  0001 C CNN "DigiKey"
 	1    7150 6250
 	1    0    0    -1
@@
 F 2 "Pin_Headers:Pin_Header_Straight_1x02_Pitch2.54mm" H 9150 6250 50  0001 C CNN
 F 3 "~" H 9150 6250 50  0001 C CNN
+F 4 "S9337-ND" H 0   0   50  0001 C CNN "DigiKey"
 	1    9150 6250
 	1    0    0    -1
@@
 F 2 "Pin_Headers:Pin_Header_Straight_1x02_Pitch2.54mm" H 9150 6650 50  0001 C CNN
 F 3 "~" H 9150 6650 50  0001 C CNN
+F 4 "S9337-ND" H 0   0   50  0001 C CNN "DigiKey"
 	1    9150 6650
 	1    0    0    -1
@@
 F 2 "Speeduino Mini:ED120_3DS" H 1350 5850 50  0001 C CNN
 F 3 "~" H 1350 5850 50  0001 C CNN
-F 4 "ED1610-ND" H 1430 5755 50  0000 L CNN "DIGIKEY"
+F 4 "ED1610-ND" H 0   0   50  0001 C CNN "DigiKey"
 	1    1350 5850
 	-1   0    0    -1
@@
 F 2 "Speeduino Mini:ED120_2DS" H 1250 4600 50  0001 C CNN
 F 3 "http://www.on-shore.com/wp-content/uploads/2015/09/ed120ds.pdf" H 1250 4600 50  0001 C CNN
-F 4 "ED1609-ND" H 1330 4455 50  0000 L CNN "DIGIKEY"
+F 4 "ED1609-ND" H 0   0   50  0001 C CNN "DigiKey"
 	1    1250 4600
 	-1   0    0    -1
@@
 F 2 "Pin_Headers:Pin_Header_Straight_1x02_Pitch2.54mm" H 1750 2200 50  0001 C CNN
 F 3 "~" H 1750 2200 50  0001 C CNN
+F 4 "S9337-ND" H 0   0   50  0001 C CNN "DigiKey"
 	1    1750 2200
 	1    0    0    -1
@@
 F 2 "Mounting_Holes:MountingHole_4.3mm_M4_Pad_Via" H 10500 800 50  0001 C CNN
 F 3 "~" H 10500 800 50  0001 C CNN
+F 4 "1772-4097-ND" H 0   0   50  0001 C CNN "DigiKey"
 	1    10500 800
 	1    0    0    -1
@@
 F 2 "Mounting_Holes:MountingHole_4.3mm_M4_Pad_Via" H 10500 1000 50  0001 C CNN
 F 3 "~" H 10500 1000 50  0001 C CNN
+F 4 "1772-4097-ND" H 0   0   50  0001 C CNN "DigiKey"
 	1    10500 1000
 	1    0    0    -1
@@
 F 2 "Mounting_Holes:MountingHole_4.3mm_M4_Pad_Via" H 10500 1200 50  0001 C CNN
 F 3 "~" H 10500 1200 50  0001 C CNN
+F 4 "1772-4097-ND" H 0   0   50  0001 C CNN "DigiKey"
 	1    10500 1200
 	1    0    0    -1
@@
 F 2 "Mounting_Holes:MountingHole_4.3mm_M4_Pad_Via" H 10500 1400 50  0001 C CNN
 F 3 "~" H 10500 1400 50  0001 C CNN
+F 4 "1772-4097-ND" H 0   0   50  0001 C CNN "DigiKey"
 	1    10500 1400
 	1    0    0    -1

Commit message: old commit from v1
Other:
- note added: "TODO add missing 1k pull-up on hall sensors"
Changed lines of the file:
@@
 EESchema Schematic File Version 4
-LIBS:speeduino_mini-cache
-EELAYER 29 0
+EELAYER 30 0
 EELAYER END
-$Descr A4 11693 8268
+$Descr A3 16535 11693
 encoding utf-8
-Sheet 1 22
+Sheet 1 23
 Title ""
 Date ""
@@
 Wire Wire Line
 	6700 6750 6500 6750
+Text Notes 4200 0    0    50   ~ 0
+TODO add missing 1k pull-up on hall sensors
+$Sheet
+S 7350 7650 1350 1050
+U 5EAF1046
+F0 "Throttle" 50
+F1 "throttle.sch" 50
+$EndSheet
 $EndSCHEMATC
