File: hardware/temperature_sensor.sch (KiCad schematic (older format))
At the start: 4 parts

Commit message: rev 1.1
Changed lines of the file:
@@
 $Descr A4 11693 8268
 encoding utf-8
-Sheet 7 21
+Sheet 6 21
 Title ""
 Date ""
@@
 AR Path="/5C65B4AD/5C65E136" Ref="R2"  Part="1"
 AR Path="/5C65E0B2/5C65E136" Ref="R4"  Part="1"
-F 0 "R4" H 5670 2891 50  0000 L CNN
+F 0 "R2" H 5670 2891 50  0000 L CNN
 F 1 "2.49k" H 5670 2800 50  0000 L CNN
 F 2 "Resistors_SMD:R_0805" V 5530 2800 50  0001 C CNN
@@
 AR Path="/5C65B4AD/5C65E15E" Ref="R3"  Part="1"
 AR Path="/5C65E0B2/5C65E15E" Ref="R5"  Part="1"
-F 0 "R5" V 6003 3550 50  0000 C CNN
+F 0 "R3" V 6003 3550 50  0000 C CNN
 F 1 "470" V 6094 3550 50  0000 C CNN
 F 2 "Resistors_SMD:R_0805" V 6230 3550 50  0001 C CNN
@@
 AR Path="/5C65B4AD/5C65E1D6" Ref="#PWR026"  Part="1"
 AR Path="/5C65E0B2/5C65E1D6" Ref="#PWR055"  Part="1"
-F 0 "#PWR055" H 6400 4100 50  0001 C CNN
+F 0 "#PWR026" H 6400 4100 50  0001 C CNN
 F 1 "GND" H 6405 4177 50  0000 C CNN
 F 2 "" H 6400 4350 50  0001 C CNN
@@
 AR Path="/5C65E0B2/5C6BC0ED" Ref="C17"  Part="1"
 AR Path="/5C65B4AD/5C6BC0ED" Ref="C14"  Part="1"
-F 0 "C17" H 5715 4041 50  0000 L CNN
+F 0 "C14" H 5715 4041 50  0000 L CNN
 F 1 "0.1uF" H 5715 3950 50  0000 L CNN
 F 2 "Capacitors_SMD:C_0805" H 5638 3800 50  0001 C CNN
@@
 AR Path="/5C65E0B2/5C6BC0F5" Ref="C18"  Part="1"
 AR Path="/5C65B4AD/5C6BC0F5" Ref="C15"  Part="1"
-F 0 "C18" H 6865 4041 50  0000 L CNN
+F 0 "C15" H 6865 4041 50  0000 L CNN
 F 1 "0.22u" H 6865 3950 50  0000 L CNN
 F 2 "Capacitors_SMD:C_0805" H 6788 3800 50  0001 C CNN
@@
 AR Path="/5C65B4AD/5C6EAF6B" Ref="#PWR024"  Part="1"
 AR Path="/5C65E0B2/5C6EAF6B" Ref="#PWR054"  Part="1"
-F 0 "#PWR054" H 5600 2400 50  0001 C CNN
+F 0 "#PWR024" H 5600 2400 50  0001 C CNN
 F 1 "+5VA" H 5615 2723 50  0000 C CNN
 F 2 "" H 5600 2550 50  0001 C CNN

Commit message: Rev 2 work in progress
Parts:
- C17, C18: footprint Capacitors_SMD:C_0805 -> Capacitors_SMD:C_0805_HandSoldering
- R2, R3: footprint Resistors_SMD:R_0805 -> Resistors_SMD:R_0805_HandSoldering
Connections:
- net +5VA renamed VCC
Changed lines of the file:
@@
 $Descr A4 11693 8268
 encoding utf-8
-Sheet 6 21
+Sheet 23 23
 Title ""
 Date ""
@@
 AR Path="/5C65B4AD/5C65E136" Ref="R2"  Part="1"
 AR Path="/5C65E0B2/5C65E136" Ref="R4"  Part="1"
-F 0 "R2" H 5670 2891 50  0000 L CNN
+F 0 "R4" H 5670 2891 50  0000 L CNN
 F 1 "2.49k" H 5670 2800 50  0000 L CNN
-F 2 "Resistors_SMD:R_0805" V 5530 2800 50  0001 C CNN
+F 2 "Resistors_SMD:R_0805_HandSoldering" V 5530 2800 50  0001 C CNN
 F 3 "~" H 5600 2800 50  0001 C CNN
 F 4 "P2.49KDACT-ND" H 5670 2709 50  0000 L CNN "DIGIKEY"
@@
 AR Path="/5C65B4AD/5C65E15E" Ref="R3"  Part="1"
 AR Path="/5C65E0B2/5C65E15E" Ref="R5"  Part="1"
-F 0 "R3" V 6003 3550 50  0000 C CNN
+F 0 "R5" V 6003 3550 50  0000 C CNN
 F 1 "470" V 6094 3550 50  0000 C CNN
-F 2 "Resistors_SMD:R_0805" V 6230 3550 50  0001 C CNN
+F 2 "Resistors_SMD:R_0805_HandSoldering" V 6230 3550 50  0001 C CNN
 F 3 "~" H 6300 3550 50  0001 C CNN
 F 4 "311-470ARCT-ND" V 6185 3550 50  0000 C CNN "DIGIKEY"
@@
 AR Path="/5C65E0B2/5C6BC0ED" Ref="C17"  Part="1"
 AR Path="/5C65B4AD/5C6BC0ED" Ref="C14"  Part="1"
-F 0 "C14" H 5715 4041 50  0000 L CNN
+F 0 "C17" H 5715 4041 50  0000 L CNN
 F 1 "0.1uF" H 5715 3950 50  0000 L CNN
-F 2 "Capacitors_SMD:C_0805" H 5638 3800 50  0001 C CNN
+F 2 "Capacitors_SMD:C_0805_HandSoldering" H 5638 3800 50  0001 C CNN
 F 3 "~" H 5600 3950 50  0001 C CNN
 F 4 "478-6048-1-ND" H 5715 3859 50  0000 L CNN "DIGIKEY"
@@
 AR Path="/5C65E0B2/5C6BC0F5" Ref="C18"  Part="1"
 AR Path="/5C65B4AD/5C6BC0F5" Ref="C15"  Part="1"
-F 0 "C15" H 6865 4041 50  0000 L CNN
+F 0 "C18" H 6865 4041 50  0000 L CNN
 F 1 "0.22u" H 6865 3950 50  0000 L CNN
-F 2 "Capacitors_SMD:C_0805" H 6788 3800 50  0001 C CNN
+F 2 "Capacitors_SMD:C_0805_HandSoldering" H 6788 3800 50  0001 C CNN
 F 3 "~" H 6750 3950 50  0001 C CNN
 F 4 "1276-7012-1-ND" H 6865 3859 50  0000 L CNN "DIGIKEY"
@@
 	1    0    0    -1
 $EndComp
-$Comp
-L power:+5VA #PWR024
-U 1 1 5C6EAF6B
-P 5600 2550
-AR Path="/5C65B4AD/5C6EAF6B" Ref="#PWR024"  Part="1"
-AR Path="/5C65E0B2/5C6EAF6B" Ref="#PWR054"  Part="1"
-F 0 "#PWR054" H 5600 2400 50  0001 C CNN
-F 1 "+5VA" H 5615 2723 50  0000 C CNN
-F 2 "" H 5600 2550 50  0001 C CNN
-F 3 "" H 5600 2550 50  0001 C CNN
-	1    5600 2550
-	1    0    0    -1
-$EndComp
+Text HLabel 5600 2550 1    50   Input ~ 0
+VCC
 $EndSCHEMATC

Commit message: hardware rev2 - layout complete
Parts:
- added JP16: Jumper, Pin_Headers:Pin_Header_Straight_1x02_Pitch2.54mm, symbol Device:Jumper
Connections:
- net IN: now also JP16.1; no longer C17.1, R3.2
- new net: C17.1, JP16.2, R3.2
Other:
- moved on the sheet: R2
Changed lines of the file:
@@
 $Descr A4 11693 8268
 encoding utf-8
-Sheet 23 22
+Sheet 5 22
 Title ""
 Date ""
@@
 Comment4 ""
 $EndDescr
-Text HLabel 5350 3550 0    50   Input ~ 0
+Text HLabel 4450 3550 0    50   Input ~ 0
 IN
 $Comp
 L Device:R R2
 U 1 1 5C65E136
-P 5600 2800
+P 4600 2800
 AR Path="/5C65B4AD/5C65E136" Ref="R2"  Part="1"
 AR Path="/5C65E0B2/5C65E136" Ref="R4"  Part="1"
-F 0 "R4" H 5670 2891 50  0000 L CNN
-F 1 "2.49k" H 5670 2800 50  0000 L CNN
-F 2 "Resistors_SMD:R_0805_HandSoldering" V 5530 2800 50  0001 C CNN
-F 3 "~" H 5600 2800 50  0001 C CNN
-F 4 "P2.49KDACT-ND" H 5670 2709 50  0000 L CNN "DIGIKEY"
-	1    5600 2800
+F 0 "R2" H 4670 2891 50  0000 L CNN
+F 1 "2.49k" H 4670 2800 50  0000 L CNN
+F 2 "Resistors_SMD:R_0805_HandSoldering" V 4530 2800 50  0001 C CNN
+F 3 "~" H 4600 2800 50  0001 C CNN
+F 4 "P2.49KDACT-ND" H 4670 2709 50  0000 L CNN "DIGIKEY"
+	1    4600 2800
 	1    0    0    -1
 $EndComp
@@
 AR Path="/5C65B4AD/5C65E15E" Ref="R3"  Part="1"
 AR Path="/5C65E0B2/5C65E15E" Ref="R5"  Part="1"
-F 0 "R5" V 6003 3550 50  0000 C CNN
+F 0 "R3" V 6003 3550 50  0000 C CNN
 F 1 "470" V 6094 3550 50  0000 C CNN
 F 2 "Resistors_SMD:R_0805_HandSoldering" V 6230 3550 50  0001 C CNN
@@
 	5350 3550 5600 3550
 Wire Wire Line
-	5600 2950 5600 3550
+	4600 2950 4600 3550
 Connection ~ 5600 3550
 Wire Wire Line
@@
 	5600 3550 5600 3800
 Wire Wire Line
-	5600 2650 5600 2550
+	4600 2650 4600 2550
 Text HLabel 7300 3550 2    50   Output ~ 0
 OUT
@@
 AR Path="/5C65E0B2/5C6BC0ED" Ref="C17"  Part="1"
 AR Path="/5C65B4AD/5C6BC0ED" Ref="C14"  Part="1"
-F 0 "C17" H 5715 4041 50  0000 L CNN
+F 0 "C14" H 5715 4041 50  0000 L CNN
 F 1 "0.1uF" H 5715 3950 50  0000 L CNN
 F 2 "Capacitors_SMD:C_0805_HandSoldering" H 5638 3800 50  0001 C CNN
@@
 AR Path="/5C65E0B2/5C6BC0F5" Ref="C18"  Part="1"
 AR Path="/5C65B4AD/5C6BC0F5" Ref="C15"  Part="1"
-F 0 "C18" H 6865 4041 50  0000 L CNN
+F 0 "C15" H 6865 4041 50  0000 L CNN
 F 1 "0.22u" H 6865 3950 50  0000 L CNN
 F 2 "Capacitors_SMD:C_0805_HandSoldering" H 6788 3800 50  0001 C CNN
@@
 	1    0    0    -1
 $EndComp
-Text HLabel 5600 2550 1    50   Input ~ 0
+Text HLabel 4600 2550 1    50   Input ~ 0
 VCC
+$Comp
+L Device:Jumper JP?
+U 1 1 5D011A46
+P 5050 3550
+AR Path="/5D011A46" Ref="JP?"  Part="1"
+AR Path="/5C65B4AD/5D011A46" Ref="JP16"  Part="1"
+AR Path="/5C65E0B2/5D011A46" Ref="JP17"  Part="1"
+F 0 "JP16" H 5050 3814 50  0000 C CNN
+F 1 "Jumper" H 5050 3723 50  0000 C CNN
+F 2 "Pin_Headers:Pin_Header_Straight_1x02_Pitch2.54mm" H 5050 3550 50  0001 C CNN
+F 3 "~" H 5050 3550 50  0001 C CNN
+	1    5050 3550
+	1    0    0    -1
+$EndComp
+Wire Wire Line
+	4450 3550 4600 3550
+Connection ~ 4600 3550
+Wire Wire Line
+	4600 3550 4750 3550
 $EndSCHEMATC

Commit message: rev 2 sent to fab
Parts:
- C17: value 0.1uF -> 0.1uF 50V; DIGIKEY 478-6048-1-ND -> (none); DigiKey (none) -> 478-6048-1-ND
- C18: value 0.22u -> 0.22uF 50V; DIGIKEY 1276-7012-1-ND -> (none); DigiKey (none) -> 445-5683-1-ND
- JP16: DigiKey (none) -> S9337-ND
- R2: DIGIKEY P2.49KDACT-ND -> (none); DigiKey (none) -> P2.49KDACT-ND
- R3: DIGIKEY 311-470ARCT-ND -> (none); DigiKey (none) -> 311-470ARCT-ND
Changed lines of the file:
@@
 AR Path="/5C65B4AD/5C65E136" Ref="R2"  Part="1"
 AR Path="/5C65E0B2/5C65E136" Ref="R4"  Part="1"
-F 0 "R2" H 4670 2891 50  0000 L CNN
+F 0 "R4" H 4670 2891 50  0000 L CNN
 F 1 "2.49k" H 4670 2800 50  0000 L CNN
 F 2 "Resistors_SMD:R_0805_HandSoldering" V 4530 2800 50  0001 C CNN
 F 3 "~" H 4600 2800 50  0001 C CNN
-F 4 "P2.49KDACT-ND" H 4670 2709 50  0000 L CNN "DIGIKEY"
+F 4 "P2.49KDACT-ND" H 0   0   50  0001 C CNN "DigiKey"
 	1    4600 2800
 	1    0    0    -1
@@
 AR Path="/5C65B4AD/5C65E15E" Ref="R3"  Part="1"
 AR Path="/5C65E0B2/5C65E15E" Ref="R5"  Part="1"
-F 0 "R3" V 6003 3550 50  0000 C CNN
+F 0 "R5" V 6003 3550 50  0000 C CNN
 F 1 "470" V 6094 3550 50  0000 C CNN
 F 2 "Resistors_SMD:R_0805_HandSoldering" V 6230 3550 50  0001 C CNN
 F 3 "~" H 6300 3550 50  0001 C CNN
-F 4 "311-470ARCT-ND" V 6185 3550 50  0000 C CNN "DIGIKEY"
+F 4 "311-470ARCT-ND" H 0   0   50  0001 C CNN "DigiKey"
 	1    6300 3550
 	0    1    1    0
@@
 AR Path="/5C65E0B2/5C6BC0ED" Ref="C17"  Part="1"
 AR Path="/5C65B4AD/5C6BC0ED" Ref="C14"  Part="1"
-F 0 "C14" H 5715 4041 50  0000 L CNN
-F 1 "0.1uF" H 5715 3950 50  0000 L CNN
+F 0 "C17" H 5715 4041 50  0000 L CNN
+F 1 "0.1uF 50V" H 5715 3950 50  0000 L CNN
 F 2 "Capacitors_SMD:C_0805_HandSoldering" H 5638 3800 50  0001 C CNN
 F 3 "~" H 5600 3950 50  0001 C CNN
-F 4 "478-6048-1-ND" H 5715 3859 50  0000 L CNN "DIGIKEY"
+F 4 "478-6048-1-ND" H 0   0   50  0001 C CNN "DigiKey"
 	1    5600 3950
 	1    0    0    -1
@@
 AR Path="/5C65E0B2/5C6BC0F5" Ref="C18"  Part="1"
 AR Path="/5C65B4AD/5C6BC0F5" Ref="C15"  Part="1"
-F 0 "C15" H 6865 4041 50  0000 L CNN
-F 1 "0.22u" H 6865 3950 50  0000 L CNN
+F 0 "C18" H 6865 4041 50  0000 L CNN
+F 1 "0.22uF 50V" H 6865 3950 50  0000 L CNN
 F 2 "Capacitors_SMD:C_0805_HandSoldering" H 6788 3800 50  0001 C CNN
 F 3 "~" H 6750 3950 50  0001 C CNN
-F 4 "1276-7012-1-ND" H 6865 3859 50  0000 L CNN "DIGIKEY"
+F 4 "445-5683-1-ND" H 0   0   50  0001 C CNN "DigiKey"
 	1    6750 3950
 	1    0    0    -1
@@
 AR Path="/5C65B4AD/5D011A46" Ref="JP16"  Part="1"
 AR Path="/5C65E0B2/5D011A46" Ref="JP17"  Part="1"
-F 0 "JP16" H 5050 3814 50  0000 C CNN
+F 0 "JP17" H 5050 3814 50  0000 C CNN
 F 1 "Jumper" H 5050 3723 50  0000 C CNN
 F 2 "Pin_Headers:Pin_Header_Straight_1x02_Pitch2.54mm" H 5050 3550 50  0001 C CNN
 F 3 "~" H 5050 3550 50  0001 C CNN
+F 4 "S9337-ND" H 0   0   50  0001 C CNN "DigiKey"
 	1    5050 3550
 	1    0    0    -1
